File: GPIO.kicad_sch (KiCad schematic)
At the start: 72 parts, among them U401 MCP23S17_SS, U402 MCP23S17_SS, U403 MCP23S17_SS, U404 MCP23S17_SS, U405 MCP23S17_SS, U406 MCP23S17_SS, U407 MCP23S17_SS, U408 MCP23S17_SS

Commit message: update
Parts:
- removed U401, U402, U403, U404, U405, U406, U407, U408: MCP23S17_SS, Package_SO:SSOP-28_5.3x10.2mm_P0.65mm, symbol Interface_Expansion:MCP23S17_SS
- added U401, U402, U403, U404, U405, U406, U407, U408: MCP23017_SS, Package_SO:SSOP-28_5.3x10.2mm_P0.65mm, symbol Interface_Expansion:MCP23017_SS
Connections:
- net +3V3: now also U401.9 (VDD), U402.9 (VDD), U403.9 (VDD), U404.9 (VDD), U405.9 (VDD), U406.9 (VDD), U407.9 (VDD), U408.9 (VDD)
- net GND: now also U401.10 (VSS), U402.10 (VSS), U403.10 (VSS), U404.10 (VSS), U405.10 (VSS), U406.10 (VSS), U407.10 (VSS), U408.10 (VSS)
- net IO.SCK: now also U401.12 (SCK), U402.12 (SCK), U403.12 (SCK), U404.12 (SCK), U405.12 (SCK), U406.12 (SCK), U407.12 (SCK), U408.12 (SCK)
- net IO0: now also U401.1 (GPB0)
- net IO1: now also U401.2 (GPB1)
- net IO10: now also U401.23 (GPA2)
- net IO100: now also U407.5 (GPB4)
- net IO101: now also U407.6 (GPB5)
- net IO102: now also U407.7 (GPB6)
- net IO103: now also U407.8 (GPB7)
- net IO104: now also U407.21 (GPA0)
- net IO105: now also U407.22 (GPA1)
- net IO106: now also U407.23 (GPA2)
- net IO107: now also U407.24 (GPA3)
- net IO108: now also U407.25 (GPA4)
- net IO109: now also U407.26 (GPA5)
- net IO11: now also U401.24 (GPA3)
- net IO110: now also U407.27 (GPA6)
- net IO111: now also U407.28 (GPA7)
- net IO112: now also U408.1 (GPB0)
- net IO113: now also U408.2 (GPB1)
- net IO114: now also U408.3 (GPB2)
- net IO115: now also U408.4 (GPB3)
- net IO116: now also U408.5 (GPB4)
- net IO117: now also U408.6 (GPB5)
- net IO118: now also U408.7 (GPB6)
- net IO119: now also U408.8 (GPB7)
- net IO12: now also U401.25 (GPA4)
- net IO120: now also U408.21 (GPA0)
- net IO121: now also U408.22 (GPA1)
- net IO122: now also U408.23 (GPA2)
- net IO123: now also U408.24 (GPA3)
- net IO124: now also U408.25 (GPA4)
- net IO125: now also U408.26 (GPA5)
- net IO126: now also U408.27 (GPA6)
- net IO127: now also U408.28 (GPA7)
- net IO13: now also U401.26 (GPA5)
- net IO14: now also U401.27 (GPA6)
- net IO15: now also U401.28 (GPA7)
- net IO16: now also U402.1 (GPB0)
- net IO17: now also U402.2 (GPB1)
- net IO18: now also U402.3 (GPB2)
- net IO19: now also U402.4 (GPB3)
- net IO2: now also U401.3 (GPB2)
- net IO20: now also U402.5 (GPB4)
- net IO21: now also U402.6 (GPB5)
- net IO22: now also U402.7 (GPB6)
- net IO23: now also U402.8 (GPB7)
- net IO24: now also U402.21 (GPA0)
- net IO25: now also U402.22 (GPA1)
- net IO26: now also U402.23 (GPA2)
- net IO27: now also U402.24 (GPA3)
- net IO28: now also U402.25 (GPA4)
- net IO29: now also U402.26 (GPA5)
- net IO3: now also U401.4 (GPB3)
- net IO30: now also U402.27 (GPA6)
- net IO31: now also U402.28 (GPA7)
- net IO32: now also U403.1 (GPB0)
- net IO33: now also U403.2 (GPB1)
- net IO34: now also U403.3 (GPB2)
- net IO35: now also U403.4 (GPB3)
- net IO36: now also U403.5 (GPB4)
- net IO37: now also U403.6 (GPB5)
- net IO38: now also U403.7 (GPB6)
- net IO39: now also U403.8 (GPB7)
- net IO4: now also U401.5 (GPB4)
- net IO40: now also U403.21 (GPA0)
- net IO41: now also U403.22 (GPA1)
- net IO42: now also U403.23 (GPA2)
- net IO43: now also U403.24 (GPA3)
- net IO44: now also U403.25 (GPA4)
- net IO45: now also U403.26 (GPA5)
- net IO46: now also U403.27 (GPA6)
- net IO47: now also U403.28 (GPA7)
- net IO48: now also U404.1 (GPB0)
- net IO49: now also U404.2 (GPB1)
- net IO5: now also U401.6 (GPB5)
- net IO50: now also U404.3 (GPB2)
- net IO51: now also U404.4 (GPB3)
- net IO52: now also U404.5 (GPB4)
- net IO53: now also U404.6 (GPB5)
- net IO54: now also U404.7 (GPB6)
- net IO55: now also U404.8 (GPB7)
- net IO56: now also U404.21 (GPA0)
- net IO57: now also U404.22 (GPA1)
- net IO58: now also U404.23 (GPA2)
- net IO59: now also U404.24 (GPA3)
- net IO6: now also U401.7 (GPB6)
- net IO60: now also U404.25 (GPA4)
- net IO61: now also U404.26 (GPA5)
- net IO62: now also U404.27 (GPA6)
- net IO63: now also U404.28 (GPA7)
- net IO64: now also U405.1 (GPB0)
- net IO65: now also U405.2 (GPB1)
- net IO66: now also U405.3 (GPB2)
- net IO67: now also U405.4 (GPB3)
- net IO68: now also U405.5 (GPB4)
- net IO69: now also U405.6 (GPB5)
- net IO7: now also U401.8 (GPB7)
- net IO70: now also U405.7 (GPB6)
- net IO71: now also U405.8 (GPB7)
- net IO72: now also U405.21 (GPA0)
- net IO73: now also U405.22 (GPA1)
- net IO74: now also U405.23 (GPA2)
- net IO75: now also U405.24 (GPA3)
- net IO76: now also U405.25 (GPA4)
- net IO77: now also U405.26 (GPA5)
- net IO78: now also U405.27 (GPA6)
- net IO79: now also U405.28 (GPA7)
- net IO8: now also U401.21 (GPA0)
- net IO80: now also U406.1 (GPB0)
- net IO81: now also U406.2 (GPB1)
- net IO82: now also U406.3 (GPB2)
- net IO83: now also U406.4 (GPB3)
- net IO84: now also U406.5 (GPB4)
- net IO85: now also U406.6 (GPB5)
- net IO86: now also U406.7 (GPB6)
- net IO87: now also U406.8 (GPB7)
- net IO88: now also U406.21 (GPA0)
- net IO89: now also U406.22 (GPA1)
- net IO9: now also U401.22 (GPA1)
- net IO90: now also U406.23 (GPA2)
- net IO91: now also U406.24 (GPA3)
- net IO92: now also U406.25 (GPA4)
- net IO93: now also U406.26 (GPA5)
- net IO94: now also U406.27 (GPA6)
- net IO95: now also U406.28 (GPA7)
- net IO96: now also U407.1 (GPB0)
- net IO97: now also U407.2 (GPB1)
- net IO98: now also U407.3 (GPB2)
- net IO99: now also U407.4 (GPB3)
- net at JP406.2 (B), R409.1: now also U402.16 (A1)
- net at R418.2: now also U406.18 (~{RESET})
- net at JP405.2 (B), R406.1: now also U401.16 (A1)
- net at R420.2: now also U408.18 (~{RESET})
- net at JP412.2 (B), R416.1: now also U404.15 (A0)
- net at JP419.2 (B), R428.1: now also U407.16 (A1)
- net at JP424.2 (B), R432.1: now also U408.15 (A0)
- net at R401.2: now also U401.18 (~{RESET})
- net at JP402.2 (B), R408.1: now also U402.17 (A2)
- net at JP404.2 (B), R414.1: now also U404.17 (A2)
- net at JP423.2 (B), R429.1: now also U407.15 (A0)
- net at JP410.2 (B), R410.1: now also U402.15 (A0)
- net at JP408.2 (B), R415.1: now also U404.16 (A1)
- net at R404.2: now also U404.18 (~{RESET})
- net at RN404.2 (R2.1): now also U404.19 (INTB)
- net at RN404.1 (R1.1): now also U404.20 (INTA)
- net at R402.2: now also U402.18 (~{RESET})
- net at RN408.1 (R1.1): now also U408.20 (INTA)
- net at RN408.2 (R2.1): now also U408.19 (INTB)
- net at JP401.2 (B), R405.1: now also U401.17 (A2)
- net at JP416.2 (B), R430.1: now also U408.17 (A2)
- net at JP407.2 (B), R412.1: now also U403.16 (A1)
- net at RN402.1 (R1.1): now also U402.20 (INTA)
- net at RN402.2 (R2.1): now also U402.19 (INTB)
- net at JP417.2 (B), R422.1: now also U405.16 (A1)
- net at JP421.2 (B), R423.1: now also U405.15 (A0)
- net at JP403.2 (B), R411.1: now also U403.17 (A2)
- net at JP422.2 (B), R426.1: now also U406.15 (A0)
- net at JP411.2 (B), R413.1: now also U403.15 (A0)
- net at JP418.2 (B), R425.1: now also U406.16 (A1)
- net at R419.2: now also U407.18 (~{RESET})
- net at JP420.2 (B), R431.1: now also U408.16 (A1)
- net at JP413.2 (B), R421.1: now also U405.17 (A2)
- net at JP409.2 (B), R407.1: now also U401.15 (A0)
- net at RN401.2 (R2.1): now also U401.19 (INTB)
- net at RN401.1 (R1.1): now also U401.20 (INTA)
- net at JP414.2 (B), R424.1: now also U406.17 (A2)
- net at JP415.2 (B), R427.1: now also U407.17 (A2)
- net at RN407.1 (R1.1): now also U407.20 (INTA)
- net at RN407.2 (R2.1): now also U407.19 (INTB)
- net at RN403.1 (R1.1): now also U403.20 (INTA)
- net at RN403.2 (R2.1): now also U403.19 (INTB)
- net at R403.2: now also U403.18 (~{RESET})
- net at RN406.1 (R1.1): now also U406.20 (INTA)
- net at RN406.2 (R2.1): now also U406.19 (INTB)
- net at R417.2: now also U405.18 (~{RESET})
- net at RN405.1 (R1.1): now also U405.20 (INTA)
- net at RN405.2 (R2.1): now also U405.19 (INTB)
- new net IO.SDA: U401.13 (SDA), U402.13 (SDA), U403.13 (SDA), U404.13 (SDA), U405.13 (SDA), U406.13 (SDA), U407.13 (SDA), U408.13 (SDA)
