File: GPIO.kicad_sch (KiCad schematic)
At the start: 56 parts

Commit message: Update
Parts:
- removed RN? (x8): 10k, symbol Device:R_Pack03
- added R405, R406, R407, R408, R409, R410, R411, R412, R413, R414, R415, R416, R421, R422, R423, R424, R425, R426, R427, R428, R429, R430, R431, R432: 10k, Resistor_SMD:R_0402_1005Metric, symbol Device:R
- JP401, JP402, JP403, JP404, JP405, JP406, JP409, JP411, JP417, JP418, JP421, JP423: renamed from JP?; footprint (none) -> Jumper:SolderJumper-2_P1.3mm_Open_TrianglePad1.0x1.5mm
- JP407, JP408, JP410, JP412, JP413, JP414, JP415, JP416, JP419, JP420, JP422, JP424: renamed from JP?; footprint (none) -> Jumper:SolderJumper-2_P1.3mm_Bridged_Pad1.0x1.5mm
- R401, R402, R403, R404, R417, R418, R419, R420: renamed from R?; value R -> 10k; footprint (none) -> Resistor_SMD:R_0402_1005Metric
- RN401, RN402, RN403, RN404, RN405, RN406, RN407, RN408: renamed from RN?; footprint (none) -> Resistor_SMD:R_Array_Convex_2x0402
- gave numbers to parts that had none: 8
Connections:
- net GND: now also R405.2, R406.2, R407.2, R408.2, R409.2, R410.2, R411.2, R412.2, R413.2, R414.2, R415.2, R416.2, R421.2, R422.2, R423.2, R424.2, R425.2, R426.2, R427.2, R428.2, R429.2, R430.2, R431.2, R432.2
- net at JP405.2 (B), U401.16 (A1): now also R406.1
- net at JP412.2 (B), U404.15 (A0): now also R416.1
- net at JP424.2 (B), U408.15 (A0): now also R432.1
- net at JP421.2 (B), U405.15 (A0): now also R423.1
- net at JP417.2 (B), U405.16 (A1): now also R422.1
- net at JP413.2 (B), U405.17 (A2): now also R421.1
- net at JP408.2 (B), U404.16 (A1): now also R415.1
- net at JP404.2 (B), U404.17 (A2): now also R414.1
- net at JP410.2 (B), U402.15 (A0): now also R410.1
- net at JP407.2 (B), U403.16 (A1): now also R412.1
- net at JP423.2 (B), U407.15 (A0): now also R429.1
- net at JP419.2 (B), U407.16 (A1): now also R428.1
- net at JP415.2 (B), U407.17 (A2): now also R427.1
- net at JP406.2 (B), U402.16 (A1): now also R409.1
- net at JP402.2 (B), U402.17 (A2): now also R408.1
- net at JP422.2 (B), U406.15 (A0): now also R426.1
- net at JP411.2 (B), U403.15 (A0): now also R413.1
- net at JP420.2 (B), U408.16 (A1): now also R431.1
- net at JP416.2 (B), U408.17 (A2): now also R430.1
- net at JP409.2 (B), U401.15 (A0): now also R407.1
- net at JP401.2 (B), U401.17 (A2): now also R405.1
- net at JP418.2 (B), U406.16 (A1): now also R425.1
- net at JP414.2 (B), U406.17 (A2): now also R424.1
- net at JP403.2 (B), U403.17 (A2): now also R411.1

Commit message: Complete SPI Design
Parts:
- added C401, C402, C403, C404, C405, C406, C407, C408: 0.1u, Capacitor_SMD:C_0402_1005Metric, symbol Device:C
- R401, R402, R403, R404, R405, R406, R407, R408, R409, R410, R411, R412, R413, R414, R415, R416, R417, R418, R419, R420, R421, R422, R423, R424, R425, R426, R427, R428, R429, R430, R431, R432: LCSC (none) -> C140214; LCSC Part Number (none) -> C140214
- RN401, RN402, RN403, RN404, RN405, RN406, RN407, RN408: LCSC (none) -> C695179; LCSC Part Number (none) -> C695179
- U401, U402, U403, U404, U405, U406, U407, U408: value MCP23S17_SS -> MCP23S17T-E/SS; LCSC (none) -> C128577; LCSC Part Number (none) -> C128577
Connections:
- net +3V3: now also C401.2, C402.2, C403.2, C404.2, C405.2, C406.2, C407.2, C408.2
- net GND: now also C401.1, C402.1, C403.1, C404.1, C405.1, C406.1, C407.1, C408.1
- net IO.SDI: now also U401.14 (SO), U402.14 (SO), U403.14 (SO), U404.14 (SO), U405.14 (SO), U406.14 (SO), U407.14 (SO), U408.14 (SO); no longer U401.13 (SI), U402.13 (SI), U403.13 (SI), U404.13 (SI), U405.13 (SI), U406.13 (SI), U407.13 (SI), U408.13 (SI)
- net IO.SDO: now also U401.13 (SI), U402.13 (SI), U403.13 (SI), U404.13 (SI), U405.13 (SI), U406.13 (SI), U407.13 (SI), U408.13 (SI); no longer U401.14 (SO), U402.14 (SO), U403.14 (SO), U404.14 (SO), U405.14 (SO), U406.14 (SO), U407.14 (SO), U408.14 (SO)
- net IO0 renamed IO.HWCLK
- net IO1 renamed IO.PB20
- net IO10 renamed IO.PB11
- net IO100 renamed IO.RIGHT3
- net IO101 renamed IO.RIGHT2
- net IO102 renamed IO.RIGHT1
- net IO103 renamed IO.RIGHT0
- net IO104 renamed IO.RED
- net IO105 renamed IO.GREEN
- net IO106 renamed IO.BLUE
- net IO107: no longer names the net of U407.24 (GPA3)
- net IO108: no longer names the net of U407.25 (GPA4)
- net IO109: no longer names the net of U407.26 (GPA5)
- net IO11 renamed IO.PB10
- net IO110: no longer names the net of U407.27 (GPA6)
- net IO111: no longer names the net of U407.28 (GPA7)
- net IO112 renamed IO.Rx
- net IO113 renamed IO.Tx
- net IO114 renamed IO.DSRn
- net IO115 renamed IO.RTSn
- net IO116 renamed IO.DCDn
- net IO117 renamed IO.CTSn
- net IO118 renamed IO.DTRn
- net IO119: no longer names the net of U408.8 (GPB7)
- net IO12 renamed IO.PB9
- net IO120: no longer names the net of U408.21 (GPA0)
- net IO121: no longer names the net of U408.22 (GPA1)
- net IO122: no longer names the net of U408.23 (GPA2)
- net IO123: no longer names the net of U408.24 (GPA3)
- net IO124: no longer names the net of U408.25 (GPA4)
- net IO125: no longer names the net of U408.26 (GPA5)
- net IO126: no longer names the net of U408.27 (GPA6)
- net IO127: no longer names the net of U408.28 (GPA7)
- net IO13 renamed IO.PB8
- net IO14: no longer names the net of U401.27 (GPA6)
- net IO15: no longer names the net of U401.28 (GPA7)
- net IO16 renamed IO.PB7
- net IO17 renamed IO.PB6
- net IO18 renamed IO.PB5
- net IO19 renamed IO.PB4
- net IO2 renamed IO.PB19
- net IO20 renamed IO.PB3
- net IO21 renamed IO.PB2
- net IO22 renamed IO.PB1
- net IO23 renamed IO.PB0
- net IO24 renamed IO.SS0_0
- net IO25 renamed IO.SS0_1
- net IO26 renamed IO.SS0_2
- net IO27 renamed IO.SS0_3
- net IO28 renamed IO.SS0_4
- net IO29 renamed IO.SS0_5
- net IO3 renamed IO.PB18
- net IO30 renamed IO.SS0_6
- net IO31 renamed IO.SS0_7
- net IO32 renamed IO.SS1_0
- net IO33 renamed IO.SS1_1
- net IO34 renamed IO.SS1_2
- net IO35 renamed IO.SS1_3
- net IO36 renamed IO.SS1_4
- net IO37 renamed IO.SS1_5
- net IO38 renamed IO.SS1_6
- net IO39 renamed IO.SS1_7
- net IO4 renamed IO.PB17
- net IO40 renamed IO.SS2_0
- net IO41 renamed IO.SS2_1
- net IO42 renamed IO.SS2_2
- net IO43 renamed IO.SS2_3
- net IO44 renamed IO.SS2_4
- net IO45 renamed IO.SS2_5
- net IO46 renamed IO.SS2_6
- net IO47 renamed IO.SS2_7
- net IO48 renamed IO.SS3_0
- net IO49 renamed IO.SS3_1
- net IO5 renamed IO.PB16
- net IO50 renamed IO.SS3_2
- net IO51 renamed IO.SS3_3
- net IO52 renamed IO.SS3_4
- net IO53 renamed IO.SS3_5
- net IO54 renamed IO.SS3_6
- net IO55 renamed IO.SS3_7
- net IO56 renamed IO.SS4_0
- net IO57 renamed IO.SS4_1
- net IO58 renamed IO.SS4_2
- net IO59 renamed IO.SS4_3
- net IO6 renamed IO.PB15
- net IO60 renamed IO.SS4_4
- net IO61 renamed IO.SS4_5
- net IO62 renamed IO.SS4_6
- net IO63 renamed IO.SS4_7
- net IO64 renamed IO.SS5_0
- net IO65 renamed IO.SS5_1
- net IO66 renamed IO.SS5_2
- net IO67 renamed IO.SS5_3
- net IO68 renamed IO.SS5_4
- net IO69 renamed IO.SS5_5
- net IO7 renamed IO.PB14
- net IO70 renamed IO.SS5_6
- net IO71 renamed IO.SS5_7
- net IO72 renamed IO.SS6_0
- net IO73 renamed IO.SS6_1
- net IO74 renamed IO.SS6_2
- net IO75 renamed IO.SS6_3
- net IO76 renamed IO.SS6_4
- net IO77 renamed IO.SS6_5
- net IO78 renamed IO.SS6_6
- net IO79 renamed IO.SS6_7
- net IO8 renamed IO.PB13
- net IO80 renamed IO.SS7_0
- net IO81 renamed IO.SS7_1
- net IO82 renamed IO.SS7_2
- net IO83 renamed IO.SS7_3
- net IO84 renamed IO.SS7_4
- net IO85 renamed IO.SS7_5
- net IO86 renamed IO.SS7_6
- net IO87 renamed IO.SS7_7
- net IO88 renamed IO.LEFT7
- net IO89 renamed IO.LEFT6
- net IO9 renamed IO.PB12
- net IO90 renamed IO.LEFT5
- net IO91 renamed IO.LEFT4
- net IO92 renamed IO.LEFT3
- net IO93 renamed IO.LEFT2
- net IO94 renamed IO.LEFT1
- net IO95 renamed IO.LEFT0
- net IO96 renamed IO.RIGHT7
- net IO97 renamed IO.RIGHT6
- net IO98 renamed IO.RIGHT5
- net IO99 renamed IO.RIGHT4
- no-connect marks 0 -> 16
Other:
- note added: "GPIO Expander 0 {HWCLK, PB[16..20]}"
- note removed: "GPIO Expander 0"

Commit message: Update 1
Parts:
- removed JP401, JP402, JP403, JP404, JP405, JP406, JP409, JP411, JP417, JP418, JP421, JP423: Jumper_2_Open, Jumper:SolderJumper-2_P1.3mm_Open_TrianglePad1.0x1.5mm, symbol Jumper:Jumper_2_Open
- removed JP407, JP408, JP410, JP412, JP413, JP414, JP415, JP416, JP419, JP420, JP422, JP424: Jumper_2_Bridged, Jumper:SolderJumper-2_P1.3mm_Bridged_Pad1.0x1.5mm, symbol Jumper:Jumper_2_Bridged
- removed R405, R406, R407, R408, R409, R410, R411, R412, R413, R414, R415, R416, R421, R422, R423, R424, R425, R426, R427, R428, R429, R430, R431, R432: 10k, Resistor_SMD:R_0402_1005Metric, symbol Device:R
- U401, U402, U403, U404, U405, U406, U407, U408: value MCP23S17T-E/SS -> MCP23017_SS; symbol Interface_Expansion:MCP23S17_SS -> Interface_Expansion:MCP23017_SS
- renumbered R417 to R405, R418 to R406, R419 to R407, R420 to R408
Connections:
- net +3V3: now also U402.15 (A0), U403.16 (A1), U404.15 (A0), U404.16 (A1), U405.17 (A2), U406.15 (A0), U406.17 (A2), U407.16 (A1), U407.17 (A2), U408.15 (A0), U408.16 (A1), U408.17 (A2)
- net GND: now also U401.15 (A0), U401.16 (A1), U401.17 (A2), U402.16 (A1), U402.17 (A2), U403.15 (A0), U403.17 (A2), U404.17 (A2), U405.15 (A0), U405.16 (A1), U406.16 (A1), U407.15 (A0)
- removed net IO.SDI: U401.14 (SO), U402.14 (SO), U403.14 (SO), U404.14 (SO), U405.14 (SO), U406.14 (SO), U407.14 (SO), U408.14 (SO)
- net IO.SDO renamed IO.SDA
- removed net IO.~{CS}: U401.11 (~{CS}), U402.11 (~{CS}), U403.11 (~{CS}), U404.11 (~{CS}), U405.11 (~{CS}), U406.11 (~{CS}), U407.11 (~{CS}), U408.11 (~{CS})

Commit message: Update
Parts:
- removed RN402, RN403, RN404, RN405, RN406, RN407, RN408: 10k, Resistor_SMD:R_Array_Convex_2x0402, symbol Device:R_Pack02
- added RN? (x7): 10k, Resistor_SMD:R_Array_Convex_2x0402, symbol Device:R_Pack02
- added U?: CD4060BM, Package_SO:SOIC-16_3.9x9.9mm_P1.27mm, symbol ECELab_PartsLibrary:CD4060BM
- added X?: SG-8018CG, Oscillator:Oscillator_SMD_SeikoEpson_SG210-4Pin_2.5x2.0mm, symbol Oscillator:SG-8002CA
Connections:
- net +3V3: now also RN?.3 (R2.2), RN?.3 (R2.2), RN?.3 (R2.2), RN?.3 (R2.2), RN?.3 (R2.2), RN?.3 (R2.2), RN?.3 (R2.2), RN?.4 (R1.2), RN?.4 (R1.2), RN?.4 (R1.2), RN?.4 (R1.2), RN?.4 (R1.2), RN?.4 (R1.2), RN?.4 (R1.2), X?.1 (OE), X?.4 (Vcc)
- net GND: now also X?.2 (GND)
- net IO.BLUE: now also U408.23 (GPA2); no longer U407.23 (GPA2)
- net IO.GREEN: now also U408.22 (GPA1); no longer U407.22 (GPA1)
- net IO.HWCLK: now also U408.8 (GPB7); no longer U401.1 (GPB0)
- net IO.LEFT0: now also U407.1 (GPB0); no longer U406.28 (GPA7)
- net IO.LEFT1: now also U407.2 (GPB1); no longer U406.27 (GPA6)
- net IO.LEFT2: now also U407.3 (GPB2); no longer U406.26 (GPA5)
- net IO.LEFT3: now also U407.4 (GPB3); no longer U406.25 (GPA4)
- net IO.LEFT4: now also U407.5 (GPB4); no longer U406.24 (GPA3)
- net IO.LEFT5: now also U407.6 (GPB5); no longer U406.23 (GPA2)
- net IO.LEFT6: now also U407.7 (GPB6); no longer U406.22 (GPA1)
- net IO.LEFT7: now also U407.8 (GPB7); no longer U406.21 (GPA0)
- net IO.PB0: now also U401.21 (GPA0); no longer U402.8 (GPB7)
- net IO.PB1: now also U401.22 (GPA1); no longer U402.7 (GPB6)
- net IO.PB10: now also U401.3 (GPB2); no longer U401.24 (GPA3)
- net IO.PB11: now also U401.4 (GPB3); no longer U401.23 (GPA2)
- net IO.PB12: now also U401.5 (GPB4); no longer U401.22 (GPA1)
- net IO.PB13: now also U401.6 (GPB5); no longer U401.21 (GPA0)
- net IO.PB14: now also U401.7 (GPB6); no longer U401.8 (GPB7)
- net IO.PB15: now also U401.8 (GPB7); no longer U401.7 (GPB6)
- net IO.PB16: now also U402.21 (GPA0); no longer U401.6 (GPB5)
- net IO.PB17: now also U402.22 (GPA1); no longer U401.5 (GPB4)
- net IO.PB18: now also U402.23 (GPA2); no longer U401.4 (GPB3)
- net IO.PB19: now also U402.24 (GPA3); no longer U401.3 (GPB2)
- net IO.PB2: now also U401.23 (GPA2); no longer U402.6 (GPB5)
- net IO.PB20: now also U402.25 (GPA4), U408.28 (GPA7); no longer U401.2 (GPB1)
- net IO.PB3: now also U401.24 (GPA3); no longer U402.5 (GPB4)
- net IO.PB4: now also U401.25 (GPA4); no longer U402.4 (GPB3)
- net IO.PB5: now also U401.26 (GPA5); no longer U402.3 (GPB2)
- net IO.PB6: now also U401.27 (GPA6); no longer U402.2 (GPB1)
- net IO.PB7: now also U401.28 (GPA7); no longer U402.1 (GPB0)
- net IO.PB8: now also U401.1 (GPB0); no longer U401.26 (GPA5)
- net IO.PB9: now also U401.2 (GPB1); no longer U401.25 (GPA4)
- net IO.RED: now also U408.21 (GPA0); no longer U407.21 (GPA0)
- net IO.RIGHT0: now also U407.21 (GPA0); no longer U407.8 (GPB7)
- net IO.RIGHT1: now also U407.22 (GPA1); no longer U407.7 (GPB6)
- net IO.RIGHT2: now also U407.23 (GPA2); no longer U407.6 (GPB5)
- net IO.RIGHT3: now also U407.24 (GPA3); no longer U407.5 (GPB4)
- net IO.RIGHT4: now also U407.25 (GPA4); no longer U407.4 (GPB3)
- net IO.RIGHT5: now also U407.26 (GPA5); no longer U407.3 (GPB2)
- net IO.RIGHT6: now also U407.27 (GPA6); no longer U407.2 (GPB1)
- net IO.RIGHT7: now also U407.28 (GPA7); no longer U407.1 (GPB0)
- net IO.SS0_0: now also U403.21 (GPA0); no longer U402.21 (GPA0)
- net IO.SS0_1: now also U403.22 (GPA1); no longer U402.22 (GPA1)
- net IO.SS0_2: now also U403.23 (GPA2); no longer U402.23 (GPA2)
- net IO.SS0_3: now also U403.24 (GPA3); no longer U402.24 (GPA3)
- net IO.SS0_4: now also U403.25 (GPA4); no longer U402.25 (GPA4)
- net IO.SS0_5: now also U403.26 (GPA5); no longer U402.26 (GPA5)
- net IO.SS0_6: now also U403.27 (GPA6); no longer U402.27 (GPA6)
- net IO.SS0_7: now also U403.28 (GPA7); no longer U402.28 (GPA7)
- net IO.SS2_0: now also U404.21 (GPA0); no longer U403.21 (GPA0)
- net IO.SS2_1: now also U404.22 (GPA1); no longer U403.22 (GPA1)
- net IO.SS2_2: now also U404.23 (GPA2); no longer U403.23 (GPA2)
- net IO.SS2_3: now also U404.24 (GPA3); no longer U403.24 (GPA3)
- net IO.SS2_4: now also U404.25 (GPA4); no longer U403.25 (GPA4)
- net IO.SS2_5: now also U404.26 (GPA5); no longer U403.26 (GPA5)
- net IO.SS2_6: now also U404.27 (GPA6); no longer U403.27 (GPA6)
- net IO.SS2_7: now also U404.28 (GPA7); no longer U403.28 (GPA7)
- net IO.SS4_0: now also U405.21 (GPA0); no longer U404.21 (GPA0)
- net IO.SS4_1: now also U405.22 (GPA1); no longer U404.22 (GPA1)
- net IO.SS4_2: now also U405.23 (GPA2); no longer U404.23 (GPA2)
- net IO.SS4_3: now also U405.24 (GPA3); no longer U404.24 (GPA3)
- net IO.SS4_4: now also U405.25 (GPA4); no longer U404.25 (GPA4)
- net IO.SS4_5: now also U405.26 (GPA5); no longer U404.26 (GPA5)
- net IO.SS4_6: now also U405.27 (GPA6); no longer U404.27 (GPA6)
- net IO.SS4_7: now also U405.28 (GPA7); no longer U404.28 (GPA7)
- net IO.SS6_0: now also U406.21 (GPA0); no longer U405.21 (GPA0)
- net IO.SS6_1: now also U406.22 (GPA1); no longer U405.22 (GPA1)
- net IO.SS6_2: now also U406.23 (GPA2); no longer U405.23 (GPA2)
- net IO.SS6_3: now also U406.24 (GPA3); no longer U405.24 (GPA3)
- net IO.SS6_4: now also U406.25 (GPA4); no longer U405.25 (GPA4)
- net IO.SS6_5: now also U406.26 (GPA5); no longer U405.26 (GPA5)
- net IO.SS6_6: now also U406.27 (GPA6); no longer U405.27 (GPA6)
- net IO.SS6_7: now also U406.28 (GPA7); no longer U405.28 (GPA7)
- net INTB.MCP6: now reaches U407.19 (INTB)
- net INTB.MCP6: now also RN?.2 (R2.1)
- net INTA.MCP6: now reaches U407.20 (INTA)
- net INTA.MCP6: now also RN?.1 (R1.1)
- net INTB.MCP7: now reaches U408.19 (INTB)
- net INTB.MCP7: now also RN?.2 (R2.1)
- net INTA.MCP7: now reaches U408.20 (INTA)
- net INTA.MCP7: now also RN?.1 (R1.1)
- net INTB.MCP1: now reaches U402.19 (INTB)
- net INTB.MCP1: now also RN?.2 (R2.1)
- net INTA.MCP1: now reaches U402.20 (INTA)
- net INTA.MCP1: now also RN?.1 (R1.1)
- net INTB.MCP4: now reaches U405.19 (INTB)
- net INTB.MCP4: now also RN?.2 (R2.1)
- net INTA.MCP4: now reaches U405.20 (INTA)
- net INTA.MCP4: now also RN?.1 (R1.1)
- net INTA.MCP2: now reaches U403.20 (INTA)
- net INTA.MCP2: now also RN?.1 (R1.1)
- net INTB.MCP2: now reaches U403.19 (INTB)
- net INTB.MCP2: now also RN?.2 (R2.1)
- net INTA.MCP0: now reaches RN401.1 (R1.1), U401.20 (INTA)
- net INTB.MCP0: now reaches RN401.2 (R2.1), U401.19 (INTB)
- net INTA.MCP5: now reaches U406.20 (INTA)
- net INTA.MCP5: now also RN?.1 (R1.1)
- net INTB.MCP5: now reaches U406.19 (INTB)
- net INTB.MCP5: now also RN?.2 (R2.1)
- net INTA.MCP3: now reaches U404.20 (INTA)
- net INTA.MCP3: now also RN?.1 (R1.1)
- net INTB.MCP3: now reaches U404.19 (INTB)
- net INTB.MCP3: now also RN?.2 (R2.1)
- net IO.SCK renamed IO.SCK1
- net IO.SCK1: no longer U401.12 (SCK), U402.12 (SCK)
- net IO.SDA renamed IO.SDA1
- net IO.SDA1: no longer U401.13 (SDA), U402.13 (SDA)
- new net IO.SCK0: U401.12 (SCK), U402.12 (SCK)
- new net IO.SDA0: U401.13 (SDA), U402.13 (SDA)
- no-connect marks 16 -> 15
Other:
- moved on the sheet: RN401

Commit message: Update 2nd iteration
Parts:
- removed U?: CD4060BM, Package_SO:SOIC-16_3.9x9.9mm_P1.27mm, symbol ECELab_PartsLibrary:CD4060BM
- removed X?: SG-8018CG, Oscillator:Oscillator_SMD_SeikoEpson_SG210-4Pin_2.5x2.0mm, symbol Oscillator:SG-8002CA
- added C409: 0.1u, Capacitor_SMD:C_0402_1005Metric, symbol Device:C
- added C410: 10n, Capacitor_SMD:C_0402_1005Metric, symbol Device:C
- added J401: Conn_01x02_Male, Connector_PinHeader_2.54mm:PinHeader_1x02_P2.54mm_Vertical, symbol Connector:Conn_01x02_Male
- added R409: 8.2k, Resistor_SMD:R_0402_1005Metric, symbol Device:R
- added R410: 68k, Resistor_SMD:R_0402_1005Metric, symbol Device:R
- added U409: BL1551B, Package_TO_SOT_SMD:SOT-363_SC-70-6, symbol Analog_Switch:TS5A3159ADCKR
- added U410: NE555DR, Package_SO:SOIC-8_3.9x4.9mm_P1.27mm, symbol Timer:NE555D
- U401, U402, U403, U404, U405, U406, U407, U408: value MCP23017_SS -> MCP23017T-E/SS; LCSC C128577 -> C558584
- gave numbers to parts that had none: 7
Connections:
- net +3V3: now also U409.3, U409.5 (V+); no longer C405.2, U406.9 (VDD)
- net GND: now also C409.2, C410.2, U409.1, U409.2 (GND), U410.1 (GND)
- net IO.PB20: now also J401.2 (Pin_2)
- net INTB.MCP1: no longer names the net of RN402.2 (R2.1), U402.19 (INTB)
- new net: C409.1, R410.2, U410.2 (TRIG), U410.6 (THR)
- new net: C410.1, U410.5 (CONT)
- new net: R409.2, R410.1, U410.7 (DIS)
- new net +5V: R409.1, U410.4 (RST), U410.8 (VCC)
- new net CLK100: J401.1 (Pin_1), U410.3 (OUT)
- new net MCP5.PWR: C405.2, U406.9 (VDD), U409.4
- new net MCP5.SEL: U409.6
Other:
- note added: "100Hz Clock"
- note added: "GPIO Expander 0"
- note removed: "GPIO Expander 0 {HWCLK, PB[16..20]}"

Commit message: Update 7/30
Parts:
- added U410: BL1551B, Package_TO_SOT_SMD:SOT-363_SC-70-6, symbol Analog_Switch:TS5A3159ADCKR
- renumbered U410 to U411
Connections:
- net +3V3: now also U410.3, U410.5 (V+); no longer C406.2, U407.9 (VDD)
- net GND: now also U410.1, U410.2 (GND)
- new net MCP6.PWR: C406.2, U407.9 (VDD), U410.4
- new net MCP6.SEL: U410.6

Commit message: Complete Design v2
Parts:
- J401: LCSC (none) -> C5116481; LCSC Part Number (none) -> C5116481
Changed lines of the file:
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@@
+      (effects (font (size 1.27 1.27)) hide)
+    )
+    (property "LCSC" "C5116481" (id 4) (at 105.41 238.125 0)
+      (effects (font (size 1.27 1.27)) hide)
+    )
+    (property "LCSC Part Number" "C5116481" (id 5) (at 105.41 238.125 0)
       (effects (font (size 1.27 1.27)) hide)
     )
