File: GPIO.kicad_sch (KiCad schematic)
At the start: 72 parts, among them U401 MCP23017_SS, U402 MCP23017_SS, U403 MCP23017_SS, U404 MCP23017_SS, U405 MCP23017_SS, U406 MCP23017_SS, U407 MCP23017_SS, U408 MCP23017_SS

Commit message: Complete Draft 1 of PCB Design
Parts:
- added C401, C402, C403, C404, C405, C406, C407, C408: 0.1u, Capacitor_SMD:C_0402_1005Metric, symbol Device:C
Connections:
- net +3V3: now also C401.2, C402.2, C403.2, C404.2, C405.2, C406.2, C407.2, C408.2
- net GND: now also C401.1, C402.1, C403.1, C404.1, C405.1, C406.1, C407.1, C408.1
- net IO0 renamed IO.HWCLK
- net IO1 renamed IO.PB20
- net IO10 renamed IO.PB11
- net IO100 renamed IO.RIGHT3
- net IO101 renamed IO.RIGHT2
- net IO102 renamed IO.RIGHT1
- net IO103 renamed IO.RIGHT0
- net IO104 renamed IO.RED
- net IO105 renamed IO.GREEN
- net IO106 renamed IO.BLUE
- net IO107: no longer names the net of U407.24 (GPA3)
- net IO108: no longer names the net of U407.25 (GPA4)
- net IO109: no longer names the net of U407.26 (GPA5)
- net IO11 renamed IO.PB10
- net IO110: no longer names the net of U407.27 (GPA6)
- net IO111: no longer names the net of U407.28 (GPA7)
- net IO112 renamed IO.Rx
- net IO113 renamed IO.Tx
- net IO114 renamed IO.DSRn
- net IO115 renamed IO.RTSn
- net IO116 renamed IO.DCDn
- net IO117 renamed IO.CTSn
- net IO118 renamed IO.DTRn
- net IO119: no longer names the net of U408.8 (GPB7)
- net IO12 renamed IO.PB9
- net IO120: no longer names the net of U408.21 (GPA0)
- net IO121: no longer names the net of U408.22 (GPA1)
- net IO122: no longer names the net of U408.23 (GPA2)
- net IO123: no longer names the net of U408.24 (GPA3)
- net IO124: no longer names the net of U408.25 (GPA4)
- net IO125: no longer names the net of U408.26 (GPA5)
- net IO126: no longer names the net of U408.27 (GPA6)
- net IO127: no longer names the net of U408.28 (GPA7)
- net IO13 renamed IO.PB8
- net IO14: no longer names the net of U401.27 (GPA6)
- net IO15: no longer names the net of U401.28 (GPA7)
- net IO16 renamed IO.PB7
- net IO17 renamed IO.PB6
- net IO18 renamed IO.PB5
- net IO19 renamed IO.PB4
- net IO2 renamed IO.PB19
- net IO20 renamed IO.PB3
- net IO21 renamed IO.PB2
- net IO22 renamed IO.PB1
- net IO23 renamed IO.PB0
- net IO24 renamed IO.SS0_0
- net IO25 renamed IO.SS0_1
- net IO26 renamed IO.SS0_2
- net IO27 renamed IO.SS0_3
- net IO28 renamed IO.SS0_4
- net IO29 renamed IO.SS0_5
- net IO3 renamed IO.PB18
- net IO30 renamed IO.SS0_6
- net IO31 renamed IO.SS0_7
- net IO32 renamed IO.SS1_0
- net IO33 renamed IO.SS1_1
- net IO34 renamed IO.SS1_2
- net IO35 renamed IO.SS1_3
- net IO36 renamed IO.SS1_4
- net IO37 renamed IO.SS1_5
- net IO38 renamed IO.SS1_6
- net IO39 renamed IO.SS1_7
- net IO4 renamed IO.PB17
- net IO40 renamed IO.SS2_0
- net IO41 renamed IO.SS2_1
- net IO42 renamed IO.SS2_2
- net IO43 renamed IO.SS2_3
- net IO44 renamed IO.SS2_4
- net IO45 renamed IO.SS2_5
- net IO46 renamed IO.SS2_6
- net IO47 renamed IO.SS2_7
- net IO48 renamed IO.SS3_0
- net IO49 renamed IO.SS3_1
- net IO5 renamed IO.PB16
- net IO50 renamed IO.SS3_2
- net IO51 renamed IO.SS3_3
- net IO52 renamed IO.SS3_4
- net IO53 renamed IO.SS3_5
- net IO54 renamed IO.SS3_6
- net IO55 renamed IO.SS3_7
- net IO56 renamed IO.SS4_0
- net IO57 renamed IO.SS4_1
- net IO58 renamed IO.SS4_2
- net IO59 renamed IO.SS4_3
- net IO6 renamed IO.PB15
- net IO60 renamed IO.SS4_4
- net IO61 renamed IO.SS4_5
- net IO62 renamed IO.SS4_6
- net IO63 renamed IO.SS4_7
- net IO64 renamed IO.SS5_0
- net IO65 renamed IO.SS5_1
- net IO66 renamed IO.SS5_2
- net IO67 renamed IO.SS5_3
- net IO68 renamed IO.SS5_4
- net IO69 renamed IO.SS5_5
- net IO7 renamed IO.PB14
- net IO70 renamed IO.SS5_6
- net IO71 renamed IO.SS5_7
- net IO72 renamed IO.SS6_0
- net IO73 renamed IO.SS6_1
- net IO74 renamed IO.SS6_2
- net IO75 renamed IO.SS6_3
- net IO76 renamed IO.SS6_4
- net IO77 renamed IO.SS6_5
- net IO78 renamed IO.SS6_6
- net IO79 renamed IO.SS6_7
- net IO8 renamed IO.PB13
- net IO80 renamed IO.SS7_0
- net IO81 renamed IO.SS7_1
- net IO82 renamed IO.SS7_2
- net IO83 renamed IO.SS7_3
- net IO84 renamed IO.SS7_4
- net IO85 renamed IO.SS7_5
- net IO86 renamed IO.SS7_6
- net IO87 renamed IO.SS7_7
- net IO88 renamed IO.LEFT7
- net IO89 renamed IO.LEFT6
- net IO9 renamed IO.PB12
- net IO90 renamed IO.LEFT5
- net IO91 renamed IO.LEFT4
- net IO92 renamed IO.LEFT3
- net IO93 renamed IO.LEFT2
- net IO94 renamed IO.LEFT1
- net IO95 renamed IO.LEFT0
- net IO96 renamed IO.RIGHT7
- net IO97 renamed IO.RIGHT6
- net IO98 renamed IO.RIGHT5
- net IO99 renamed IO.RIGHT4
- no-connect marks 0 -> 16
Other:
- note added: "GPIO Expander 0 {HWCLK, PB[16..20]}"
- note removed: "GPIO Expander 0"

Commit message: Draft 1 complete
Parts:
- C401, C402, C403, C404, C405, C406, C407, C408: LCSC (none) -> C1525; LCSC Part Number (none) -> C1525
- R401, R402, R403, R404, R405, R406, R407, R408, R409, R410, R411, R412, R413, R414, R415, R416, R417, R418, R419, R420, R421, R422, R423, R424, R425, R426, R427, R428, R429, R430, R431, R432: LCSC (none) -> C140214; LCSC Part Number (none) -> C140214
- RN401, RN402, RN403, RN404, RN405, RN406, RN407, RN408: LCSC (none) -> C695179; LCSC Part Number (none) -> C695179
- U401, U402, U403, U404, U405, U406, U407, U408: LCSC (none) -> C558584; LCSC Part Number (none) -> C558584

Commit message: Update to v1.2
Parts:
- removed JP401, JP402, JP403, JP404, JP405, JP406, JP409, JP411, JP417, JP418, JP421, JP423: Jumper_2_Open, Jumper:SolderJumper-2_P1.3mm_Open_TrianglePad1.0x1.5mm, symbol Jumper:Jumper_2_Open
- removed JP407, JP408, JP410, JP412, JP413, JP414, JP415, JP416, JP419, JP420, JP422, JP424: Jumper_2_Bridged, Jumper:SolderJumper-2_P1.3mm_Bridged_Pad1.0x1.5mm, symbol Jumper:Jumper_2_Bridged
- removed R405, R406, R407, R408, R409, R410, R411, R412, R413, R414, R415, R416, R421, R422, R423, R424, R425, R426, R427, R428, R429, R430, R431, R432: 10k, Resistor_SMD:R_0402_1005Metric, symbol Device:R
Connections:
- net +3V3: now also U402.15 (A0), U403.16 (A1), U404.15 (A0), U404.16 (A1), U405.17 (A2), U406.15 (A0), U406.17 (A2), U407.16 (A1), U407.17 (A2), U408.15 (A0), U408.16 (A1), U408.17 (A2)
- net GND: now also U401.15 (A0), U401.16 (A1), U401.17 (A2), U402.16 (A1), U402.17 (A2), U403.15 (A0), U403.17 (A2), U404.17 (A2), U405.15 (A0), U405.16 (A1), U406.16 (A1), U407.15 (A0)

Commit message: Complete Design
Parts:
- added C401, C402, C403, C404, C405, C406, C407, C414, C416, C417, C418, C425, C426: 0.1u, Capacitor_SMD:C_0402_1005Metric, symbol Device:C
- added C412: 3.3u, Capacitor_SMD:C_0402_1005Metric, symbol Device:C
- added C413, C415: 4.7u, Capacitor_SMD:C_0402_1005Metric, symbol Device:C
- added C423, C424: 27p, Capacitor_SMD:C_0402_1005Metric, symbol Device:C
- added C427: 10n, Capacitor_SMD:C_0402_1005Metric, symbol Device:C
- added D401: PMEG40, Diode_SMD:D_SOD-323, symbol Device:D_Schottky
- added FB401, FB402: 600R, Inductor_SMD:L_0603_1608Metric, symbol Device:FerriteBead
- added FB403: 120R, Inductor_SMD:L_0603_1608Metric, symbol Device:FerriteBead
- added J401: USB_C_Receptacle_USB2.0, Connector_USB:USB_C_Receptacle_HRO_TYPE-C-31-M-12, symbol Connector:USB_C_Receptacle_USB2.0
- added J402: Conn_01x02_Male, Connector_PinHeader_2.54mm:PinHeader_1x02_P2.54mm_Vertical, symbol Connector:Conn_01x02_Male
- added R405, R406: 12k, Resistor_SMD:R_0402_1005Metric, symbol Device:R
- added R411, R412, R413: 10k, Resistor_SMD:R_0402_1005Metric, symbol Device:R
- added R414, R415: 5.1k, Resistor_SMD:R_0402_1005Metric, symbol Device:R
- added R416: 2.2k, Resistor_SMD:R_0402_1005Metric, symbol Device:R
- added R417: 8.2k, Resistor_SMD:R_0402_1005Metric, symbol Device:R
- added R418: 68k, Resistor_SMD:R_0402_1005Metric, symbol Device:R
- added U410: 93LC56BT-I/OT, Package_TO_SOT_SMD:SOT-23-6, symbol Memory_EEPROM:93LCxxBxxOT
- added U411: NE555DR, Package_SO:SOIC-8_3.9x4.9mm_P1.27mm, symbol Timer:NE555D
- added U415: FT4232HL-REEL, Package_QFP:LQFP-64_10x10mm_P0.5mm, symbol Interface_USB:FT4232H
- added Y401: 12MHz, Crystal:Crystal_SMD_HC49-SD, symbol Device:Crystal
- renumbered C401 to C408, C402 to C409, C403 to C410, C404 to C411, C405 to C419, C406 to C420, C407 to C421, C408 to C422, R417 to R407, R418 to R408, R419 to R409, R420 to R410, U405 to U406, U406 to U407, U407 to U408, U408 to U409
Connections:
- net +3V3: now also C401.1, C402.1, C403.1, C404.1, C425.1, FB401.1, FB402.1, R406.2, R411.1, R412.1, R413.1, U410.6 (VCC), U415.20 (VCCIO), U415.31 (VCCIO), U415.42 (VCCIO), U415.50 (VREGIN), U415.56 (VCCIO)
- net GND: now also C401.2, C402.2, C403.2, C404.2, C405.2, C406.2, C407.2, C412.2, C413.2, C414.2, C415.2, C416.2, C417.2, C418.2, C423.1, C424.1, C425.2, C426.2, C427.2, J401.A1 (GND), J401.A12 (GND), J401.B1 (GND), J401.B12 (GND), J401.S1 (SHIELD), R405.2, R414.2, R415.1, U410.2 (GND), U411.1 (GND), U415.1 (GND), U415.10 (AGND), U415.11 (GND), U415.13 (TEST), U415.15 (GND), U415.25 (GND), U415.35 (GND), U415.47 (GND), U415.5 (GND), U415.51 (GND)
- net IO.LEFT0: now also U415.38 (CDBUS0)
- net IO.LEFT1: now also U415.39 (CDBUS1)
- net IO.LEFT2: now also U415.40 (CDBUS2)
- net IO.LEFT3: now also U415.41 (CDBUS3)
- net IO.LEFT4: now also U415.43 (CDBUS4)
- net IO.LEFT5: now also U415.44 (CDBUS5)
- net IO.LEFT6: now also U415.45 (CDBUS6)
- net IO.LEFT7: now also U415.46 (CDBUS7)
- net IO.PB20: now also J402.2 (Pin_2)
- net IO.RIGHT0: now also U415.48 (DDBUS0)
- net IO.RIGHT1: now also U415.52 (DDBUS1)
- net IO.RIGHT2: now also U415.53 (DDBUS2)
- net IO.RIGHT3: now also U415.54 (DDBUS3)
- net IO.RIGHT4: now also U415.55 (DDBUS4)
- net IO.RIGHT5: now also U415.57 (DDBUS5)
- net IO.RIGHT6: now also U415.58 (DDBUS6)
- net IO.RIGHT7: now also U415.59 (DDBUS7)
- net IO.SS6_0: now also U415.26 (BDBUS0)
- net IO.SS6_1: now also U415.27 (BDBUS1)
- net IO.SS6_2: now also U415.28 (BDBUS2)
- net IO.SS6_3: now also U415.29 (BDBUS3)
- net IO.SS6_4: now also U415.30 (BDBUS4)
- net IO.SS6_5: now also U415.32 (BDBUS5)
- net IO.SS6_6: now also U415.33 (BDBUS6)
- net IO.SS6_7: now also U415.34 (BDBUS7)
- net IO.SS7_0: now also U415.16 (ADBUS0)
- net IO.SS7_1: now also U415.17 (ADBUS1)
- net IO.SS7_2: now also U415.18 (ADBUS2)
- net IO.SS7_3: now also U415.19 (ADBUS3)
- net IO.SS7_4: now also U415.21 (ADBUS4)
- net IO.SS7_5: now also U415.22 (ADBUS5)
- net IO.SS7_6: now also U415.23 (ADBUS6)
- net IO.SS7_7: now also U415.24 (ADBUS7)
- new net: J401.A5 (CC1), R414.1
- new net: J401.B5 (CC2), R415.2
- new net: D401.1 (K), FB403.1
- new net: R406.1, U415.14 (~{RESET})
- new net: R405.1, U415.6 (REF)
- new net: R411.2, R416.1, U410.1 (DO)
- new net: R417.2, R418.1, U411.7 (DIS)
- new net: C426.1, R418.2, U411.2 (TRIG), U411.6 (THR)
- new net: C427.1, U411.5 (CONT)
- new net +1V8: C405.1, C406.1, C407.1, C412.1, U415.12 (VCORE), U415.37 (VCORE), U415.49 (VREGOUT), U415.64 (VCORE)
- new net +5V: C418.1, FB403.2, R417.1, U411.4 (RST), U411.8 (VCC)
- new net CLK100: J402.1 (Pin_1), U411.3 (OUT)
- new net EECLK2: R412.2, U410.4 (CLK), U415.62 (EECLK)
- new net EECS2: R413.2, U410.5 (CS), U415.63 (EECS)
- new net EEDATA2: R416.2, U410.3 (DI), U415.61 (EEDATA)
- new net FTDI2.D+: J401.A6 (D+), J401.B6 (D+), U415.8 (DP)
- new net FTDI2.D-: J401.A7 (D-), J401.B7 (D-), U415.7 (DM)
- new net PWRU_IN2: C417.1, D401.2 (A), J401.A4 (VBUS), J401.A9 (VBUS), J401.B4 (VBUS), J401.B9 (VBUS)
- new net VPHY2: C413.1, C414.1, FB401.2, U415.4 (VPHY)
- new net VPLL2: C415.1, C416.1, FB402.2, U415.9 (VPLL)
- new net XCSI: C423.2, U415.2 (OSCI), Y401.1
- new net XCSO: C424.2, U415.3 (OSCO), Y401.2
- no-connect marks 16 -> 20
Other:
- note added: "100Hz Clock"
- note added: "Decoupling Capacitors"
- note added: "FT232H EEPROM"
- note added: "FT232H Filtering & Decoupling"
- note added: "FTDI FT232H"
- note added: "USB_C"

Commit message: Complete V1.3
Parts:
- U411: value NE555DR -> LMC555CMX/NOPB; LCSC C7593 -> C90760; LCSC Part Number C7593 -> C90760
Connections:
- net +3V3: now also R417.1, U411.4 (RST), U411.8 (VCC)
- net +5V: no longer R417.1, U411.4 (RST), U411.8 (VCC)
Changed lines of the file:
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@@
+    (pin "1")
+  )
+  (symbol (lib_id "power:+3V3") (at 494.03 250.19 0) (unit 1)
+    (in_bom yes) (on_board yes) (fields_autoplaced)
+    (property "Reference" "#PWR?" (id 0) (at 494.03 254 0)
+      (effects (font (size 1.27 1.27)) hide)
+    )
+    (property "Value" "+3V3" (id 1) (at 494.03 245.11 0))
+    (property "Footprint" "" (id 2) (at 494.03 250.19 0)
+      (effects (font (size 1.27 1.27)) hide)
+    )
+    (property "Datasheet" "" (id 3) (at 494.03 250.19 0)
+      (effects (font (size 1.27 1.27)) hide)
+    )
     (pin "1")
   )
@@
       (effects (font (size 1.27 1.27)) (justify left))
     )
-    (property "Value" "NE555DR" (id 1) (at 496.0494 261.62 0)
+    (property "Value" "LMC555CMX/NOPB" (id 1) (at 496.0494 261.62 0)
       (effects (font (size 1.27 1.27)) (justify left))
     )
@@
       (effects (font (size 1.27 1.27)) hide)
     )
-    (property "LCSC" "C7593" (id 4) (at 494.03 271.78 0)
-      (effects (font (size 1.27 1.27)) hide)
-    )
-    (property "LCSC Part Number" "C7593" (id 5) (at 494.03 271.78 0)
+    (property "LCSC" "C90760" (id 4) (at 494.03 271.78 0)
+      (effects (font (size 1.27 1.27)) hide)
+    )
+    (property "LCSC Part Number" "C90760" (id 5) (at 494.03 271.78 0)
       (effects (font (size 1.27 1.27)) hide)
     )
@@
       (effects (font (size 1.27 1.27)) hide)
     )
-    (pin "1")
-  )
-  (symbol (lib_id "power:+5V") (at 494.03 250.19 0) (unit 1)
-    (in_bom yes) (on_board yes) (fields_autoplaced)
-    (property "Reference" "#PWR0480" (id 0) (at 494.03 254 0)
-      (effects (font (size 1.27 1.27)) hide)
-    )
-    (property "Value" "+5V" (id 1) (at 494.03 244.475 0))
-    (property "Footprint" "" (id 2) (at 494.03 250.19 0)
-      (effects (font (size 1.27 1.27)) hide)
-    )
-    (property "Datasheet" "" (id 3) (at 494.03 250.19 0)
-      (effects (font (size 1.27 1.27)) hide)
-    )
