File: FTDI.kicad_sch (KiCad schematic)
At the start: 22 parts

Commit message: Update
Parts:
- C301, C302, C303, C304, C305, C308, C309: renamed from C?; footprint (none) -> Capacitor_SMD:C_0402_1005Metric
- J301: renamed from J?; footprint (none) -> Connector_PinHeader_2.54mm:PinHeader_1x04_P2.54mm_Vertical
- J302: renamed from J?; footprint (none) -> Connector_PinHeader_2.54mm:PinHeader_1x03_P2.54mm_Vertical
- R301, R302, R303, R304: renamed from R?; footprint (none) -> Resistor_SMD:R_0402_1005Metric
- SW301: renamed from SW?; footprint (none) -> Button_Switch_SMD:SW_SPDT_PCM12
- U301: renamed from U?; footprint (none) -> Package_SO:SOIC-16W_5.3x10.2mm_P1.27mm
- U302: renamed from U?; value FT232H -> FT232HL; footprint (none) -> Package_QFP:LQFP-48_7x7mm_P0.5mm
- Y301: renamed from Y?; footprint (none) -> Crystal:Crystal_SMD_HC49-SD
- gave numbers to parts that had none: 5
Connections:
- net +3.3V is gone; now on net +3V3: FB301.1, FB302.1
- net ACBUS0: no longer names the net of U302.21 (ACBUS0)
- net ACBUS1: no longer names the net of U302.25 (ACBUS1)
- net ACBUS2: no longer names the net of U302.26 (ACBUS2)
- net ACBUS3: no longer names the net of U302.27 (ACBUS3)
- net ACBUS4: no longer names the net of U302.28 (ACBUS4)
- net ACBUS5: no longer names the net of U302.29 (ACBUS5)
- net ACBUS6: no longer names the net of U302.30 (ACBUS6)
- net ACBUS7: no longer names the net of U302.31 (ACBUS7)
- net ACBUS8: no longer names the net of U302.32 (ACBUS8)
- net ACBUS9: no longer names the net of U302.33 (ACBUS9)
- net ADBUS4: no longer names the net of U302.17 (ADBUS4)
- net ADBUS5: no longer names the net of U302.18 (ADBUS5)
- net ADBUS6: no longer names the net of U302.19 (ADBUS6)
- net ADBUS7: no longer names the net of U302.20 (ADBUS7)
- no-connect marks 0 -> 14

Commit message: Complete SPI Design
Parts:
- removed R303: 10K, Resistor_SMD:R_0402_1005Metric, symbol Device:R
- removed SW301: SW_SPDT, Button_Switch_SMD:SW_SPDT_PCM12, symbol Switch:SW_SPDT
- removed U301: SN74LVC257AD, Package_SO:SOIC-16W_5.3x10.2mm_P1.27mm, symbol 74xx:74LS157
- added C308: 0.1u, Capacitor_SMD:C_0402_1005Metric, symbol Device:C
- added J303: Conn_01x04_Male, Connector_PinHeader_2.54mm:PinHeader_1x04_P2.54mm_Horizontal, symbol Connector:Conn_01x04_Male
- added U302: SN74LVC157ADR, Package_SO:SOIC-16_3.9x9.9mm_P1.27mm, symbol 74xx:74LS157
- C301, C302, C303, C304, C305: LCSC (none) -> C1525; LCSC Part Number (none) -> C1525
- C306, C307: LCSC (none) -> C76991; LCSC Part Number (none) -> C76991
- C309: renamed from C308; LCSC (none) -> C1557; LCSC Part Number (none) -> C1557
- C310: renamed from C309; LCSC (none) -> C1557; LCSC Part Number (none) -> C1557
- FB301, FB302: LCSC (none) -> C1002; LCSC Part Number (none) -> C1002
- J301: footprint Connector_PinHeader_2.54mm:PinHeader_1x04_P2.54mm_Vertical -> Connector_PinHeader_2.54mm:PinHeader_1x04_P2.54mm_Horizontal; LCSC (none) -> C91552; LCSC Part Number (none) -> C91552
- J302: LCSC (none) -> C49257; LCSC Part Number (none) -> C49257
- R301, R302: LCSC (none) -> C25752; LCSC Part Number (none) -> C25752
- R303: renamed from R304; LCSC (none) -> C25879; LCSC Part Number (none) -> C25879
- U301: renamed from U302; value FT232HL -> FT232HQ-REEL; footprint Package_QFP:LQFP-48_7x7mm_P0.5mm -> Package_DFN_QFN:QFN-48-1EP_8x8mm_P0.5mm_EP6.2x6.2mm; LCSC (none) -> C82158; LCSC Part Number (none) -> C82158
- U303: LCSC (none) -> C190271; LCSC Part Number (none) -> C190271
- Y301: LCSC (none) -> C14871; LCSC Part Number (none) -> C14871
Connections:
- net +3V3: now also C308.2, U302.16 (VCC)
- net CONN.SCK: now also U302.3 (1B)
- net CONN.SDI: now also J301.3 (Pin_3), U302.10 (3B); no longer J301.2 (Pin_2)
- net CONN.SDO: now also J301.2 (Pin_2), U302.6 (2B); no longer J301.3 (Pin_3)
- net CONN.~{CS}: now also U302.13 (4B)
- net FTDI.SCK: now also U302.2 (1A)
- net FTDI.SDI: now also U301.15 (ADBUS2), U302.11 (3A); no longer U301.14 (ADBUS1)
- net FTDI.SDO: now also U301.14 (ADBUS1), U302.5 (2A); no longer U301.15 (ADBUS2)
- net FTDI.~{CS}: now also U302.14 (4A)
- net GND: now also U301.49 (GND), C308.1, U302.15 (~{G}), U302.8 (GND)
- net IO.SCK: now also J303.1 (Pin_1), U302.4 (1Y)
- net IO.SDI: now also J303.3 (Pin_3), U302.9 (3Y)
- net IO.SDO: now also J303.2 (Pin_2), U302.7 (2Y)
- net IO.~{CS}: now also J303.4 (Pin_4), U302.12 (4Y)
- net MUX.SEL renamed SEL
- net SEL: now also U302.1 (~{A}/B)
Other:
- note added: "I2C: SCL = Clock SDA = Serial Data (Both master and slave) Pull up res = 10k"
- note added: "Jumper Headers for selecting FTDI or Header"
- note removed: "Default = FTDI"
- note removed: "MUX for selecting FTDI or Header (Default=FTDI)"
- note removed: "Propagation Delay = 4.6ns"
- note removed: "SDI = MOSI (Master Out - Slave In) SDO = MISO (Master In - Slave Out) ~{CS} = Active Low SCK = SPI Clock (Output of FTDI)"
- note removed: "SEL = L, Output = A SEL = H, Output = B"

Commit message: Update 1
Parts:
- removed J303: Conn_01x04_Male, Connector_PinHeader_2.54mm:PinHeader_1x04_P2.54mm_Horizontal, symbol Connector:Conn_01x04_Male
- added R301, R302: 10k, Resistor_SMD:R_0402_1005Metric, symbol Device:R
- renumbered R301 to R303, R302 to R304, R303 to R305
Connections:
- net +3V3: now also R301.1, R302.1
- net FTDI.SCK: now also R302.2
- net FTDI.SDI: no longer U301.15 (ADBUS2)
- net FTDI.SDO: no longer U301.14 (ADBUS1)
- net FTDI.~{CS}: no longer U301.16 (ADBUS3)
- new net FTDI.SDA: R301.2, U301.14 (ADBUS1)
