File: ECELab_v1.kicad_pcb (KiCad board)
At the start: 4 copper layers, 82.4 x 76.2 mm, 90 parts, among them J201 USB_C_Receptacle_USB2.0, J202 Conn_01x02_Male, J301 Conn_01x04_Male, J302 Conn_01x03_Male, U201 AZ1117IH-3.3TRG1, U301 FT232HQ-REEL, U302 SN74LVC157ADR, U303 93LC56BT-I/OT, U401 MCP23017_SS, U402 MCP23017_SS, U403 MCP23017_SS, U404 MCP23017_SS, U405 MCP23017_SS, U406 MCP23017_SS, U407 MCP23017_SS, U408 MCP23017_SS, U501 ICE40-HX8K_Breakout_Board, U601 RASPBERRY_PI_4B_4GB, Y301 12MHz

Commit message: Update 2nd iteration
Parts:
- removed C207, C208, C209, C210: 0.1u, Capacitor_SMD:C_0402_1005Metric
- removed D205, D206, D207, D208: PMEG40, Diode_SMD:D_SOD-323
- removed FB203, FB204: 120R, Inductor_SMD:L_0603_1608Metric
- removed U303: 93LC56BT-I/OT, Package_TO_SOT_SMD:SOT-23-6
- added C311: 4.7u, Capacitor_SMD:C_0402_1005Metric, F.Cu at (129.3, 133.0)
- added C312: 0.1u, Capacitor_SMD:C_0402_1005Metric, F.Cu at (111.8, 151.7)
- added C313: 27p, Capacitor_SMD:C_0402_1005Metric, F.Cu at (111.8, 153.7)
- added C314: 27p, Capacitor_SMD:C_0402_1005Metric, F.Cu at (132.1, 133.0)
- added C315: 0.1u, Capacitor_SMD:C_0402_1005Metric, F.Cu at (116.8, 147.2)
- added C409: 0.1u, Capacitor_SMD:C_0402_1005Metric, F.Cu at (154.7, 135.9)
- added C410: 10n, Capacitor_SMD:C_0402_1005Metric, F.Cu at (150.7, 140.9)
- added C701: 0.1u, Capacitor_SMD:C_0402_1005Metric, F.Cu at (189.1, 195.2)
- added C702: 0.1u, Capacitor_SMD:C_0402_1005Metric, F.Cu at (175.5, 207.4)
- added C703: 0.1u, Capacitor_SMD:C_0402_1005Metric, F.Cu at (197.8, 184.8)
- added C704: 0.1u, Capacitor_SMD:C_0402_1005Metric, F.Cu at (178.3, 206.4)
- added C705: 0.1u, Capacitor_SMD:C_0402_1005Metric, F.Cu at (175.5, 205.5)
- added C706: 0.1u, Capacitor_SMD:C_0402_1005Metric, F.Cu at (196.6, 186.8)
- added C707: 0.1u, Capacitor_SMD:C_0402_1005Metric, F.Cu at (172.6, 207.4)
- added C708: 3.3u, Capacitor_SMD:C_0402_1005Metric, F.Cu at (172.6, 209.4)
- added C709: 4.7u, Capacitor_SMD:C_0402_1005Metric, F.Cu at (193.8, 187.3)
- added C710: 0.1u, Capacitor_SMD:C_0402_1005Metric, F.Cu at (190.8, 193.2)
- added C711: 4.7u, Capacitor_SMD:C_0402_1005Metric, F.Cu at (178.9, 204.4)
- added C712: 0.1u, Capacitor_SMD:C_0402_1005Metric, F.Cu at (186.2, 197.2)
- added C713: 27p, Capacitor_SMD:C_0402_1005Metric, F.Cu at (193.7, 189.3)
- added C714: 27p, Capacitor_SMD:C_0402_1005Metric, F.Cu at (193.7, 191.2)
- added C715: 0.1u, Capacitor_SMD:C_0402_1005Metric, F.Cu at (181.9, 202.4)
- added C716: 0.1u, Capacitor_SMD:C_0402_1005Metric, F.Cu at (190.8, 189.3)
- added C717: 0.1u, Capacitor_SMD:C_0402_1005Metric, F.Cu at (190.8, 191.2)
- added D701: D5V0L1B2S9-7, Diode_SMD:D_SOD-923, F.Cu at (175.4, 209.4)
- added FB701: 600R, Inductor_SMD:L_0603_1608Metric, F.Cu at (155.8, 207.4)
- added FB702: 600R, Inductor_SMD:L_0603_1608Metric, F.Cu at (159.8, 207.4)
- added FB703: 120R, Inductor_SMD:L_0603_1608Metric, F.Cu at (191.4, 185.0)
- added J401: Conn_01x02_Male, Connector_PinHeader_2.54mm:PinHeader_1x02_P2.54mm_Vertical, F.Cu at (147.9, 134.3)
- added J701: Conn_02x02_Odd_Even, Connector_PinHeader_2.54mm:PinHeader_2x02_P2.54mm_Vertical, F.Cu at (179.8, 196.6)
- added J702: Conn_01x08_Male, Connector_PinHeader_2.54mm:PinHeader_1x08_P2.54mm_Vertical, F.Cu at (160.7, 186.1)
- added J703: Conn_01x08_Male, Connector_PinHeader_2.54mm:PinHeader_1x08_P2.54mm_Vertical, F.Cu at (156.1, 186.1)
- added J704: USB_C_Receptacle_USB2.0, Connector_USB:USB_C_Receptacle_HRO_TYPE-C-31-M-12, F.Cu at (183.6, 189.6)
- added R306: 2.2k, Resistor_SMD:R_0402_1005Metric, F.Cu at (111.0, 149.8)
- added R409: 8.2k, Resistor_SMD:R_0402_1005Metric, F.Cu at (151.7, 138.9)
- added R410: 68k, Resistor_SMD:R_0402_1005Metric, F.Cu at (138.6, 142.4)
- added R701: 12k, Resistor_SMD:R_0402_1005Metric, F.Cu at (179.0, 202.4)
- added R702: 12k, Resistor_SMD:R_0402_1005Metric, F.Cu at (194.9, 184.8)
- added R703: 10k, Resistor_SMD:R_0402_1005Metric, F.Cu at (186.2, 195.2)
- added R704: 10k, Resistor_SMD:R_0402_1005Metric, F.Cu at (169.7, 207.5)
- added R705: 10k, Resistor_SMD:R_0402_1005Metric, F.Cu at (190.9, 187.3)
- added R706: 5.1k, Resistor_SMD:R_0402_1005Metric, F.Cu at (169.7, 209.4)
- added R707: 5.1k, Resistor_SMD:R_0402_1005Metric, F.Cu at (169.7, 205.5)
- added R708: 2.2k, Resistor_SMD:R_0402_1005Metric, F.Cu at (172.6, 205.5)
- added RN301: 10k, Resistor_SMD:R_Array_Convex_2x0402, F.Cu at (226.4, 185.2)
- added RN302: 10k, Resistor_SMD:R_Array_Convex_2x0402, F.Cu at (213.0, 197.5)
- added RN601: 10k, Resistor_SMD:R_Array_Convex_2x0402, F.Cu at (129.7, 161.5)
- added TP201: TestPoint, TestPoint:TestPoint_Pad_D2.0mm, F.Cu at (105.8, 172.5)
- added TP202: TestPoint, TestPoint:TestPoint_Pad_D2.0mm, F.Cu at (101.6, 175.4)
- added TP203: TestPoint, TestPoint:TestPoint_Pad_D2.0mm, F.Cu at (116.8, 162.0)
- added U409: BL1551B, Package_TO_SOT_SMD:SOT-363_SC-70-6, F.Cu at (155.9, 215.4)
- added U410: NE555DR, Package_SO:SOIC-8_3.9x4.9mm_P1.27mm, F.Cu at (141.3, 135.2)
- added U701: FT2232HL, Package_QFP:LQFP-64_10x10mm_P0.5mm, F.Cu at (170.3, 197.2)
- added U702: 93LC56BT-I/OT, Package_TO_SOT_SMD:SOT-23-6, F.Cu at (165.6, 206.7)
- added Y701: 12MHz, Crystal:Crystal_SMD_HC49-SD, F.Cu at (170.4, 186.9)
- C306, C307: value 10u -> 0.1u
- C308: value 0.1u -> 3.3u
- C309: value 27p -> 4.7u
- C310: value 27p -> 0.1u
- C401, C402, C404, C406, R401, R402, R403, R407, RN401, RN402, RN403, RN407, U601: moved to B.Cu
- D201, D202: value PMEG40 -> LED; footprint Diode_SMD:D_SOD-323 -> LED_SMD:LED_0402_1005Metric
- D203: value LED -> D5V0L1B2S9-7; footprint LED_SMD:LED_0402_1005Metric -> Diode_SMD:D_SOD-923
- D204: value LED -> GBLC03CI; footprint LED_SMD:LED_0402_1005Metric -> Diode_SMD:D_SOD-323
- J201: value USB_C_Receptacle_USB2.0 -> Conn_01x03_Male; footprint Connector_USB:USB_C_Receptacle_HRO_TYPE-C-31-M-12 -> Connector_PinHeader_2.54mm:PinHeader_1x03_P2.54mm_Horizontal
- J202: value Conn_01x02_Male -> USB_C_Receptacle_USB2.0; footprint Connector_PinHeader_2.54mm:PinHeader_1x02_P2.54mm_Horizontal -> Connector_USB:USB_C_Receptacle_HRO_TYPE-C-31-M-12
- J301: value Conn_01x04_Male -> Conn_02x06_Odd_Even; footprint Connector_PinHeader_2.54mm:PinHeader_1x04_P2.54mm_Horizontal -> Connector_PinHeader_2.54mm:PinHeader_2x06_P2.54mm_Vertical
- J302: value Conn_01x03_Male -> Conn_01x04_Male; footprint Connector_PinHeader_2.54mm:PinHeader_1x03_P2.54mm_Vertical -> Connector_PinHeader_2.54mm:PinHeader_1x04_P2.54mm_Horizontal
- R301, R302: value 10k -> 12k
- R303, R304: value 12k -> 10k
- R305: value 2.2k -> 10k
- U301: value FT232HQ-REEL -> FT2232HL; footprint Package_DFN_QFN:QFN-48-1EP_8x8mm_P0.5mm_EP6.2x6.2mm -> Package_QFP:LQFP-64_10x10mm_P0.5mm
- U302: value SN74LVC157ADR -> 93LC56BT-I/OT; footprint Package_SO:SOIC-16_3.9x9.9mm_P1.27mm -> Package_TO_SOT_SMD:SOT-23-6
- U401, U402, U403, U407: value MCP23017_SS -> MCP23017T-E/SS; moved to B.Cu
- U404, U405, U406, U408: value MCP23017_SS -> MCP23017T-E/SS
- moved R301 149.7 mm to (102.4, 147.5)
- moved U301 146.2 mm to (104.2, 139.2)
- moved U302 146.0 mm to (107.0, 148.7)
- moved R302 144.3 mm to (108.9, 151.9)
- moved FB302 140.5 mm to (98.9, 147.7)
- moved C602 138.6 mm to (132.6, 162.9)
- moved C601 138.2 mm to (132.6, 161.0)
- moved C308 138.0 mm to (119.7, 147.2), turned to 0 degrees
- moved R303 136.9 mm to (113.9, 147.8), turned to 0 degrees
- moved C303 134.2 mm to (126.2, 139.9), turned to 0 degrees
- moved C302 132.3 mm to (126.2, 135.9)
- moved Y301 132.2 mm to (97.0, 152.5), turned to 0 degrees
- moved C307 132.0 mm to (105.8, 154.8), turned to 0 degrees
- moved C304 129.7 mm to (126.2, 137.9), turned to 0 degrees
- moved R304 129.4 mm to (111.0, 147.8), turned to 0 degrees
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Connections:
- C201 pad 1: Net-(C201-Pad1) -> +5V
- C202 pad 1: Net-(C202-Pad1) -> +3V3
- C205 pad 1: EXT5V_IN -> PI4.3V3
- C206 pad 1: +5V -> +3V3
- C304 pad 1: GND -> +3V3
- C304 pad 2: Net-(C304-Pad2) -> GND
- C305 pad 1: GND -> +1V8
- C305 pad 2: +1V8 -> GND
- C306 pad 1: VPHY -> +1V8
- C307 pad 1: VPLL -> +1V8
- C308 pad 1: GND -> +1V8
- C308 pad 2: +3V3 -> GND
- C309 pad 1: GND -> VPHY
- C309 pad 2: /FTDI/XCSI -> GND
- C310 pad 1: GND -> VPHY
- C310 pad 2: /FTDI/XCSO -> GND
- C405 pad 2: +3V3 -> MCP5.PWR
- D201 pad 1: Net-(C201-Pad1) -> GND
- D201 pad 2: +5V -> Net-(D201-Pad2)
- D202 pad 1: +3V3 -> GND
- D202 pad 2: Net-(C202-Pad1) -> Net-(D202-Pad2)
- D203 pad 2: Net-(D203-Pad2) -> +5V
- D204 pad 2: Net-(D204-Pad2) -> +3V3
- FB201 pad 1: Net-(D205-Pad1) -> PWRU_IN
- FB202 pad 1: Net-(D206-Pad1) -> PI4.3V3
- FB202 pad 2: +5V -> +3V3
- J301 pad 1: CONN.SCK -> IO.SCK0
- J301 pad 2: CONN.SDO -> IO.SCK1
- J301 pad 3: CONN.SDI -> IO.SDA0
- J301 pad 4: CONN.~{CS} -> IO.SDA1
- J302 pad 1: +3V3 -> IO.SCK1
- J302 pad 2: SEL -> IO.SDA1
- J302 pad 3: GND -> IO.SCK0
- R201 pad 2: Net-(D203-Pad2) -> Net-(D201-Pad2)
- R202 pad 1: Net-(J201-PadA5) -> Net-(J202-PadA5)
- R203 pad 2: Net-(J201-PadB5) -> Net-(J202-PadB5)
- R204 pad 2: Net-(D204-Pad2) -> Net-(D202-Pad2)
- R301 pad 1: +3V3 -> Net-(R301-Pad1)
- R301 pad 2: FTDI.SDA -> GND
- R302 pad 1: +3V3 -> Net-(R302-Pad1)
- R302 pad 2: FTDI.SCK -> +3V3
- R303 pad 1: Net-(R303-Pad1) -> +3V3
- R303 pad 2: +3V3 -> Net-(R303-Pad2)
- R304 pad 1: Net-(R304-Pad1) -> +3V3
- R304 pad 2: GND -> EECLK
- R305 pad 1: Net-(R305-Pad1) -> +3V3
- R305 pad 2: EEDATA -> EECS
- RN401 pad 1: Net-(RN401-Pad1) -> INTA.MCP0
- RN401 pad 2: Net-(RN401-Pad2) -> INTB.MCP0
- RN402 pad 1: Net-(RN402-Pad1) -> INTA.MCP1
- RN403 pad 1: Net-(RN403-Pad1) -> INTA.MCP2
- RN403 pad 2: Net-(RN403-Pad2) -> INTB.MCP2
- RN404 pad 1: Net-(RN404-Pad1) -> INTA.MCP3
- RN404 pad 2: Net-(RN404-Pad2) -> INTB.MCP3
- RN405 pad 1: Net-(RN405-Pad1) -> INTA.MCP4
- RN405 pad 2: Net-(RN405-Pad2) -> INTB.MCP4
- RN406 pad 1: Net-(RN406-Pad1) -> INTA.MCP5
- RN406 pad 2: Net-(RN406-Pad2) -> INTB.MCP5
- RN407 pad 1: Net-(RN407-Pad1) -> INTA.MCP6
- RN407 pad 2: Net-(RN407-Pad2) -> INTB.MCP6
- RN408 pad 1: Net-(RN408-Pad1) -> INTA.MCP7
- RN408 pad 2: Net-(RN408-Pad2) -> INTB.MCP7
- U201 pad 2: Net-(C202-Pad1) -> +3V3
- U201 pad 3: Net-(C201-Pad1) -> +5V
- U301 pad 1: /FTDI/XCSI -> GND
- U301 pad 12: +3V3 -> +1V8
- U301 pad 13: FTDI.SCK -> GND
- U301 pad 14: FTDI.SDA -> Net-(R302-Pad1)
- U301 pad 15: unconnected-(U301-Pad15) -> GND
- U301 pad 16: unconnected-(U301-Pad16) -> FTDI.SCK0
- U301 pad 17: unconnected-(U301-Pad17) -> FTDI.SDA0
- U301 pad 18: unconnected-(U301-Pad18) -> FTDI.SDA0
- U301 pad 2: /FTDI/XCSO -> /FTDI/XCSI
- U301 pad 20: unconnected-(U301-Pad20) -> +3V3
- U301 pad 22: GND -> unconnected-(U301-Pad22)
- U301 pad 23: GND -> unconnected-(U301-Pad23)
- U301 pad 24: +3V3 -> unconnected-(U301-Pad24)
- U301 pad 25: unconnected-(U301-Pad25) -> GND
- U301 pad 3: VPHY -> /FTDI/XCSO
- U301 pad 31: unconnected-(U301-Pad31) -> +3V3
- U301 pad 34: Net-(R303-Pad1) -> unconnected-(U301-Pad34)
- U301 pad 36: GND -> unconnected-(U301-Pad36)
- U301 pad 37: Net-(C304-Pad2) -> +1V8
- U301 pad 38: +1V8 -> FTDI.SCK1
- U301 pad 39: +3V3 -> FTDI.SDA1
- U301 pad 4: GND -> VPHY
- U301 pad 40: +3V3 -> FTDI.SDA1
- U301 pad 41: GND -> unconnected-(U301-Pad41)
- U301 pad 42: GND -> +3V3
- U301 pad 43: EEDATA -> unconnected-(U301-Pad43)
- U301 pad 44: EECLK -> unconnected-(U301-Pad44)
- U301 pad 45: EECS -> unconnected-(U301-Pad45)
- U301 pad 46: +3V3 -> unconnected-(U301-Pad46)
- U301 pad 48: GND -> unconnected-(U301-Pad48)
- U301 pad 49: GND -> +1V8
- U301 pad 5: Net-(R304-Pad1) -> GND
- U301 pad 6: FTDI.D- -> Net-(R301-Pad1)
- U301 pad 7: FTDI.D+ -> FTDI.D-
- U301 pad 8: VPLL -> FTDI.D+
- U301 pad 9: GND -> VPLL
- U302 pad 1: SEL -> Net-(R303-Pad2)
- U302 pad 2: FTDI.SCK -> GND
- U302 pad 3: CONN.SCK -> EEDATA
- U302 pad 4: IO.SCK -> EECLK
- U302 pad 5: FTDI.SDO -> EECS
- U302 pad 6: CONN.SDO -> +3V3
- U401 pad 1: IO.HWCLK -> IO.PB8
- U401 pad 12: IO.SCK -> IO.SCK0
- U401 pad 13: IO.SDA -> IO.SDA0
- U401 pad 19: Net-(RN401-Pad2) -> INTB.MCP0
- U401 pad 2: IO.PB20 -> IO.PB9
- U401 pad 20: Net-(RN401-Pad1) -> INTA.MCP0
- U401 pad 21: IO.PB13 -> IO.PB0
- U401 pad 22: IO.PB12 -> IO.PB1
- U401 pad 23: IO.PB11 -> IO.PB2
- U401 pad 24: IO.PB10 -> IO.PB3
- U401 pad 25: IO.PB9 -> IO.PB4
- U401 pad 26: IO.PB8 -> IO.PB5
- U401 pad 27: unconnected-(U401-Pad27) -> IO.PB6
- U401 pad 28: unconnected-(U401-Pad28) -> IO.PB7
- U401 pad 3: IO.PB19 -> IO.PB10
- U401 pad 4: IO.PB18 -> IO.PB11
- U401 pad 5: IO.PB17 -> IO.PB12
- U401 pad 6: IO.PB16 -> IO.PB13
- U401 pad 7: IO.PB15 -> IO.PB14
- U401 pad 8: IO.PB14 -> IO.PB15
- U402 pad 1: IO.PB7 -> unconnected-(U402-Pad1)
- U402 pad 12: IO.SCK -> IO.SCK0
- U402 pad 13: IO.SDA -> IO.SDA0
- U402 pad 2: IO.PB6 -> unconnected-(U402-Pad2)
- U402 pad 20: Net-(RN402-Pad1) -> INTA.MCP1
- U402 pad 21: IO.SS0_0 -> IO.PB16
- U402 pad 22: IO.SS0_1 -> IO.PB17
- U402 pad 23: IO.SS0_2 -> IO.PB18
- U402 pad 24: IO.SS0_3 -> IO.PB19
- U402 pad 25: IO.SS0_4 -> IO.PB20
- U402 pad 26: IO.SS0_5 -> unconnected-(U402-Pad26)
- U402 pad 27: IO.SS0_6 -> unconnected-(U402-Pad27)
- U402 pad 28: IO.SS0_7 -> unconnected-(U402-Pad28)
- U402 pad 3: IO.PB5 -> unconnected-(U402-Pad3)
- U402 pad 4: IO.PB4 -> unconnected-(U402-Pad4)
- U402 pad 5: IO.PB3 -> unconnected-(U402-Pad5)
- U402 pad 6: IO.PB2 -> unconnected-(U402-Pad6)
- U402 pad 7: IO.PB1 -> unconnected-(U402-Pad7)
- U402 pad 8: IO.PB0 -> unconnected-(U402-Pad8)
- U403 pad 12: IO.SCK -> IO.SCK1
- U403 pad 13: IO.SDA -> IO.SDA1
- U403 pad 19: Net-(RN403-Pad2) -> INTB.MCP2
- U403 pad 20: Net-(RN403-Pad1) -> INTA.MCP2
- U403 pad 21: IO.SS2_0 -> IO.SS0_0
- U403 pad 22: IO.SS2_1 -> IO.SS0_1
- U403 pad 23: IO.SS2_2 -> IO.SS0_2
- U403 pad 24: IO.SS2_3 -> IO.SS0_3
- U403 pad 25: IO.SS2_4 -> IO.SS0_4
- U403 pad 26: IO.SS2_5 -> IO.SS0_5
- U403 pad 27: IO.SS2_6 -> IO.SS0_6
- U403 pad 28: IO.SS2_7 -> IO.SS0_7
- U404 pad 12: IO.SCK -> IO.SCK1
- U404 pad 13: IO.SDA -> IO.SDA1
- U404 pad 19: Net-(RN404-Pad2) -> INTB.MCP3
- U404 pad 20: Net-(RN404-Pad1) -> INTA.MCP3
- U404 pad 21: IO.SS4_0 -> IO.SS2_0
- U404 pad 22: IO.SS4_1 -> IO.SS2_1
- U404 pad 23: IO.SS4_2 -> IO.SS2_2
- U404 pad 24: IO.SS4_3 -> IO.SS2_3
- U404 pad 25: IO.SS4_4 -> IO.SS2_4
- U404 pad 26: IO.SS4_5 -> IO.SS2_5
- U404 pad 27: IO.SS4_6 -> IO.SS2_6
- U404 pad 28: IO.SS4_7 -> IO.SS2_7
- U405 pad 12: IO.SCK -> IO.SCK1
- U405 pad 13: IO.SDA -> IO.SDA1
- U405 pad 19: Net-(RN405-Pad2) -> INTB.MCP4
- U405 pad 20: Net-(RN405-Pad1) -> INTA.MCP4
- U405 pad 21: IO.SS6_0 -> IO.SS4_0
- U405 pad 22: IO.SS6_1 -> IO.SS4_1
- U405 pad 23: IO.SS6_2 -> IO.SS4_2
- U405 pad 24: IO.SS6_3 -> IO.SS4_3
- U405 pad 25: IO.SS6_4 -> IO.SS4_4
- U405 pad 26: IO.SS6_5 -> IO.SS4_5
- U405 pad 27: IO.SS6_6 -> IO.SS4_6
- U405 pad 28: IO.SS6_7 -> IO.SS4_7
- U406 pad 12: IO.SCK -> IO.SCK1
- U406 pad 13: IO.SDA -> IO.SDA1
- U406 pad 19: Net-(RN406-Pad2) -> INTB.MCP5
- U406 pad 20: Net-(RN406-Pad1) -> INTA.MCP5
- U406 pad 21: IO.LEFT7 -> IO.SS6_0
- U406 pad 22: IO.LEFT6 -> IO.SS6_1
- U406 pad 23: IO.LEFT5 -> IO.SS6_2
- U406 pad 24: IO.LEFT4 -> IO.SS6_3
- U406 pad 25: IO.LEFT3 -> IO.SS6_4
- U406 pad 26: IO.LEFT2 -> IO.SS6_5
- U406 pad 27: IO.LEFT1 -> IO.SS6_6
- U406 pad 28: IO.LEFT0 -> IO.SS6_7
- U406 pad 9: +3V3 -> MCP5.PWR
- U407 pad 1: IO.RIGHT7 -> IO.LEFT0
- U407 pad 12: IO.SCK -> IO.SCK1
- U407 pad 13: IO.SDA -> IO.SDA1
- U407 pad 19: Net-(RN407-Pad2) -> INTB.MCP6
- U407 pad 2: IO.RIGHT6 -> IO.LEFT1
- U407 pad 20: Net-(RN407-Pad1) -> INTA.MCP6
- U407 pad 21: IO.RED -> IO.RIGHT0
- U407 pad 22: IO.GREEN -> IO.RIGHT1
- U407 pad 23: IO.BLUE -> IO.RIGHT2
- U407 pad 24: unconnected-(U407-Pad24) -> IO.RIGHT3
- U407 pad 25: unconnected-(U407-Pad25) -> IO.RIGHT4
- U407 pad 26: unconnected-(U407-Pad26) -> IO.RIGHT5
- U407 pad 27: unconnected-(U407-Pad27) -> IO.RIGHT6
- U407 pad 28: unconnected-(U407-Pad28) -> IO.RIGHT7
- U407 pad 3: IO.RIGHT5 -> IO.LEFT2
- U407 pad 4: IO.RIGHT4 -> IO.LEFT3
- U407 pad 5: IO.RIGHT3 -> IO.LEFT4
- U407 pad 6: IO.RIGHT2 -> IO.LEFT5
- U407 pad 7: IO.RIGHT1 -> IO.LEFT6
- U407 pad 8: IO.RIGHT0 -> IO.LEFT7
- U408 pad 12: IO.SCK -> IO.SCK1
- U408 pad 13: IO.SDA -> IO.SDA1
- U408 pad 19: Net-(RN408-Pad2) -> INTB.MCP7
- U408 pad 20: Net-(RN408-Pad1) -> INTA.MCP7
- U408 pad 21: unconnected-(U408-Pad21) -> IO.RED
- U408 pad 22: unconnected-(U408-Pad22) -> IO.GREEN
- U408 pad 23: unconnected-(U408-Pad23) -> IO.BLUE
- U408 pad 28: unconnected-(U408-Pad28) -> IO.PB20
- U408 pad 8: unconnected-(U408-Pad8) -> IO.HWCLK
- U501 pad 119: IO.IO0 -> unconnected-(U501-Pad119)
- U501 pad 158: FPGA.1V2 -> unconnected-(U501-Pad158)
- U501 pad 159: IO.IO1 -> unconnected-(U501-Pad159)
- U501 pad 160: FPGA.1V2 -> unconnected-(U501-Pad160)
- U501 pad 38: FPGA.3V3 -> unconnected-(U501-Pad38)
- U501 pad 39: IO.IO3 -> unconnected-(U501-Pad39)
- U501 pad 40: FPGA.3V3 -> unconnected-(U501-Pad40)
- U501 pad 79: IO.IO2 -> unconnected-(U501-Pad79)
- U601 pad 11: unconnected-(U601-Pad11) -> INTA.MCP5
- U601 pad 12: unconnected-(U601-Pad12) -> INTA.MCP6
- U601 pad 13: unconnected-(U601-Pad13) -> INTB.MCP5
- U601 pad 15: unconnected-(U601-Pad15) -> INTB.MCP6
- U601 pad 16: unconnected-(U601-Pad16) -> INTA.MCP7
- U601 pad 18: unconnected-(U601-Pad18) -> INTB.MCP7
- U601 pad 27: unconnected-(U601-Pad27) -> IO.SDA0
- U601 pad 28: unconnected-(U601-Pad28) -> IO.SCK0
- U601 pad 29: IO.IO0 -> INTA.MCP0
- U601 pad 3: IO.SDA -> IO.SDA1
- U601 pad 31: IO.IO1 -> INTB.MCP0
- U601 pad 32: IO.IO2 -> INTA.MCP1
- U601 pad 33: IO.IO3 -> INTA.MCP2
- U601 pad 35: unconnected-(U601-Pad35) -> INTA.MCP3
- U601 pad 36: unconnected-(U601-Pad36) -> INTB.MCP2
- U601 pad 37: unconnected-(U601-Pad37) -> INTB.MCP4
- U601 pad 38: unconnected-(U601-Pad38) -> INTB.MCP3
- U601 pad 40: unconnected-(U601-Pad40) -> INTA.MCP4
- U601 pad 5: IO.SCK -> IO.SCK1
Routing:
- net +3V3: track 228.3 -> 32.8 mm, vias 15 -> 2
- net +5V: track 104.1 -> 0.00 mm, vias 2 -> 0
- net GND: track 92.7 -> 0.00 mm, vias 18 -> 0
- net IO.~{CS}: track 51.5 -> 0.00 mm, vias 1 -> 0
- net IO.SDI: track 48.8 -> 0.00 mm, vias 1 -> 0
- net IO.SCK: track 46.7 -> 0.00 mm, vias 2 -> 0
- net IO.SS1_3: track 0.00 -> 44.2 mm
- net IO.SDO: track 43.6 -> 0.00 mm, vias 1 -> 0
- net IO.BLUE: track 0.00 -> 40.4 mm, vias 0 -> 1
- net IO.SS1_5: track 0.00 -> 39.9 mm
- net IO.RED: track 0.00 -> 38.9 mm, vias 0 -> 1
- net IO.SS1_1: track 0.00 -> 38.8 mm
- net IO.GREEN: track 0.00 -> 38.6 mm, vias 0 -> 1
- net IO.SS5_7: track 18.8 -> 56.9 mm
- net IO.SS5_6: track 33.4 -> 70.7 mm
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Other:
- board size 82.4 x 76.2 mm -> 89 x 76.2 mm

Commit message: Update 7/30
Parts:
- removed the J701 at (179.8, 196.6)
- added J601: Conn_02x02_Odd_Even, Connector_PinHeader_2.54mm:PinHeader_2x02_P2.54mm_Vertical, F.Cu at (137.6, 190.0)
- added J602: Conn_02x02_Odd_Even, Connector_PinHeader_2.54mm:PinHeader_2x02_P2.54mm_Vertical, F.Cu at (144.8, 190.0)
- added J702: Conn_01x08_Male, Connector_PinHeader_2.54mm:PinHeader_1x08_P2.54mm_Vertical, F.Cu at (111.5, 190.0)
- added J704: Conn_01x08_Male, Connector_PinHeader_2.54mm:PinHeader_1x08_P2.54mm_Vertical, F.Cu at (116.2, 190.0)
- added U410: BL1551B, Package_TO_SOT_SMD:SOT-363_SC-70-6, B.Cu at (187.2, 118.0)
- C701, C703, C704, C705, C706, C707, C708, C715, R701, R702, R703, R704, R705, R708, RN301, RN302, U701, U702: moved to B.Cu
- J201: footprint Connector_PinHeader_2.54mm:PinHeader_1x03_P2.54mm_Horizontal -> Connector_PinHeader_2.54mm:PinHeader_1x03_P2.54mm_Vertical
- J302: footprint Connector_PinHeader_2.54mm:PinHeader_1x04_P2.54mm_Horizontal -> Connector_PinHeader_2.54mm:PinHeader_1x04_P2.54mm_Vertical
- moved D701 145.1 mm to (222.6, 72.2)
- moved R706 140.9 mm to (217.6, 77.0), turned to -90 degrees
- moved FB701 138.9 mm to (214.1, 81.3), turned to 90 degrees
- moved FB702 138.3 mm to (216.6, 81.3), turned to 90 degrees
- moved R707 136.1 mm to (214.6, 77.0), turned to 90 degrees
- moved C705 135.8 mm to (218.0, 76.5), turned to 90 degrees
- moved U409 134.0 mm to (213.3, 94.3)
- moved C707 133.3 mm to (210.1, 79.6), turned to 180 degrees
- moved C702 132.0 mm to (220.6, 83.4), turned to -90 degrees
- moved R701 131.0 mm to (215.1, 76.5), turned to 90 degrees
- moved U702 130.6 mm to (206.8, 82.8), turned to 180 degrees
- moved C711 129.4 mm to (217.9, 81.0), turned to -90 degrees
- moved R704 126.5 mm to (208.2, 86.9), turned to 180 degrees
- moved R708 125.9 mm to (208.2, 84.7)
- moved C708 125.5 mm to (208.2, 89.1), turned to 180 degrees
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- renumbered J702 to J701, J704 to J705, U410 to U411
Connections:
- net IO.SS4_0 renamed /GPIO Expansion/IO.SS4_0
- net IO.SS4_1 renamed /GPIO Expansion/IO.SS4_1
- net IO.SS4_2 renamed /GPIO Expansion/IO.SS4_2
- net IO.SS4_3 renamed /GPIO Expansion/IO.SS4_3
- net IO.SS4_4 renamed /GPIO Expansion/IO.SS4_4
- net IO.SS4_5 renamed /GPIO Expansion/IO.SS4_5
- net IO.SS4_6 renamed /GPIO Expansion/IO.SS4_6
- net IO.SS4_7 renamed /GPIO Expansion/IO.SS4_7
- net IO.SS5_0 renamed /GPIO Expansion/IO.SS5_0
- net IO.SS5_1 renamed /GPIO Expansion/IO.SS5_1
- net IO.SS5_2 renamed /GPIO Expansion/IO.SS5_2
- net IO.SS5_3 renamed /GPIO Expansion/IO.SS5_3
- net IO.SS5_4 renamed /GPIO Expansion/IO.SS5_4
- net IO.SS5_5 renamed /GPIO Expansion/IO.SS5_5
- net IO.SS5_6 renamed /GPIO Expansion/IO.SS5_6
- net IO.SS5_7 renamed /GPIO Expansion/IO.SS5_7
- C406 pad 2: +3V3 -> MCP6.PWR
- J701 pad 1: IO.SS7_0 -> /GPIO Expansion/IO.SS7_0
- J701 pad 2: IO.SS7_1 -> /GPIO Expansion/IO.SS7_1
- J701 pad 3: IO.SS7_2 -> /GPIO Expansion/IO.SS7_2
- J701 pad 4: IO.SS7_3 -> /GPIO Expansion/IO.SS7_3
- J701 pad 5: IO.SS7_4 -> /GPIO Expansion/IO.SS7_4
- J701 pad 6: IO.SS7_5 -> /GPIO Expansion/IO.SS7_5
- J701 pad 7: IO.SS7_6 -> /GPIO Expansion/IO.SS7_6
- J701 pad 8: IO.SS7_7 -> /GPIO Expansion/IO.SS7_7
- U406 pad 1: IO.SS7_0 -> /GPIO Expansion/IO.SS7_0
- U406 pad 2: IO.SS7_1 -> /GPIO Expansion/IO.SS7_1
- U406 pad 3: IO.SS7_2 -> /GPIO Expansion/IO.SS7_2
- U406 pad 4: IO.SS7_3 -> /GPIO Expansion/IO.SS7_3
- U406 pad 5: IO.SS7_4 -> /GPIO Expansion/IO.SS7_4
- U406 pad 6: IO.SS7_5 -> /GPIO Expansion/IO.SS7_5
- U406 pad 7: IO.SS7_6 -> /GPIO Expansion/IO.SS7_6
- U406 pad 8: IO.SS7_7 -> /GPIO Expansion/IO.SS7_7
- U407 pad 1: IO.LEFT0 -> /GPIO Expansion/IO.LEFT0
- U407 pad 2: IO.LEFT1 -> /GPIO Expansion/IO.LEFT1
- U407 pad 21: IO.RIGHT0 -> /GPIO Expansion/IO.RIGHT0
- U407 pad 22: IO.RIGHT1 -> /GPIO Expansion/IO.RIGHT1
- U407 pad 23: IO.RIGHT2 -> /GPIO Expansion/IO.RIGHT2
- U407 pad 24: IO.RIGHT3 -> /GPIO Expansion/IO.RIGHT3
- U407 pad 25: IO.RIGHT4 -> /GPIO Expansion/IO.RIGHT4
- U407 pad 26: IO.RIGHT5 -> /GPIO Expansion/IO.RIGHT5
- U407 pad 27: IO.RIGHT6 -> /GPIO Expansion/IO.RIGHT6
- U407 pad 28: IO.RIGHT7 -> /GPIO Expansion/IO.RIGHT7
- U407 pad 3: IO.LEFT2 -> /GPIO Expansion/IO.LEFT2
- U407 pad 4: IO.LEFT3 -> /GPIO Expansion/IO.LEFT3
- U407 pad 5: IO.LEFT4 -> /GPIO Expansion/IO.LEFT4
- U407 pad 6: IO.LEFT5 -> /GPIO Expansion/IO.LEFT5
- U407 pad 7: IO.LEFT6 -> /GPIO Expansion/IO.LEFT6
- U407 pad 8: IO.LEFT7 -> /GPIO Expansion/IO.LEFT7
- U407 pad 9: +3V3 -> MCP6.PWR
- U501 pad 123: IO.SS7_3 -> /GPIO Expansion/IO.SS7_3
- U501 pad 124: IO.LEFT7 -> /GPIO Expansion/IO.LEFT7
- U501 pad 125: IO.SS7_5 -> /GPIO Expansion/IO.SS7_5
- U501 pad 126: IO.SS7_4 -> /GPIO Expansion/IO.SS7_4
- U501 pad 127: IO.LEFT6 -> /GPIO Expansion/IO.LEFT6
- U501 pad 128: IO.SS7_6 -> /GPIO Expansion/IO.SS7_6
- U501 pad 131: IO.SS7_1 -> /GPIO Expansion/IO.SS7_1
- U501 pad 132: IO.SS7_0 -> /GPIO Expansion/IO.SS7_0
- U501 pad 133: IO.SS7_7 -> /GPIO Expansion/IO.SS7_7
- U501 pad 134: IO.SS7_2 -> /GPIO Expansion/IO.SS7_2
- U501 pad 136: IO.LEFT5 -> /GPIO Expansion/IO.LEFT5
- U501 pad 141: IO.LEFT4 -> /GPIO Expansion/IO.LEFT4
- U501 pad 15: IO.RIGHT2 -> /GPIO Expansion/IO.RIGHT2
- U501 pad 150: IO.LEFT3 -> /GPIO Expansion/IO.LEFT3
- U501 pad 155: IO.LEFT2 -> /GPIO Expansion/IO.LEFT2
- U501 pad 23: IO.RIGHT3 -> /GPIO Expansion/IO.RIGHT3
- U501 pad 3: IO.RIGHT0 -> /GPIO Expansion/IO.RIGHT0
- U501 pad 30: IO.RIGHT4 -> /GPIO Expansion/IO.RIGHT4
- U501 pad 37: IO.RIGHT5 -> /GPIO Expansion/IO.RIGHT5
- U501 pad 46: IO.LEFT1 -> /GPIO Expansion/IO.LEFT1
- U501 pad 51: IO.LEFT0 -> /GPIO Expansion/IO.LEFT0
- U501 pad 67: IO.RIGHT7 -> /GPIO Expansion/IO.RIGHT7
- U501 pad 76: IO.RIGHT6 -> /GPIO Expansion/IO.RIGHT6
- U501 pad 8: IO.RIGHT1 -> /GPIO Expansion/IO.RIGHT1
- U601 pad 22: unconnected-(U601-Pad22) -> MCP5.SEL
- U601 pad 24: unconnected-(U601-Pad24) -> MCP6.SEL
- U701 pad 1: Net-(U701-Pad1) -> GND
- U701 pad 10: Net-(U701-Pad1) -> GND
- U701 pad 11: Net-(U701-Pad1) -> GND
- U701 pad 15: Net-(U701-Pad1) -> GND
- U701 pad 16: unconnected-(U701-Pad16) -> /GPIO Expansion/IO.SS7_0
- U701 pad 17: unconnected-(U701-Pad17) -> /GPIO Expansion/IO.SS7_1
- U701 pad 18: unconnected-(U701-Pad18) -> /GPIO Expansion/IO.SS7_2
- U701 pad 19: unconnected-(U701-Pad19) -> /GPIO Expansion/IO.SS7_3
- U701 pad 21: MCP5.SEL -> /GPIO Expansion/IO.SS7_4
- U701 pad 22: IO.SS7_0 -> /GPIO Expansion/IO.SS7_5
- U701 pad 23: IO.SS7_1 -> /GPIO Expansion/IO.SS7_6
- U701 pad 24: IO.SS7_2 -> /GPIO Expansion/IO.SS7_7
- U701 pad 25: Net-(U701-Pad1) -> GND
- U701 pad 26: IO.SS7_3 -> IO.SS6_0
- U701 pad 27: IO.SS7_4 -> IO.SS6_1
- U701 pad 28: IO.SS7_5 -> IO.SS6_2
- U701 pad 29: IO.SS7_6 -> IO.SS6_3
- U701 pad 30: IO.SS7_7 -> IO.SS6_4
- U701 pad 32: unconnected-(U701-Pad32) -> IO.SS6_5
- U701 pad 33: unconnected-(U701-Pad33) -> IO.SS6_6
- U701 pad 34: unconnected-(U701-Pad34) -> IO.SS6_7
- U701 pad 35: Net-(U701-Pad1) -> GND
- U701 pad 38: unconnected-(U701-Pad38) -> /GPIO Expansion/IO.LEFT0
- U701 pad 39: unconnected-(U701-Pad39) -> /GPIO Expansion/IO.LEFT1
- U701 pad 40: unconnected-(U701-Pad40) -> /GPIO Expansion/IO.LEFT2
- U701 pad 41: unconnected-(U701-Pad41) -> /GPIO Expansion/IO.LEFT3
- U701 pad 43: IO.SS6_0 -> /GPIO Expansion/IO.LEFT4
- U701 pad 44: IO.SS6_1 -> /GPIO Expansion/IO.LEFT5
- U701 pad 45: IO.SS6_2 -> /GPIO Expansion/IO.LEFT6
- U701 pad 46: IO.SS6_3 -> /GPIO Expansion/IO.LEFT7
- U701 pad 47: Net-(U701-Pad1) -> GND
- U701 pad 48: IO.SS6_4 -> /GPIO Expansion/IO.RIGHT0
- U701 pad 5: Net-(U701-Pad1) -> GND
- U701 pad 51: Net-(U701-Pad1) -> GND
- U701 pad 52: IO.SS6_5 -> /GPIO Expansion/IO.RIGHT1
- U701 pad 53: IO.SS6_6 -> /GPIO Expansion/IO.RIGHT2
- U701 pad 54: IO.SS6_7 -> /GPIO Expansion/IO.RIGHT3
- U701 pad 55: unconnected-(U701-Pad55) -> /GPIO Expansion/IO.RIGHT4
- U701 pad 57: unconnected-(U701-Pad57) -> /GPIO Expansion/IO.RIGHT5
- U701 pad 58: unconnected-(U701-Pad58) -> /GPIO Expansion/IO.RIGHT6
- U701 pad 59: unconnected-(U701-Pad59) -> /GPIO Expansion/IO.RIGHT7
Routing:
- net /GPIO Expansion/IO.RIGHT5: track 0.00 -> 139.7 mm, vias 0 -> 2
- net /GPIO Expansion/IO.RIGHT6: track 0.00 -> 119.1 mm, vias 0 -> 3
- net /GPIO Expansion/IO.LEFT2: track 0.00 -> 115.4 mm, vias 0 -> 2
- net IO.SDA1: track 0.00 -> 113.8 mm, vias 0 -> 8
- net IO.SCK1: track 0.00 -> 113.1 mm, vias 0 -> 7
- net /GPIO Expansion/IO.LEFT7: track 0.00 -> 110.0 mm, vias 0 -> 2
- net /GPIO Expansion/IO.LEFT3: track 0.00 -> 107.2 mm, vias 0 -> 3
- net /GPIO Expansion/IO.RIGHT4: track 0.00 -> 106.4 mm, vias 0 -> 2
- net /GPIO Expansion/IO.LEFT4: track 0.00 -> 104.1 mm, vias 0 -> 3
- net /GPIO Expansion/IO.LEFT5: track 0.00 -> 103.6 mm, vias 0 -> 3
- net /GPIO Expansion/IO.LEFT6: track 0.00 -> 100.9 mm, vias 0 -> 2
- net /GPIO Expansion/IO.RIGHT3: track 0.00 -> 99.7 mm, vias 0 -> 3
- net /GPIO Expansion/IO.RIGHT0: track 0.00 -> 95.7 mm, vias 0 -> 2
- net /GPIO Expansion/IO.RIGHT7: track 0.00 -> 95.3 mm, vias 0 -> 3
- net /GPIO Expansion/IO.RIGHT2: track 0.00 -> 91.5 mm, vias 0 -> 3
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
Commit message: Update 8/2
Parts:
- removed the J701 at (128.6, 183.8)
- removed J702, J703, J704: Conn_01x08_Male, Connector_PinHeader_2.54mm:PinHeader_1x08_P2.54mm_Vertical
- added J203: Conn_01x02_Male, Connector_PinHeader_2.54mm:PinHeader_1x02_P2.54mm_Vertical, F.Cu at (248.7, 142.1)
- added J303: Conn_01x06_Male, Connector_PinHeader_2.54mm:PinHeader_1x06_P2.54mm_Vertical, F.Cu at (255.1, 120.8)
- added J304: Conn_01x06_Male, Connector_PinHeader_2.54mm:PinHeader_1x06_P2.54mm_Vertical, F.Cu at (255.1, 90.3)
- added J305: Conn_01x04_Male, Connector_PinHeader_2.54mm:PinHeader_1x04_P2.54mm_Horizontal, F.Cu at (238.2, 79.2)
- C302, C303, C304, C306, C308, C313, C314, C315, C601, C602, R301, R303, R304, R305, R306, U302, Y301: moved to B.Cu
- J302: footprint Connector_PinHeader_2.54mm:PinHeader_1x04_P2.54mm_Vertical -> Connector_PinHeader_2.54mm:PinHeader_1x04_P2.54mm_Horizontal
- moved J201 180.3 mm to (253.7, 82.5), turned to -90 degrees
- moved C205 161.1 mm to (246.2, 135.1), turned to -90 degrees
- moved C206 153.5 mm to (241.4, 136.0), turned to 90 degrees
- moved D202 149.8 mm to (205.1, 70.5), turned to -90 degrees
- moved D201 147.1 mm to (208.3, 70.5), turned to -90 degrees
- moved D204 145.9 mm to (243.0, 135.4), turned to -90 degrees
- moved TP202 144.9 mm to (242.6, 142.1)
- moved R204 140.7 mm to (205.1, 73.5), turned to 90 degrees
- moved C201 132.6 mm to (219.8, 129.1), turned to 90 degrees
- moved FB202 131.4 mm to (244.8, 135.4), turned to -90 degrees
- moved RN601 129.9 mm to (245.4, 102.6)
- moved U201 127.2 mm to (214.8, 131.8), turned to 180 degrees
- moved C307 127.0 mm to (200.1, 69.8), turned to -90 degrees
- moved TP201 125.9 mm to (228.0, 142.1)
- moved C204 125.7 mm to (181.3, 77.5), turned to 90 degrees
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- renumbered J705 to J701
Connections:
- net /GPIO Expansion/IO.LEFT0 renamed IO.LEFT0
- net /GPIO Expansion/IO.LEFT1 renamed IO.LEFT1
- net /GPIO Expansion/IO.LEFT2 renamed IO.LEFT2
- net /GPIO Expansion/IO.LEFT3 renamed IO.LEFT3
- net /GPIO Expansion/IO.LEFT4 renamed IO.LEFT4
- net /GPIO Expansion/IO.LEFT5 renamed IO.LEFT5
- net /GPIO Expansion/IO.LEFT6 renamed IO.LEFT6
- net /GPIO Expansion/IO.LEFT7 renamed IO.LEFT7
- net /GPIO Expansion/IO.RIGHT0 renamed IO.RIGHT0
- net /GPIO Expansion/IO.RIGHT1 renamed IO.RIGHT1
- net /GPIO Expansion/IO.RIGHT2 renamed IO.RIGHT2
- net /GPIO Expansion/IO.RIGHT3 renamed IO.RIGHT3
- net /GPIO Expansion/IO.RIGHT4 renamed IO.RIGHT4
- net /GPIO Expansion/IO.RIGHT5 renamed IO.RIGHT5
- net /GPIO Expansion/IO.RIGHT6 renamed IO.RIGHT6
- net /GPIO Expansion/IO.RIGHT7 renamed IO.RIGHT7
- net /GPIO Expansion/IO.SS4_0 renamed IO.SS4_0
- net /GPIO Expansion/IO.SS4_1 renamed IO.SS4_1
- net /GPIO Expansion/IO.SS4_2 renamed IO.SS4_2
- net /GPIO Expansion/IO.SS4_3 renamed IO.SS4_3
- net /GPIO Expansion/IO.SS4_4 renamed IO.SS4_4
- net /GPIO Expansion/IO.SS4_5 renamed IO.SS4_5
- net /GPIO Expansion/IO.SS4_6 renamed IO.SS4_6
- net /GPIO Expansion/IO.SS4_7 renamed IO.SS4_7
- net /GPIO Expansion/IO.SS5_0 renamed IO.SS5_0
- net /GPIO Expansion/IO.SS5_1 renamed IO.SS5_1
- net /GPIO Expansion/IO.SS5_2 renamed IO.SS5_2
- net /GPIO Expansion/IO.SS5_3 renamed IO.SS5_3
- net /GPIO Expansion/IO.SS5_4 renamed IO.SS5_4
- net /GPIO Expansion/IO.SS5_5 renamed IO.SS5_5
- net /GPIO Expansion/IO.SS5_6 renamed IO.SS5_6
- net /GPIO Expansion/IO.SS5_7 renamed IO.SS5_7
- net /GPIO Expansion/IO.SS7_0 renamed IO.SS7_0
- net /GPIO Expansion/IO.SS7_1 renamed IO.SS7_1
- net /GPIO Expansion/IO.SS7_2 renamed IO.SS7_2
- net /GPIO Expansion/IO.SS7_3 renamed IO.SS7_3
- net /GPIO Expansion/IO.SS7_4 renamed IO.SS7_4
- net /GPIO Expansion/IO.SS7_5 renamed IO.SS7_5
- net /GPIO Expansion/IO.SS7_6 renamed IO.SS7_6
- net /GPIO Expansion/IO.SS7_7 renamed IO.SS7_7
- C709 pad 1: VPHY -> VPHY2
- C710 pad 1: VPHY -> VPHY2
- C711 pad 1: VPLL -> VPLL2
- C712 pad 1: VPLL -> VPLL2
- FB701 pad 2: VPHY -> VPHY2
- FB702 pad 2: VPLL -> VPLL2
- J201 pad 2: +3V3 -> +5V
- J201 pad 3: +5V -> +3V3
- R704 pad 2: EECLK -> EECLK2
- R705 pad 2: EECS -> EECS2
- R708 pad 2: EEDATA -> EEDATA2
- TP201 pad 1: +5V -> +3V3
- TP202 pad 1: +3V3 -> +5V
- U301 pad 19: unconnected-(U301-Pad19) -> INTA.MCP6
- U301 pad 21: unconnected-(U301-Pad21) -> INTB.MCP6
- U301 pad 22: unconnected-(U301-Pad22) -> INTB.MCP3
- U301 pad 23: unconnected-(U301-Pad23) -> INTA.MCP3
- U301 pad 24: unconnected-(U301-Pad24) -> INTA.MCP4
- U301 pad 26: unconnected-(U301-Pad26) -> INTB.MCP4
- U301 pad 27: unconnected-(U301-Pad27) -> INTA.MCP1
- U301 pad 28: unconnected-(U301-Pad28) -> INTA.MCP0
- U301 pad 29: unconnected-(U301-Pad29) -> INTB.MCP0
- U301 pad 30: unconnected-(U301-Pad30) -> INTA.MCP2
- U301 pad 32: unconnected-(U301-Pad32) -> INTB.MCP2
- U301 pad 53: unconnected-(U301-Pad53) -> MCP5.SEL
- U301 pad 54: unconnected-(U301-Pad54) -> INTA.MCP5
- U301 pad 55: unconnected-(U301-Pad55) -> INTB.MCP5
- U301 pad 57: unconnected-(U301-Pad57) -> INTB.MCP7
- U301 pad 58: unconnected-(U301-Pad58) -> INTA.MCP7
- U301 pad 59: unconnected-(U301-Pad59) -> MCP6.SEL
- U601 pad 11: INTA.MCP5 -> INTB.MCP6
- U601 pad 13: INTB.MCP5 -> unconnected-(U601-Pad13)
- U601 pad 15: INTB.MCP6 -> INTB.MCP7
- U601 pad 18: INTB.MCP7 -> unconnected-(U601-Pad18)
- U601 pad 21: unconnected-(U601-Pad21) -> INTB.MCP5
- U601 pad 22: MCP5.SEL -> INTA.MCP5
- U601 pad 24: MCP6.SEL -> MCP5.SEL
- U601 pad 26: unconnected-(U601-Pad26) -> INTB.MCP2
- U601 pad 29: INTA.MCP0 -> INTA.MCP2
- U601 pad 31: INTB.MCP0 -> INTA.MCP0
- U601 pad 32: INTA.MCP1 -> INTB.MCP0
- U601 pad 33: INTA.MCP2 -> INTA.MCP1
- U601 pad 35: INTA.MCP3 -> INTA.MCP4
- U601 pad 36: INTB.MCP2 -> INTB.MCP4
- U601 pad 37: INTB.MCP4 -> INTB.MCP3
- U601 pad 38: INTB.MCP3 -> INTA.MCP3
- U601 pad 40: INTA.MCP4 -> MCP6.SEL
- U701 pad 4: VPHY -> VPHY2
- U701 pad 61: EEDATA -> EEDATA2
- U701 pad 62: EECLK -> EECLK2
- U701 pad 63: EECS -> EECS2
- U701 pad 9: VPLL -> VPLL2
- U702 pad 3: EEDATA -> EEDATA2
- U702 pad 4: EECLK -> EECLK2
- U702 pad 5: EECS -> EECS2
Routing:
- net +3V3: track 79.4 -> 513.6 mm, vias 2 -> 22
- net +5V: track 0.00 -> 203.0 mm, vias 0 -> 6
- net IO.SDA0: track 26.7 -> 197.5 mm, vias 4 -> 6
- net GND: track 0.97 -> 165.5 mm, vias 1 -> 32
- net IO.SCK0: track 28.4 -> 185.3 mm, vias 4 -> 6
- net IO.SDA1: track 113.8 -> 259.4 mm
- net IO.SCK1: track 113.1 -> 244.5 mm
- net INTA.MCP1: track 2.03 -> 133.2 mm, vias 0 -> 2
- net MCP6.SEL: track 0.00 -> 129.5 mm, vias 0 -> 5
- net INTA.MCP0: track 2.01 -> 125.2 mm, vias 0 -> 2
- net INTB.MCP3: track 1.98 -> 123.1 mm, vias 0 -> 5
- net INTB.MCP0: track 1.99 -> 121.6 mm, vias 0 -> 2
- net INTA.MCP3: track 2.00 -> 118.5 mm, vias 0 -> 5
- net INTB.MCP6: track 2.11 -> 113.8 mm, vias 0 -> 4
- net INTA.MCP6: track 2.14 -> 110.8 mm, vias 0 -> 4
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Other:
- outline, holes or cut-outs redrawn
