File: ECELab_v1.kicad_pcb (KiCad board)
At the start: 2 copper layers, 121 parts, among them J201 USB_C_Receptacle_USB2.0, J202 Conn_01x02_Male, J301 Conn_01x04_Male, J302 Conn_01x03_Male, J501 Conn_01x12_Male, SW301 SW_SPDT, U201 AZ1117IH-3.3TRG1, U301 SN74LVC257AD, U302 FT232HL, U303 93LC56BT-I/OT, U401 MCP23S17_SS, U402 MCP23S17_SS, U403 MCP23S17_SS, U404 MCP23S17_SS, U405 MCP23S17_SS, U406 MCP23S17_SS, U407 MCP23S17_SS, U408 MCP23S17_SS, U501 ICE40-HX8K_Breakout_Board, Y301 12MHz

Commit message: update
Parts:
- added R301: 10k, Resistor_SMD:R_0402_1005Metric, F.Cu at (160.2, 60.0)
- added R302: 10k, Resistor_SMD:R_0402_1005Metric, F.Cu at (160.2, 58.0)
- J301: value Conn_01x04_Male -> Conn_01x02_Male; footprint Connector_PinHeader_2.54mm:PinHeader_1x04_P2.54mm_Vertical -> Connector_PinHeader_2.54mm:PinHeader_1x02_P2.54mm_Vertical
- U401, U402, U403, U404, U405, U406, U407, U408: value MCP23S17_SS -> MCP23017_SS
- moved U501 38.4 mm to (145.4, 113.2)
- moved U408 31.8 mm to (20.6, 122.5)
- moved J301 30.2 mm to (156.4, 59.3)
- moved U405 28.1 mm to (41.7, 110.5)
- moved U407 21.3 mm to (20.6, 110.5)
- moved U401 17.5 mm to (52.2, 122.5)
- moved U402 14.0 mm to (31.1, 110.5)
- moved U406 10.1 mm to (31.1, 122.5)
- moved U404 1.96 mm to (52.2, 110.5)
- moved U403 1.96 mm to (41.7, 122.5)
- renumbered R301 to R303, R302 to R304, R303 to R305, R304 to R306
Connections:
- net CONN.SDI renamed CONN.SDA
- net FTDI.SDI renamed FTDI.SDA
- net IO.SDI renamed IO.SDA
- U301 pad 10: CONN.SDO -> unconnected-(U301-Pad10)
- U301 pad 11: FTDI.SDO -> unconnected-(U301-Pad11)
- U301 pad 12: IO.~{CS} -> unconnected-(U301-Pad12)
- U301 pad 13: CONN.~{CS} -> unconnected-(U301-Pad13)
- U301 pad 14: FTDI.~{CS} -> unconnected-(U301-Pad14)
- U301 pad 9: IO.SDO -> unconnected-(U301-Pad9)
- U302 pad 15: FTDI.SDO -> unconnected-(U302-Pad15)
- U302 pad 16: FTDI.~{CS} -> unconnected-(U302-Pad16)
- U401 pad 11: IO.~{CS} -> unconnected-(U401-Pad11)
- U401 pad 14: IO.SDO -> unconnected-(U401-Pad14)
- U402 pad 11: IO.~{CS} -> unconnected-(U402-Pad11)
- U402 pad 14: IO.SDO -> unconnected-(U402-Pad14)
- U403 pad 11: IO.~{CS} -> unconnected-(U403-Pad11)
- U403 pad 14: IO.SDO -> unconnected-(U403-Pad14)
- U404 pad 11: IO.~{CS} -> unconnected-(U404-Pad11)
- U404 pad 14: IO.SDO -> unconnected-(U404-Pad14)
- U405 pad 11: IO.~{CS} -> unconnected-(U405-Pad11)
- U405 pad 14: IO.SDO -> unconnected-(U405-Pad14)
- U406 pad 11: IO.~{CS} -> unconnected-(U406-Pad11)
- U406 pad 14: IO.SDO -> unconnected-(U406-Pad14)
- U407 pad 11: IO.~{CS} -> unconnected-(U407-Pad11)
- U407 pad 14: IO.SDO -> unconnected-(U407-Pad14)
- U408 pad 11: IO.~{CS} -> unconnected-(U408-Pad11)
- U408 pad 14: IO.SDO -> unconnected-(U408-Pad14)

Commit message: Complete Draft 1 of PCB Design
Parts:
- removed J501: Conn_01x12_Male, Connector_PinHeader_2.54mm:PinHeader_1x12_P2.54mm_Vertical
- removed the R305 at (146.0, 54.1)
- removed SW301: SW_SPDT, Button_Switch_SMD:SW_SPDT_PCM12
- added ?: , , F.Cu at (165.0, 66.8)
- added ?: , , F.Cu at (108.7, 148.1)
- added ?: , , F.Cu at (165.0, 148.1)
- added ?: , , F.Cu at (247.4, 148.1)
- added ?: , , F.Cu at (108.7, 66.8)
- added C209: 0.1u, Capacitor_SMD:C_0402_1005Metric, F.Cu at (154.6, 143.7)
- added C210: 0.1u, Capacitor_SMD:C_0402_1005Metric, F.Cu at (160.9, 144.3)
- added C401: 0.1u, Capacitor_SMD:C_0402_1005Metric, B.Cu at (196.7, 119.7)
- added C402: 0.1u, Capacitor_SMD:C_0402_1005Metric, B.Cu at (221.2, 97.6)
- added C403: 0.1u, Capacitor_SMD:C_0402_1005Metric, B.Cu at (219.9, 121.6)
- added C404: 0.1u, Capacitor_SMD:C_0402_1005Metric, B.Cu at (219.9, 144.4)
- added C405: 0.1u, Capacitor_SMD:C_0402_1005Metric, B.Cu at (195.0, 75.5)
- added C406: 0.1u, Capacitor_SMD:C_0402_1005Metric, B.Cu at (217.9, 75.2)
- added C407: 0.1u, Capacitor_SMD:C_0402_1005Metric, B.Cu at (197.0, 143.2)
- added C408: 0.1u, Capacitor_SMD:C_0402_1005Metric, B.Cu at (196.6, 96.9)
- added C601: 0.1u, Capacitor_SMD:C_0402_1005Metric, F.Cu at (162.5, 138.3)
- added C602: 0.1u, Capacitor_SMD:C_0402_1005Metric, F.Cu at (162.5, 140.8)
- added D208: PMEG40, Diode_SMD:D_SOD-323, F.Cu at (156.8, 144.3)
- added FB204: 120R, Inductor_SMD:L_0603_1608Metric, F.Cu at (159.1, 144.6)
- added G***: LOGO, ECELab_Footprints:purduelogo, F.Cu at (140.0, 81.8)
- added G***: LOGO, ECELab_Footprints:purduelogo, B.Cu at (139.5, 81.8)
- added J203: Conn_01x06_Male, Connector_PinHeader_2.54mm:PinHeader_1x06_P2.54mm_Horizontal, F.Cu at (115.7, 103.2)
- added J302: Conn_01x03_Male, Connector_PinHeader_2.54mm:PinHeader_1x03_P2.54mm_Horizontal, F.Cu at (132.9, 140.9)
- added REF**: MountingHole_2.7mm_Pad, MountingHole:MountingHole_2.7mm_Pad, F.Cu at (247.4, 66.8)
- added TP201: TestPoint, TestPoint:TestPoint_Plated_Hole_D4.0mm, F.Cu at (117.1, 67.3)
- added TP202: TestPoint, TestPoint:TestPoint_Plated_Hole_D4.0mm, F.Cu at (126.5, 67.3)
- added TP203: TestPoint, TestPoint:TestPoint_Plated_Hole_D4.0mm, F.Cu at (135.8, 67.3)
- added U601: RASPBERRY_PI_4B_4GB, ECELab_Footprints:MODULE_RASPBERRY_PI_4B_4GB, F.Cu at (134.3, 107.5)
- C301, C302, C303, C305, R303, U303: moved to B.Cu
- J202: footprint Connector_PinHeader_2.00mm:PinHeader_1x02_P2.00mm_Vertical -> Connector_PinHeader_2.54mm:PinHeader_1x02_P2.54mm_Horizontal
- J301: value Conn_01x02_Male -> Conn_01x04_Male; footprint Connector_PinHeader_2.54mm:PinHeader_1x02_P2.54mm_Vertical -> Connector_PinHeader_2.54mm:PinHeader_1x04_P2.54mm_Horizontal
- R305: renamed from R306; moved to B.Cu
- moved U407 201.2 mm to (218.4, 73.7), turned to 90 degrees
- moved U402 187.8 mm to (218.4, 96.5), turned to 90 degrees
- moved U403 177.8 mm to (218.4, 142.2), turned to 90 degrees
- moved U408 176.1 mm to (195.6, 142.2), turned to 90 degrees
- moved R408 175.5 mm to (221.3, 89.6), turned to 90 degrees
- moved JP419 174.5 mm to (210.8, 73.7)
- moved U406 171.5 mm to (195.6, 73.7), turned to 90 degrees
- moved R402 168.1 mm to (219.9, 89.6), turned to -90 degrees
- moved R410 166.9 mm to (224.3, 89.6), turned to 90 degrees
- moved U404 166.4 mm to (218.4, 119.4), turned to 90 degrees
- moved JP406 166.3 mm to (210.8, 96.5)
- moved R427 165.9 mm to (221.0, 66.8), turned to 90 degrees
- moved R409 165.5 mm to (222.8, 89.6), turned to 90 degrees
- moved R411 164.2 mm to (221.4, 135.4), turned to 90 degrees
- moved JP422 163.5 mm to (203.2, 77.5), turned to 180 degrees
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- renumbered J302 to J303
Connections:
- net IO44 renamed IO.SS2_4
- J301 pad 1: CONN.SCK -> CONN.SDA
- J301 pad 2: CONN.SDA -> CONN.SCK
- U401 pad 1: IO0 -> IO.HWCLK
- U401 pad 2: IO1 -> IO.PB20
- U401 pad 21: IO8 -> IO.PB13
- U401 pad 22: IO9 -> IO.PB12
- U401 pad 23: IO10 -> IO.PB11
- U401 pad 24: IO11 -> IO.PB10
- U401 pad 25: IO12 -> IO.PB9
- U401 pad 26: IO13 -> IO.PB8
- U401 pad 27: IO14 -> unconnected-(U401-Pad27)
- U401 pad 28: IO15 -> unconnected-(U401-Pad28)
- U401 pad 3: IO2 -> IO.PB19
- U401 pad 4: IO3 -> IO.PB18
- U401 pad 5: IO4 -> IO.PB17
- U401 pad 6: IO5 -> IO.PB16
- U401 pad 7: IO6 -> IO.PB15
- U401 pad 8: IO7 -> IO.PB14
- U402 pad 1: IO16 -> IO.PB7
- U402 pad 2: IO17 -> IO.PB6
- U402 pad 21: IO24 -> IO.SS0_0
- U402 pad 22: IO25 -> IO.SS0_1
- U402 pad 23: IO26 -> IO.SS0_2
- U402 pad 24: IO27 -> IO.SS0_3
- U402 pad 25: IO28 -> IO.SS0_4
- U402 pad 26: IO29 -> IO.SS0_5
- U402 pad 27: IO30 -> IO.SS0_6
- U402 pad 28: IO31 -> IO.SS0_7
- U402 pad 3: IO18 -> IO.PB5
- U402 pad 4: IO19 -> IO.PB4
- U402 pad 5: IO20 -> IO.PB3
- U402 pad 6: IO21 -> IO.PB2
- U402 pad 7: IO22 -> IO.PB1
- U402 pad 8: IO23 -> IO.PB0
- U403 pad 1: IO32 -> IO.SS1_0
- U403 pad 2: IO33 -> IO.SS1_1
- U403 pad 21: IO40 -> IO.SS2_0
- U403 pad 22: IO41 -> IO.SS2_1
- U403 pad 23: IO42 -> IO.SS2_2
- U403 pad 24: IO43 -> IO.SS2_3
- U403 pad 26: IO45 -> IO.SS2_5
- U403 pad 27: IO46 -> IO.SS2_6
- U403 pad 28: IO47 -> IO.SS2_7
- U403 pad 3: IO34 -> IO.SS1_2
- U403 pad 4: IO35 -> IO.SS1_3
- U403 pad 5: IO36 -> IO.SS1_4
- U403 pad 6: IO37 -> IO.SS1_5
- U403 pad 7: IO38 -> IO.SS1_6
- U403 pad 8: IO39 -> IO.SS1_7
- U404 pad 1: IO48 -> IO.SS3_0
- U404 pad 2: IO49 -> IO.SS3_1
- U404 pad 21: IO56 -> IO.SS4_0
- U404 pad 22: IO57 -> IO.SS4_1
- U404 pad 23: IO58 -> IO.SS4_2
- U404 pad 24: IO59 -> IO.SS4_3
- U404 pad 25: IO60 -> IO.SS4_4
- U404 pad 26: IO61 -> IO.SS4_5
- U404 pad 27: IO62 -> IO.SS4_6
- U404 pad 28: IO63 -> IO.SS4_7
- U404 pad 3: IO50 -> IO.SS3_2
- U404 pad 4: IO51 -> IO.SS3_3
- U404 pad 5: IO52 -> IO.SS3_4
- U404 pad 6: IO53 -> IO.SS3_5
- U404 pad 7: IO54 -> IO.SS3_6
- U404 pad 8: IO55 -> IO.SS3_7
- U405 pad 1: IO64 -> IO.SS5_0
- U405 pad 2: IO65 -> IO.SS5_1
- U405 pad 21: IO72 -> IO.SS6_0
- U405 pad 22: IO73 -> IO.SS6_1
- U405 pad 23: IO74 -> IO.SS6_2
- U405 pad 24: IO75 -> IO.SS6_3
- U405 pad 25: IO76 -> IO.SS6_4
- U405 pad 26: IO77 -> IO.SS6_5
- U405 pad 27: IO78 -> IO.SS6_6
- U405 pad 28: IO79 -> IO.SS6_7
- U405 pad 3: IO66 -> IO.SS5_2
- U405 pad 4: IO67 -> IO.SS5_3
- U405 pad 5: IO68 -> IO.SS5_4
- U405 pad 6: IO69 -> IO.SS5_5
- U405 pad 7: IO70 -> IO.SS5_6
- U405 pad 8: IO71 -> IO.SS5_7
- U406 pad 1: IO80 -> IO.SS7_0
- U406 pad 2: IO81 -> IO.SS7_1
- U406 pad 21: IO88 -> IO.LEFT7
- U406 pad 22: IO89 -> IO.LEFT6
- U406 pad 23: IO90 -> IO.LEFT5
- U406 pad 24: IO91 -> IO.LEFT4
- U406 pad 25: IO92 -> IO.LEFT3
- U406 pad 26: IO93 -> IO.LEFT2
- U406 pad 27: IO94 -> IO.LEFT1
- U406 pad 28: IO95 -> IO.LEFT0
- U406 pad 3: IO82 -> IO.SS7_2
- U406 pad 4: IO83 -> IO.SS7_3
- U406 pad 5: IO84 -> IO.SS7_4
- U406 pad 6: IO85 -> IO.SS7_5
- U406 pad 7: IO86 -> IO.SS7_6
- U406 pad 8: IO87 -> IO.SS7_7
- U407 pad 1: IO96 -> IO.RIGHT7
- U407 pad 2: IO97 -> IO.RIGHT6
- U407 pad 21: IO104 -> IO.RED
- U407 pad 22: IO105 -> IO.GREEN
- U407 pad 23: IO106 -> IO.BLUE
- U407 pad 24: IO107 -> unconnected-(U407-Pad24)
- U407 pad 25: IO108 -> unconnected-(U407-Pad25)
- U407 pad 26: IO109 -> unconnected-(U407-Pad26)
- U407 pad 27: IO110 -> unconnected-(U407-Pad27)
- U407 pad 28: IO111 -> unconnected-(U407-Pad28)
- U407 pad 3: IO98 -> IO.RIGHT5
- U407 pad 4: IO99 -> IO.RIGHT4
- U407 pad 5: IO100 -> IO.RIGHT3
- U407 pad 6: IO101 -> IO.RIGHT2
- U407 pad 7: IO102 -> IO.RIGHT1
- U407 pad 8: IO103 -> IO.RIGHT0
- U408 pad 1: IO112 -> IO.Rx
- U408 pad 2: IO113 -> IO.Tx
- U408 pad 21: IO120 -> unconnected-(U408-Pad21)
- U408 pad 22: IO121 -> unconnected-(U408-Pad22)
- U408 pad 23: IO122 -> unconnected-(U408-Pad23)
- U408 pad 24: IO123 -> unconnected-(U408-Pad24)
- U408 pad 25: IO124 -> unconnected-(U408-Pad25)
- U408 pad 26: IO125 -> unconnected-(U408-Pad26)
- U408 pad 27: IO126 -> unconnected-(U408-Pad27)
- U408 pad 28: IO127 -> unconnected-(U408-Pad28)
- U408 pad 3: IO114 -> IO.DSRn
- U408 pad 4: IO115 -> IO.RTSn
- U408 pad 5: IO116 -> IO.DCDn
- U408 pad 6: IO117 -> IO.CTSn
- U408 pad 7: IO118 -> IO.DTRn
- U408 pad 8: IO119 -> unconnected-(U408-Pad8)
- U501 pad 100: IO81 -> IO.PB13
- U501 pad 101: IO65 -> IO.PB14
- U501 pad 102: IO80 -> IO.PB15
- U501 pad 103: IO66 -> IO.PB16
- U501 pad 104: IO79 -> IO.PB17
- U501 pad 107: IO67 -> IO.PB18
- U501 pad 108: IO78 -> IO.PB19
- U501 pad 109: IO68 -> IO.Rx
- U501 pad 11: IO3 -> IO.SS0_6
- U501 pad 110: IO77 -> IO.PB20
- U501 pad 111: IO69 -> IO.SS5_7
- U501 pad 112: IO76 -> IO.Tx
- U501 pad 115: IO70 -> IO.DSRn
- U501 pad 116: IO75 -> IO.RTSn
- U501 pad 117: IO71 -> IO.DCDn
- U501 pad 118: IO74 -> IO.CTSn
- U501 pad 119: IO72 -> unconnected-(U501-Pad119)
- U501 pad 12: IO24 -> IO.SS0_5
- U501 pad 120: IO73 -> IO.DTRn
- U501 pad 123: IO88 -> IO.SS7_3
- U501 pad 124: IO115 -> IO.LEFT7
- U501 pad 125: IO89 -> IO.SS7_5
- U501 pad 126: IO114 -> IO.SS7_4
- U501 pad 127: IO90 -> IO.LEFT6
- U501 pad 128: IO113 -> IO.SS7_6
- U501 pad 13: IO4 -> IO.SS0_4
- U501 pad 131: IO91 -> IO.SS7_1
- U501 pad 132: IO112 -> IO.SS7_0
- U501 pad 133: IO92 -> IO.SS7_7
- U501 pad 134: IO111 -> IO.SS7_2
- U501 pad 135: IO93 -> IO.SS6_3
- U501 pad 136: IO110 -> IO.LEFT5
- U501 pad 139: IO94 -> IO.SS6_5
- U501 pad 14: IO23 -> IO.SS0_3
- U501 pad 140: IO109 -> IO.SS6_4
- U501 pad 141: IO95 -> IO.LEFT4
- U501 pad 142: IO108 -> IO.SS6_6
- U501 pad 143: IO96 -> IO.SS6_1
- U501 pad 144: IO107 -> IO.SS6_0
- U501 pad 147: IO97 -> IO.SS6_7
- U501 pad 148: IO106 -> IO.SS6_2
- U501 pad 149: IO98 -> IO.SS5_3
- U501 pad 15: IO5 -> IO.RIGHT2
- U501 pad 150: IO105 -> IO.LEFT3
- U501 pad 151: IO99 -> IO.SS5_5
- U501 pad 152: IO104 -> IO.SS5_4
- U501 pad 155: IO100 -> IO.LEFT2
- U501 pad 156: IO103 -> IO.SS5_6
- U501 pad 157: IO101 -> IO.SS5_0
- U501 pad 159: IO102 -> unconnected-(U501-Pad159)
- U501 pad 16: IO22 -> IO.SS1_7
- U501 pad 19: IO6 -> IO.HWCLK
- U501 pad 20: IO21 -> IO.SS1_2
- U501 pad 21: IO7 -> IO.SS1_1
- U501 pad 22: IO20 -> IO.SS1_0
- U501 pad 23: IO8 -> IO.RIGHT3
- U501 pad 24: IO19 -> IO.SS1_6
- U501 pad 27: IO9 -> IO.SS1_5
- U501 pad 28: IO18 -> IO.SS1_4
- U501 pad 29: IO10 -> IO.SS1_3
- U501 pad 3: IO0 -> IO.RIGHT0
- U501 pad 30: IO17 -> IO.RIGHT4
- U501 pad 31: IO11 -> IO.SS2_7
- U501 pad 32: IO16 -> IO.SS2_2
- U501 pad 35: IO12 -> IO.SS2_1
- U501 pad 36: IO15 -> IO.SS2_0
- U501 pad 37: IO13 -> IO.RIGHT5
- U501 pad 39: IO14 -> unconnected-(U501-Pad39)
- U501 pad 4: IO27 -> IO.SS0_7
- U501 pad 43: IO28 -> IO.SS5_2
- U501 pad 44: IO57 -> IO.SS5_1
- U501 pad 45: IO29 -> IO.SS4_3
- U501 pad 46: IO56 -> IO.LEFT1
- U501 pad 47: IO30 -> IO.SS4_5
- U501 pad 48: IO55 -> IO.SS4_4
- U501 pad 5: IO1 -> IO.SS0_2
- U501 pad 51: IO31 -> IO.LEFT0
- U501 pad 52: IO54 -> IO.SS4_6
- U501 pad 53: IO32 -> IO.SS4_1
- U501 pad 54: IO53 -> IO.SS4_0
- U501 pad 55: IO33 -> IO.SS4_7
- U501 pad 56: IO52 -> IO.SS4_2
- U501 pad 59: IO34 -> IO.BLUE
- U501 pad 6: IO26 -> IO.SS0_1
- U501 pad 60: IO51 -> IO.GREEN
- U501 pad 61: IO35 -> IO.SS3_3
- U501 pad 62: IO50 -> IO.RED
- U501 pad 63: IO36 -> IO.SS3_5
- U501 pad 64: IO49 -> IO.SS3_4
- U501 pad 67: IO37 -> IO.RIGHT7
- U501 pad 68: IO48 -> IO.SS3_6
- U501 pad 69: IO38 -> IO.SS3_1
- U501 pad 7: IO2 -> IO.SS0_0
- U501 pad 70: IO47 -> IO.SS3_0
- U501 pad 71: IO39 -> IO.SS3_7
- U501 pad 72: IO46 -> IO.SS3_2
- U501 pad 75: IO40 -> IO.SS2_3
- U501 pad 76: IO45 -> IO.RIGHT6
- U501 pad 77: IO41 -> IO.SS2_5
- U501 pad 79: IO42 -> unconnected-(U501-Pad79)
- U501 pad 8: IO25 -> IO.RIGHT1
- U501 pad 80: IO43 -> IO.SS2_6
- U501 pad 83: IO58 -> IO.PB4
- U501 pad 84: IO87 -> IO.PB5
- U501 pad 85: IO59 -> IO.PB1
- U501 pad 86: IO86 -> IO.PB6
- U501 pad 87: IO60 -> IO.PB0
- U501 pad 88: IO85 -> IO.PB7
- U501 pad 91: IO61 -> IO.PB2
- U501 pad 92: IO84 -> IO.PB8
- U501 pad 93: IO62 -> IO.PB3
- U501 pad 94: IO83 -> IO.PB9
- U501 pad 95: IO63 -> IO.PB10
- U501 pad 96: IO82 -> IO.PB11
- U501 pad 99: IO64 -> IO.PB12
Routing:
- net +3V3: track 0.00 -> 658.7 mm, vias 0 -> 32
- net IO.SCK: track 0.00 -> 267.0 mm, vias 0 -> 8
- net IO.SDA: track 0.00 -> 265.3 mm, vias 0 -> 9
- net +5V: track 0.00 -> 152.0 mm, vias 0 -> 2
- net GND: track 0.00 -> 115.4 mm, vias 0 -> 195
- net IO.LEFT2: track 0.00 -> 84.1 mm, vias 0 -> 1
- net IO.RIGHT5: track 0.00 -> 77.8 mm
- net IO.RIGHT6: track 0.00 -> 77.7 mm
- net IO.SS1_7: track 0.00 -> 74.4 mm
- net IO.SS0_3: track 0.00 -> 73.8 mm, vias 0 -> 2
- net IO.LEFT3: track 0.00 -> 73.4 mm, vias 0 -> 1
- net IO.SS1_2: track 0.00 -> 71.1 mm, vias 0 -> 1
- net IO.SS0_4: track 0.00 -> 70.2 mm, vias 0 -> 2
- net IO.LEFT0: track 0.00 -> 70.1 mm, vias 0 -> 1
- net IO.PB7: track 0.00 -> 69.1 mm, vias 0 -> 1
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- added copper zone on F.Cu, net +3V3
- added copper zone on B.Cu, net GND
- added copper zone on F.Cu, net GND
Other:
- board outline added: 147.5 x 89.3 mm
- board text added: "0 0 0"
- board text added: "0 0 1"
- board text added: "0 1 0"
- board text added: "0 1 1"
- board text added: "1 0 0"
- board text added: "1 0 1"
- board text added: "1 1 0"
- board text added: "1 1 1"
- board text added: "3V3"
- board text added: "3V3 PWR"
- board text added: "5V"
- board text added: "5V PWR"
- board text added: "C.SCK"
- board text added: "C.SDA"
- board text added: "CONN / GND"
- board text added: "ECELab PCB Design v1 Minh Nguyen Junfei Li"
- board text added: "EXT_5V"
- board text added: "FTDI / 3V3"
- board text added: "GND"
- board text added: "IOExp 0 [0 0 0]"
- board text added: "IOExp 1 [0 0 1]"
- board text added: "IOExp 2 [0 1 0]"
- board text added: "IOExp 3 [0 1 1]"
- board text added: "IOExp 4 [1 0 0]"
- board text added: "IOExp 5 [1 0 1]"
- board text added: "IOExp 6 [1 1 0]"
- board text added: "IOExp 7 [1 1 1]"
- board text added: "OUTPUT"
- board text added: "Raspberry Pi 4"
- board text added: "SEL"

Commit message: Draft 1 complete
Parts:
- removed ? (x5): , 
- removed REF**: MountingHole_2.7mm_Pad, MountingHole:MountingHole_2.7mm_Pad
- removed the U301 at (142.0, 133.5)
- added TP204: TestPoint, TestPoint:TestPoint_Plated_Hole_D4.0mm, F.Cu at (108.0, 84.3)
- added TP205: TestPoint, TestPoint:TestPoint_Plated_Hole_D4.0mm, F.Cu at (108.0, 77.0)
- C301, C302, C303, C305, C401, C402, C403, C404, C405, C406, C407, C408, R303, R305: moved to F.Cu
- J302: footprint Connector_PinHeader_2.54mm:PinHeader_1x03_P2.54mm_Horizontal -> Connector_PinHeader_2.54mm:PinHeader_1x03_P2.54mm_Vertical
- R201: value 250 -> 220
- U301: renamed from U302; value FT232HL -> FT232HQ-REEL; footprint Package_QFP:LQFP-48_7x7mm_P0.5mm -> Package_DFN_QFN:QFN-48-1EP_8x8mm_P0.5mm_EP6.2x6.2mm
- U302: renamed from U303; moved to F.Cu
- moved J302 8.61 mm to (140.5, 136.8), turned to 180 degrees
- moved C301 8.54 mm to (142.3, 115.3), turned to 90 degrees
- moved C302 8.50 mm to (136.1, 126.2), turned to 0 degrees
- moved C408 6.97 mm to (200.9, 102.3)
- moved Y301 6.97 mm to (132.3, 110.8)
- moved C406 6.37 mm to (213.2, 79.5), turned to 90 degrees
- moved J303 6.27 mm to (135.6, 136.8), turned to 180 degrees
- moved C303 5.67 mm to (142.8, 126.3), turned to 180 degrees
- moved C401 5.10 mm to (196.1, 124.8), turned to 0 degrees
- moved C404 4.77 mm to (223.3, 147.7)
- moved C407 4.60 mm to (197.0, 147.8)
- moved C402 4.44 mm to (219.9, 101.8)
- moved C405 4.43 mm to (196.8, 79.5), turned to 90 degrees
- moved U302 4.08 mm to (143.3, 112.2), turned to 0 degrees
- moved C305 3.89 mm to (143.6, 115.3), turned to -90 degrees
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- renumbered J203 to J202, J202 to J203
Connections:
- J302 pad 1: +3V3 -> CONN.SDA
- J302 pad 2: MUX.SEL -> IO.SDA
- J302 pad 3: GND -> FTDI.SDA
- J303 pad 1: +3V3 -> CONN.SCK
- J303 pad 2: MUX.SEL -> IO.SCK
- J303 pad 3: GND -> FTDI.SCK
Routing:
- net GND: track 115.4 -> 180.9 mm, vias 195 -> 202
- net EXT5V_IN: track 5.87 -> 38.8 mm
- net MUX.SEL: track 19.8 -> 0.00 mm
- net EECS: track 2.70 -> 11.7 mm, vias 1 -> 2
- net +3V3: track 658.7 -> 667.4 mm, vias 32 -> 34
- net EECLK: track 2.93 -> 10.5 mm, vias 1 -> 2
- net FTDI.SDA: track 20.4 -> 13.2 mm, vias 2 -> 1
- net /FTDI/XCSI: track 16.0 -> 9.13 mm
- net CONN.SCK: track 35.7 -> 29.4 mm
- net IO.SDA: track 265.3 -> 270.5 mm
- net IO.SCK: track 267.0 -> 271.7 mm
- net CONN.SDA: track 39.0 -> 34.5 mm
- net /FTDI/XCSO: track 9.30 -> 13.7 mm
- net FTDI.SCK: track 17.1 -> 12.8 mm, vias 2 -> 1
- net FTDI.D+: track 29.3 -> 26.6 mm
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Other:
- board text added: "0"
- board text added: "1"
- board text added: "5V 3V3"
- board text added: "5V SDA"
- board text added: "A1 A2"
- board text added: "A7 A8"
- board text added: "B10 A11"
- board text added: "B11 B12"
- board text added: "B14 B13"
- board text added: "B15 A15"
- board text added: "B16 C16"
- board text added: "B2 B1"
- board text added: "B3 B4"
- board text added: "B9 A9"
- board text added: "C2 C1"
- board text added: "C3 B5"
- board text added: "C4 A5"
- board text added: "C5 B6"
- board text added: "C6 A6"
- board text added: "C7 B7"
- board text added: "C9 A10"
- board text added: "CONN I2C"
- board text added: "CONN.SCK"
- board text added: "CONN.SDA"
- board text added: "D14 D16"
- board text added: "D15 E16"
- board text added: "D2 D1"
- board text added: "E14 F16"
- board text added: "F1 E2"
- board text added: "F14 G14"
- board text added: "F15 G16"
- board text added: "FPGA USB [HERE]"
- board text added: "FTDI.SCK"
- board text added: "FTDI.SDA"
- board text added: "G1 F2"
- board text added: "G15 H16"
- board text added: "GND GND"
- board text added: "GND SCK"
- board text added: "GND X"
- board text added: "H1 G2"
- board text added: "H14 J15"
- board text added: "IO.SCK"
- board text added: "IO.SDA"
- board text added: "IO0 A16"
- board text added: "IO1 1.2"
- board text added: "IO2 R16"
- board text added: "IO3 3.3"
- board text added: "J1 J2"
- board text added: "J14 K14"
- board text added: "J3 H2"
- board text added: "K1 K3"
- board text added: "K16 K15"
- board text added: "L1 L3"
- board text added: "L16 M16"
- board text added: "M1 M2"
- board text added: "M11 N10"
- board text added: "M15 N16"
- board text added: "MODE"
- board text added: "N2 N3"
- board text added: "NOT INPUT"
- board text added: "P10 T11"
- board text added: "P13 N12"
- board text added: "P15 P16"
- board text added: "P2 P1"
- board text added: "P9 P8"
- board text added: "PWR INPUT"
- board text added: "R1 3.3"
- board text added: "R10 T10"
- board text added: "R15 1.2"
- board text added: "R4 R3"
- board text added: "R5 T5"
- board text added: "R6 T6"
- board text added: "R9 T9"
- board text added: "Sel CONN: CONN.SDA=IO.SDA CONN.SCK=IO.SCK"
- board text added: "Sel FTDI: FTDI.SDA=IO.SDA FTDI.SCK=IO.SCK"
- board text added: "T14 T13"
- board text added: "T16 T15"
- board text added: "T2 T1"
- board text added: "T3 R2"
- board text added: "T8 T7"
- board text added: "X 3V3"
- board text added: "X GND"
- board text removed: "0 0 0"
- board text removed: "0 0 1"
- board text removed: "0 1 0"
- board text removed: "0 1 1"
- board text removed: "1 0 0"
- board text removed: "1 0 1"
- board text removed: "1 1 0"
- board text removed: "1 1 1"
- board text removed: "3V3 PWR"
- board text removed: "5V PWR"
- board text removed: "CONN / GND"
- board text removed: "FTDI / 3V3"
- board text removed: "SEL"

Commit message: Update to v1.2
Parts:
- removed JP401, JP402, JP403, JP404, JP405, JP406, JP409, JP411, JP417, JP418, JP421, JP423: Jumper_2_Open, Jumper:SolderJumper-2_P1.3mm_Open_TrianglePad1.0x1.5mm
- removed JP407, JP408, JP410, JP412, JP413, JP414, JP415, JP416, JP419, JP420, JP422, JP424: Jumper_2_Bridged, Jumper:SolderJumper-2_P1.3mm_Bridged_Pad1.0x1.5mm
- removed R405, R406, R407, R408, R409, R410, R411, R412, R413, R414, R415, R416, R421, R422, R423, R424, R425, R426, R427, R428, R429, R430, R431, R432: 10k, Resistor_SMD:R_0402_1005Metric
- removed TP201, TP202, TP203, TP204, TP205: TestPoint, TestPoint:TestPoint_Plated_Hole_D4.0mm
- moved G*** 81.5 mm to (72.3, 131.2)
- moved G*** 81.5 mm to (73.1, 131.2)
- moved J302 71.3 mm to (78.8, 172.5)
- moved J303 71.3 mm to (74.0, 172.6)
- moved J202 42.3 mm to (74.5, 112.9)
- moved J203 38.2 mm to (78.7, 120.4)
- moved J301 37.9 mm to (81.9, 158.2)
- moved C203 17.3 mm to (116.4, 140.8)
- moved C205 17.3 mm to (119.6, 124.8)
- moved C301 17.3 mm to (142.5, 132.6)
- moved C303 17.3 mm to (143.0, 143.6)
- moved C304 17.3 mm to (145.1, 132.6)
- moved C305 17.3 mm to (143.8, 132.6)
- moved D201 17.3 mm to (121.0, 134.4)
- moved D202 17.3 mm to (128.4, 134.4)
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Connections:
- net IO.BLUE renamed /GPIO Expansion/IO.BLUE
- net IO.GREEN renamed /GPIO Expansion/IO.GREEN
- net IO.HWCLK renamed /GPIO Expansion/IO.HWCLK
- net IO.LEFT0 renamed /GPIO Expansion/IO.LEFT0
- net IO.LEFT1 renamed /GPIO Expansion/IO.LEFT1
- net IO.LEFT2 renamed /GPIO Expansion/IO.LEFT2
- net IO.LEFT3 renamed /GPIO Expansion/IO.LEFT3
- net IO.LEFT4 renamed /GPIO Expansion/IO.LEFT4
- net IO.LEFT5 renamed /GPIO Expansion/IO.LEFT5
- net IO.LEFT6 renamed /GPIO Expansion/IO.LEFT6
- net IO.LEFT7 renamed /GPIO Expansion/IO.LEFT7
- net IO.PB0 renamed /GPIO Expansion/IO.PB0
- net IO.PB1 renamed /GPIO Expansion/IO.PB1
- net IO.PB10 renamed /GPIO Expansion/IO.PB10
- net IO.PB11 renamed /GPIO Expansion/IO.PB11
- net IO.PB12 renamed /GPIO Expansion/IO.PB12
- net IO.PB13 renamed /GPIO Expansion/IO.PB13
- net IO.PB14 renamed /GPIO Expansion/IO.PB14
- net IO.PB15 renamed /GPIO Expansion/IO.PB15
- net IO.PB16 renamed /GPIO Expansion/IO.PB16
- net IO.PB17 renamed /GPIO Expansion/IO.PB17
- net IO.PB18 renamed /GPIO Expansion/IO.PB18
- net IO.PB19 renamed /GPIO Expansion/IO.PB19
- net IO.PB2 renamed /GPIO Expansion/IO.PB2
- net IO.PB20 renamed /GPIO Expansion/IO.PB20
- net IO.PB3 renamed /GPIO Expansion/IO.PB3
- net IO.PB4 renamed /GPIO Expansion/IO.PB4
- net IO.PB5 renamed /GPIO Expansion/IO.PB5
- net IO.PB6 renamed /GPIO Expansion/IO.PB6
- net IO.PB7 renamed /GPIO Expansion/IO.PB7
- net IO.PB8 renamed /GPIO Expansion/IO.PB8
- net IO.PB9 renamed /GPIO Expansion/IO.PB9
- net IO.RED renamed /GPIO Expansion/IO.RED
- net IO.RIGHT0 renamed /GPIO Expansion/IO.RIGHT0
- net IO.RIGHT1 renamed /GPIO Expansion/IO.RIGHT1
- net IO.RIGHT2 renamed /GPIO Expansion/IO.RIGHT2
- net IO.RIGHT3 renamed /GPIO Expansion/IO.RIGHT3
- net IO.RIGHT4 renamed /GPIO Expansion/IO.RIGHT4
- net IO.RIGHT5 renamed /GPIO Expansion/IO.RIGHT5
- net IO.RIGHT6 renamed /GPIO Expansion/IO.RIGHT6
- net IO.RIGHT7 renamed /GPIO Expansion/IO.RIGHT7
- U401 pad 15: Net-(JP409-Pad2) -> GND
- U401 pad 16: Net-(JP405-Pad2) -> GND
- U401 pad 17: Net-(JP401-Pad2) -> GND
- U402 pad 15: Net-(JP410-Pad2) -> +3V3
- U402 pad 16: Net-(JP406-Pad2) -> GND
- U402 pad 17: Net-(JP402-Pad2) -> GND
- U403 pad 15: Net-(JP411-Pad2) -> GND
- U403 pad 16: Net-(JP407-Pad2) -> +3V3
- U403 pad 17: Net-(JP403-Pad2) -> GND
- U404 pad 15: Net-(JP412-Pad2) -> +3V3
- U404 pad 16: Net-(JP408-Pad2) -> +3V3
- U404 pad 17: Net-(JP404-Pad2) -> GND
- U405 pad 15: Net-(JP421-Pad2) -> GND
- U405 pad 16: Net-(JP417-Pad2) -> GND
- U405 pad 17: Net-(JP413-Pad2) -> +3V3
- U406 pad 15: Net-(JP422-Pad2) -> +3V3
- U406 pad 16: Net-(JP418-Pad2) -> GND
- U406 pad 17: Net-(JP414-Pad2) -> +3V3
- U407 pad 15: Net-(JP423-Pad2) -> GND
- U407 pad 16: Net-(JP419-Pad2) -> +3V3
- U407 pad 17: Net-(JP415-Pad2) -> +3V3
- U408 pad 15: Net-(JP424-Pad2) -> +3V3
- U408 pad 16: Net-(JP420-Pad2) -> +3V3
- U408 pad 17: Net-(JP416-Pad2) -> +3V3
Routing:
- net +3V3: track 667.4 -> 515.6 mm, vias 34 -> 33
- net +5V: track 152.0 -> 45.8 mm, vias 2 -> 1
- net EXT5V_IN: track 38.8 -> 2.56 mm
- net CONN.SDA: track 34.5 -> 0.00 mm
- net CONN.SCK: track 29.4 -> 0.00 mm
- net Net-(JP410-Pad2): track 24.6 -> 0.00 mm, vias 2 -> 0
- net IO.SCK: track 271.7 -> 248.9 mm
- net Net-(JP412-Pad2): track 22.0 -> 0.00 mm, vias 2 -> 0
- net Net-(JP411-Pad2): track 21.7 -> 0.00 mm, vias 2 -> 0
- net Net-(JP423-Pad2): track 20.8 -> 0.00 mm, vias 2 -> 0
- net Net-(JP406-Pad2): track 18.7 -> 0.00 mm, vias 2 -> 0
- net Net-(JP403-Pad2): track 18.5 -> 0.00 mm, vias 2 -> 0
- net Net-(JP407-Pad2): track 18.4 -> 0.00 mm, vias 2 -> 0
- net IO.SDA: track 270.5 -> 252.6 mm
- net Net-(JP408-Pad2): track 17.2 -> 0.00 mm, vias 2 -> 0
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- removed copper zone on F.Cu, net +3V3
Other:
- outline, holes or cut-outs redrawn
- board text removed: "0"
- board text removed: "1"
- board text removed: "IOExp 0 [0 0 0]"
- board text removed: "IOExp 1 [0 0 1]"
- board text removed: "IOExp 2 [0 1 0]"
- board text removed: "IOExp 3 [0 1 1]"
- board text removed: "IOExp 4 [1 0 0]"
- board text removed: "IOExp 5 [1 0 1]"
- board text removed: "IOExp 6 [1 1 0]"
- board text removed: "IOExp 7 [1 1 1]"
- board text removed: "PWR INPUT"
