File: ECELab_v1.kicad_pcb (KiCad board)
At the start: 2 copper layers, 147.5 x 89.3 mm, 90 parts, among them J201 USB_C_Receptacle_USB2.0, J202 Conn_01x06_Male, J203 Conn_01x02_Male, J301 Conn_01x04_Male, J302 Conn_01x03_Male, J303 Conn_01x03_Male, U201 AZ1117IH-3.3TRG1, U301 FT232HQ-REEL, U302 93LC56BT-I/OT, U401 MCP23017_SS, U402 MCP23017_SS, U403 MCP23017_SS, U404 MCP23017_SS, U405 MCP23017_SS, U406 MCP23017_SS, U407 MCP23017_SS, U408 MCP23017_SS, U501 ICE40-HX8K_Breakout_Board, U601 RASPBERRY_PI_4B_4GB, Y301 12MHz

Commit message: Complete Design
Parts:
- removed C205, C206: 0.1u, Capacitor_SMD:C_0402_1005Metric
- removed D206: PMEG40, Diode_SMD:D_SOD-323
- removed FB202: 120R, Inductor_SMD:L_0603_1608Metric
- removed G*** (x2): LOGO, ECELab_Footprints:purduelogo
- removed J203: Conn_01x02_Male, Connector_PinHeader_2.54mm:PinHeader_1x02_P2.54mm_Horizontal
- added C401: 0.1u, Capacitor_SMD:C_0402_1005Metric, F.Cu at (128.7, 126.4)
- added C402: 0.1u, Capacitor_SMD:C_0402_1005Metric, F.Cu at (134.2, 126.4)
- added C403: 0.1u, Capacitor_SMD:C_0402_1005Metric, F.Cu at (139.3, 117.9)
- added C404: 0.1u, Capacitor_SMD:C_0402_1005Metric, F.Cu at (137.2, 113.9)
- added C405: 0.1u, Capacitor_SMD:C_0402_1005Metric, F.Cu at (126.1, 112.4)
- added C406: 0.1u, Capacitor_SMD:C_0402_1005Metric, F.Cu at (139.0, 120.9)
- added C407: 0.1u, Capacitor_SMD:C_0402_1005Metric, F.Cu at (124.6, 123.5)
- added C412: 3.3u, Capacitor_SMD:C_0402_1005Metric, F.Cu at (136.2, 112.8)
- added C413: 4.7u, Capacitor_SMD:C_0402_1005Metric, F.Cu at (122.5, 114.6)
- added C414: 0.1u, Capacitor_SMD:C_0402_1005Metric, F.Cu at (122.5, 113.5)
- added C415: 4.7u, Capacitor_SMD:C_0402_1005Metric, F.Cu at (122.7, 120.5)
- added C416: 0.1u, Capacitor_SMD:C_0402_1005Metric, F.Cu at (122.7, 121.6)
- added C417: 0.1u, Capacitor_SMD:C_0402_1005Metric, F.Cu at (115.5, 115.2)
- added C418: 0.1u, Capacitor_SMD:C_0402_1005Metric, F.Cu at (115.5, 111.8)
- added C423: 27p, Capacitor_SMD:C_0402_1005Metric, F.Cu at (122.5, 112.3)
- added C424: 27p, Capacitor_SMD:C_0402_1005Metric, F.Cu at (122.5, 111.0)
- added C425: 0.1u, Capacitor_SMD:C_0402_1005Metric, F.Cu at (126.8, 109.2)
- added C426: 0.1u, Capacitor_SMD:C_0402_1005Metric, F.Cu at (175.3, 145.8)
- added C427: 10n, Capacitor_SMD:C_0402_1005Metric, F.Cu at (184.0, 149.6)
- added D401: PMEG40, Diode_SMD:D_SOD-323, F.Cu at (116.1, 113.7)
- added FB401: 600R, Inductor_SMD:L_0603_1608Metric, F.Cu at (122.2, 116.0)
- added FB402: 600R, Inductor_SMD:L_0603_1608Metric, F.Cu at (122.2, 119.2)
- added FB403: 120R, Inductor_SMD:L_0603_1608Metric, F.Cu at (118.1, 111.8)
- added J401: USB_C_Receptacle_USB2.0, Connector_USB:USB_C_Receptacle_HRO_TYPE-C-31-M-12, F.Cu at (109.0, 117.7)
- added J402: Conn_01x02_Male, Connector_PinHeader_2.54mm:PinHeader_1x02_P2.54mm_Vertical, F.Cu at (165.6, 146.4)
- added J501: Conn_02x20_Odd_Even, Connector_PinHeader_2.54mm:PinHeader_2x20_P2.54mm_Vertical, F.Cu at (170.9, 83.5)
- added J502: Conn_02x20_Odd_Even, Connector_PinHeader_2.54mm:PinHeader_2x20_P2.54mm_Vertical, F.Cu at (180.1, 83.5)
- added J503: Conn_02x20_Odd_Even, Connector_PinHeader_2.54mm:PinHeader_2x20_P2.54mm_Vertical, F.Cu at (230.4, 83.5)
- added J504: Conn_02x20_Odd_Even, Connector_PinHeader_2.54mm:PinHeader_2x20_P2.54mm_Vertical, F.Cu at (239.5, 83.5)
- added J601: Raspberry Pi 4B, Connector_PinSocket_2.54mm:PinSocket_2x20_P2.54mm_Vertical, F.Cu at (156.7, 140.9)
- added R405: 12k, Resistor_SMD:R_0402_1005Metric, F.Cu at (122.7, 117.4)
- added R406: 12k, Resistor_SMD:R_0402_1005Metric, F.Cu at (122.7, 122.7)
- added R411: 10k, Resistor_SMD:R_0402_1005Metric, F.Cu at (135.9, 109.1)
- added R412: 10k, Resistor_SMD:R_0402_1005Metric, F.Cu at (127.8, 109.2)
- added R413: 10k, Resistor_SMD:R_0402_1005Metric, F.Cu at (128.9, 109.2)
- added R414: 5.1k, Resistor_SMD:R_0402_1005Metric, F.Cu at (115.5, 116.5)
- added R415: 5.1k, Resistor_SMD:R_0402_1005Metric, F.Cu at (115.7, 120.0)
- added R416: 2.2k, Resistor_SMD:R_0402_1005Metric, F.Cu at (134.8, 109.1)
- added R417: 8.2k, Resistor_SMD:R_0402_1005Metric, F.Cu at (184.1, 145.1)
- added R418: 68k, Resistor_SMD:R_0402_1005Metric, F.Cu at (184.1, 147.2)
- added REF**: MountingHole_3.5mm, MountingHole:MountingHole_3.5mm, F.Cu at (240.8, 72.0)
- added REF**: MountingHole_3.5mm, MountingHole:MountingHole_3.5mm, F.Cu at (172.2, 140.6)
- added REF**: MountingHole_3.5mm, MountingHole:MountingHole_3.5mm, F.Cu at (240.8, 140.6)
- added REF**: MountingHole_3.5mm, MountingHole:MountingHole_3.5mm, F.Cu at (172.2, 72.0)
- added U410: 93LC56BT-I/OT, Package_TO_SOT_SMD:SOT-23-6, F.Cu at (131.6, 108.7)
- added U411: NE555DR, Package_SO:SOIC-8_3.9x4.9mm_P1.27mm, F.Cu at (179.7, 147.2)
- added U415: FT4232HL-REEL, Package_QFP:LQFP-64_10x10mm_P0.5mm, F.Cu at (130.9, 118.7)
- added Y401: 12MHz, Crystal:Crystal_SMD_HC49-SD, F.Cu at (118.7, 107.7)
- J202: footprint Connector_PinHeader_2.54mm:PinHeader_1x06_P2.54mm_Horizontal -> Connector_PinHeader_2.54mm:PinHeader_1x06_P2.54mm_Vertical
- moved J302 95.9 mm to (142.5, 100.9)
- moved J303 95.9 mm to (137.7, 100.9)
- moved J301 68.4 mm to (116.3, 99.0)
- moved J202 59.8 mm to (129.8, 90.1), turned to 90 degrees
- moved R204 17.2 mm to (108.6, 130.5)
- moved D204 17.2 mm to (106.0, 130.5)
- moved D203 17.2 mm to (106.0, 128.2)
- moved R201 17.2 mm to (108.6, 128.2)
- moved C204 2.51 mm to (119.1, 141.3)
- moved C302 2.51 mm to (135.8, 146.0)
- moved C307 2.51 mm to (133.1, 144.4)
- moved C308 2.51 mm to (135.6, 134.1)
- moved C309 2.51 mm to (133.9, 135.4)
- moved FB301 2.51 mm to (132.8, 137.1)
- moved FB302 2.51 mm to (132.8, 142.8)
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- renumbered C401 to C408, C402 to C409, C403 to C410, C404 to C411, C405 to C419, C406 to C420, C407 to C421, C408 to C422, R417 to R407, R418 to R408, R419 to R409, R420 to R410, U405 to U406, U406 to U407, U407 to U408, U408 to U409
Connections:
- U401 pad 1: /GPIO Expansion/IO.HWCLK -> IO.HWCLK
- U401 pad 2: /GPIO Expansion/IO.PB20 -> IO.PB20
- U401 pad 21: /GPIO Expansion/IO.PB13 -> IO.PB13
- U401 pad 22: /GPIO Expansion/IO.PB12 -> IO.PB12
- U401 pad 23: /GPIO Expansion/IO.PB11 -> IO.PB11
- U401 pad 24: /GPIO Expansion/IO.PB10 -> IO.PB10
- U401 pad 25: /GPIO Expansion/IO.PB9 -> IO.PB9
- U401 pad 26: /GPIO Expansion/IO.PB8 -> IO.PB8
- U401 pad 3: /GPIO Expansion/IO.PB19 -> IO.PB19
- U401 pad 4: /GPIO Expansion/IO.PB18 -> IO.PB18
- U401 pad 5: /GPIO Expansion/IO.PB17 -> IO.PB17
- U401 pad 6: /GPIO Expansion/IO.PB16 -> IO.PB16
- U401 pad 7: /GPIO Expansion/IO.PB15 -> IO.PB15
- U401 pad 8: /GPIO Expansion/IO.PB14 -> IO.PB14
- U402 pad 1: /GPIO Expansion/IO.PB7 -> IO.PB7
- U402 pad 2: /GPIO Expansion/IO.PB6 -> IO.PB6
- U402 pad 21: IO.SS0_0 -> /GPIO Expansion/IO.SS0_0
- U402 pad 22: IO.SS0_1 -> /GPIO Expansion/IO.SS0_1
- U402 pad 23: IO.SS0_2 -> /GPIO Expansion/IO.SS0_2
- U402 pad 24: IO.SS0_3 -> /GPIO Expansion/IO.SS0_3
- U402 pad 25: IO.SS0_4 -> /GPIO Expansion/IO.SS0_4
- U402 pad 26: IO.SS0_5 -> /GPIO Expansion/IO.SS0_5
- U402 pad 27: IO.SS0_6 -> /GPIO Expansion/IO.SS0_6
- U402 pad 28: IO.SS0_7 -> /GPIO Expansion/IO.SS0_7
- U402 pad 3: /GPIO Expansion/IO.PB5 -> IO.PB5
- U402 pad 4: /GPIO Expansion/IO.PB4 -> IO.PB4
- U402 pad 5: /GPIO Expansion/IO.PB3 -> IO.PB3
- U402 pad 6: /GPIO Expansion/IO.PB2 -> IO.PB2
- U402 pad 7: /GPIO Expansion/IO.PB1 -> IO.PB1
- U402 pad 8: /GPIO Expansion/IO.PB0 -> IO.PB0
- U403 pad 1: IO.SS1_0 -> /GPIO Expansion/IO.SS1_0
- U403 pad 2: IO.SS1_1 -> /GPIO Expansion/IO.SS1_1
- U403 pad 21: IO.SS2_0 -> /GPIO Expansion/IO.SS2_0
- U403 pad 22: IO.SS2_1 -> /GPIO Expansion/IO.SS2_1
- U403 pad 23: IO.SS2_2 -> /GPIO Expansion/IO.SS2_2
- U403 pad 24: IO.SS2_3 -> /GPIO Expansion/IO.SS2_3
- U403 pad 25: IO.SS2_4 -> /GPIO Expansion/IO.SS2_4
- U403 pad 26: IO.SS2_5 -> /GPIO Expansion/IO.SS2_5
- U403 pad 27: IO.SS2_6 -> /GPIO Expansion/IO.SS2_6
- U403 pad 28: IO.SS2_7 -> /GPIO Expansion/IO.SS2_7
- U403 pad 3: IO.SS1_2 -> /GPIO Expansion/IO.SS1_2
- U403 pad 4: IO.SS1_3 -> /GPIO Expansion/IO.SS1_3
- U403 pad 5: IO.SS1_4 -> /GPIO Expansion/IO.SS1_4
- U403 pad 6: IO.SS1_5 -> /GPIO Expansion/IO.SS1_5
- U403 pad 7: IO.SS1_6 -> /GPIO Expansion/IO.SS1_6
- U403 pad 8: IO.SS1_7 -> /GPIO Expansion/IO.SS1_7
- U404 pad 1: IO.SS3_0 -> /GPIO Expansion/IO.SS3_0
- U404 pad 2: IO.SS3_1 -> /GPIO Expansion/IO.SS3_1
- U404 pad 3: IO.SS3_2 -> /GPIO Expansion/IO.SS3_2
- U404 pad 4: IO.SS3_3 -> /GPIO Expansion/IO.SS3_3
- U404 pad 5: IO.SS3_4 -> /GPIO Expansion/IO.SS3_4
- U404 pad 6: IO.SS3_5 -> /GPIO Expansion/IO.SS3_5
- U404 pad 7: IO.SS3_6 -> /GPIO Expansion/IO.SS3_6
- U404 pad 8: IO.SS3_7 -> /GPIO Expansion/IO.SS3_7
- U407 pad 21: /GPIO Expansion/IO.LEFT7 -> IO.LEFT7
- U407 pad 22: /GPIO Expansion/IO.LEFT6 -> IO.LEFT6
- U407 pad 23: /GPIO Expansion/IO.LEFT5 -> IO.LEFT5
- U407 pad 24: /GPIO Expansion/IO.LEFT4 -> IO.LEFT4
- U407 pad 25: /GPIO Expansion/IO.LEFT3 -> IO.LEFT3
- U407 pad 26: /GPIO Expansion/IO.LEFT2 -> IO.LEFT2
- U407 pad 27: /GPIO Expansion/IO.LEFT1 -> IO.LEFT1
- U407 pad 28: /GPIO Expansion/IO.LEFT0 -> IO.LEFT0
- U408 pad 1: /GPIO Expansion/IO.RIGHT7 -> IO.RIGHT7
- U408 pad 2: /GPIO Expansion/IO.RIGHT6 -> IO.RIGHT6
- U408 pad 21: /GPIO Expansion/IO.RED -> IO.RED
- U408 pad 22: /GPIO Expansion/IO.GREEN -> IO.GREEN
- U408 pad 23: /GPIO Expansion/IO.BLUE -> IO.BLUE
- U408 pad 3: /GPIO Expansion/IO.RIGHT5 -> IO.RIGHT5
- U408 pad 4: /GPIO Expansion/IO.RIGHT4 -> IO.RIGHT4
- U408 pad 5: /GPIO Expansion/IO.RIGHT3 -> IO.RIGHT3
- U408 pad 6: /GPIO Expansion/IO.RIGHT2 -> IO.RIGHT2
- U408 pad 7: /GPIO Expansion/IO.RIGHT1 -> IO.RIGHT1
- U408 pad 8: /GPIO Expansion/IO.RIGHT0 -> IO.RIGHT0
Routing:
- net +3V3: track 515.6 -> 758.2 mm, vias 33 -> 37
- net IO.RIGHT5: track 0.00 -> 195.5 mm, vias 0 -> 2
- net IO.RIGHT6: track 0.00 -> 195.0 mm, vias 0 -> 2
- net IO.RIGHT4: track 0.00 -> 181.2 mm, vias 0 -> 2
- net IO.RIGHT7: track 0.00 -> 179.7 mm, vias 0 -> 2
- net IO.RIGHT3: track 0.00 -> 175.3 mm, vias 0 -> 2
- net IO.LEFT0: track 0.00 -> 168.5 mm, vias 0 -> 3
- net IO.RIGHT2: track 0.00 -> 166.4 mm, vias 0 -> 2
- net IO.RIGHT1: track 0.00 -> 156.5 mm, vias 0 -> 2
- net IO.LEFT1: track 0.00 -> 156.2 mm, vias 0 -> 4
- net +5V: track 45.8 -> 197.1 mm, vias 1 -> 7
- net IO.RIGHT0: track 0.00 -> 148.6 mm, vias 0 -> 2
- net IO.LEFT2: track 0.00 -> 114.0 mm, vias 0 -> 2
- net IO.LEFT3: track 0.00 -> 104.4 mm, vias 0 -> 2
- net IO.LEFT4: track 0.00 -> 101.8 mm, vias 0 -> 2
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- added copper zone on In1.Cu, net GND
- added copper zone on In2.Cu, net GND
Other:
- outline, holes or cut-outs redrawn
- copper layers 2 -> 4
- board text added: "ECELabs PCB Design v1.2 Minh Nguyen Junfei Li"
- board text removed: "ECELab PCB Design v1 Minh Nguyen Junfei Li"
- board text removed: "EXT_5V"
- board text removed: "MODE"
- board text removed: "NOT INPUT"
- board text removed: "OUTPUT"
- board text removed: "Sel CONN: CONN.SDA=IO.SDA CONN.SCK=IO.SCK"
- board text removed: "Sel FTDI: FTDI.SDA=IO.SDA FTDI.SCK=IO.SCK"
