File: PSU.kicad_sch (KiCad schematic)
At the start: 25 parts

Commit message: Update
Parts:
- C201, C202: renamed from C?; footprint (none) -> Capacitor_SMD:C_0402_1005Metric
- C203, C204, C205, C206, C207, C208: renamed from C?; value 100n -> 0.1u; footprint Capacitor_SMD:C_0603_1608Metric -> Capacitor_SMD:C_0402_1005Metric
- D201, D202, D205, D206, D207: renamed from D?; footprint Diode_SMD:D_SOD-323_HandSoldering -> Diode_SMD:D_SOD-323
- FB201, FB202, FB203: renamed from FB?; footprint Inductor_SMD:L_0603_1608Metric_Pad1.05x0.95mm_HandSolder -> Inductor_SMD:L_0603_1608Metric
- U201: renamed from U?; value AZ1117-3.3 -> AZ1117IH-3.3TRG1
- gave numbers to parts that had none: 8
Connections:
- net +3.3V is gone; now on net +3V3: R204.1
Other:
- note added: "PWR Flags"
- note removed: "Mooring of PS and USB"

Commit message: Complete Draft 1 of PCB Design
Parts:
- added C209, C210: 0.1u, Capacitor_SMD:C_0402_1005Metric, symbol Device:C
- added D208: PMEG40, Diode_SMD:D_SOD-323, symbol Device:D_Schottky
- added FB204: 120R, Inductor_SMD:L_0603_1608Metric, symbol Device:FerriteBead
- added J203: Conn_01x06_Male, Connector_PinHeader_2.54mm:PinHeader_1x06_P2.54mm_Horizontal, symbol Connector:Conn_01x06_Male
- added TP201, TP202, TP203: TestPoint, TestPoint:TestPoint_Plated_Hole_D4.0mm, symbol Connector:TestPoint
- J202: footprint Connector_PinHeader_2.00mm:PinHeader_1x02_P2.00mm_Vertical -> Connector_PinHeader_2.54mm:PinHeader_1x02_P2.54mm_Horizontal
Connections:
- net +3V3: now also C210.1, FB204.2, J203.3 (Pin_3), J203.4 (Pin_4), TP202.1
- net +5V: now also J203.1 (Pin_1), J203.2 (Pin_2), TP201.1
- net GND: now also C209.2, C210.2, J203.5 (Pin_5), J203.6 (Pin_6), TP203.1
- new net: D208.1 (K), FB204.1
- new net PI4.3V3: C209.1, D208.2 (A)
Other:
- note added: "Pi4 3V3 Power"
- note added: "Test Points"

Commit message: Draft 1 complete
Parts:
- added TP204, TP205: TestPoint, TestPoint:TestPoint_Plated_Hole_D4.0mm, symbol Connector:TestPoint
- C201: LCSC (none) -> C76991; LCSC Part Number (none) -> C76991
- C202: LCSC (none) -> C907955; LCSC Part Number (none) -> C907955
- C203, C204, C205, C206, C207, C208, C209, C210: LCSC (none) -> C1525; LCSC Part Number (none) -> C1525
- D201, D202, D205, D206, D207, D208: LCSC (none) -> C36975; LCSC Part Number (none) -> C36975
- D203: LCSC (none) -> C136765; LCSC Part Number (none) -> C136765
- D204: LCSC (none) -> C131223; LCSC Part Number (none) -> C131223
- FB201, FB202, FB203, FB204: LCSC (none) -> C279682; LCSC Part Number (none) -> C279682
- J201: LCSC (none) -> C165948; LCSC Part Number (none) -> C165948
- J202: renamed from J203; LCSC (none) -> C56816; LCSC Part Number (none) -> C56816
- J203: renamed from J202; LCSC (none) -> C2905424; LCSC Part Number (none) -> C2905424
- R201: value 250 -> 220; LCSC (none) -> C25091; LCSC Part Number (none) -> C25091
- R202, R203: LCSC (none) -> C105872; LCSC Part Number (none) -> C105872
- R204: LCSC (none) -> C159101; LCSC Part Number (none) -> C159101
- U201: LCSC (none) -> C108495; LCSC Part Number (none) -> C108495
Connections:
- net EXT5V_IN: now also TP204.1
- net GND: now also TP205.1
Other:
- moved on the sheet: J202, TP201, TP202, TP203

Commit message: Update 1
Parts:
- removed J202: Conn_01x06_Male, Connector_PinHeader_2.54mm:PinHeader_1x06_P2.54mm_Horizontal, symbol Connector:Conn_01x06_Male
- removed TP201, TP202, TP203, TP204, TP205: TestPoint, TestPoint:TestPoint_Plated_Hole_D4.0mm, symbol Connector:TestPoint
- renumbered J203 to J202
Other:
- note removed: "Test Points"

Commit message: Update
Parts:
- removed C205, C206: 0.1u, Capacitor_SMD:C_0402_1005Metric, symbol Device:C
- removed D207: PMEG40, Diode_SMD:D_SOD-323, symbol Device:D_Schottky
- removed FB202: 120R, Inductor_SMD:L_0603_1608Metric, symbol Device:FerriteBead
- removed J202: Conn_01x02_Male, Connector_PinHeader_2.54mm:PinHeader_1x02_P2.54mm_Horizontal, symbol Connector:Conn_01x02_Male
- D201, D202, D205, D206: value PMEG40 -> PMEG3030EP,115; footprint Diode_SMD:D_SOD-323 -> Diode_SMD:D_SOD-128; LCSC C36975 -> C255587; LCSC Part Number C36975 -> C255587
- D207: renamed from D208; value PMEG40 -> PMEG3030EP,115; footprint Diode_SMD:D_SOD-323 -> Diode_SMD:D_SOD-128; LCSC C36975 -> C255587; LCSC Part Number C36975 -> C255587
- renumbered C207 to C205, C208 to C206, C209 to C207, C210 to C208, FB203 to FB202, FB204 to FB203
Connections:
- net EXT5V_IN is gone; now on net FPGA.3V3: D206.2 (A)
- net at D206.1 (K): now also FB202.1
Other:
- note removed: "External 5V PWR Supply and Protection Circuit"
- moved on the sheet: C205, C206, C207, C208, D207, FB202, FB203

Commit message: Update 2nd iteration
Parts:
- removed C205, C206: 0.1u, Capacitor_SMD:C_0402_1005Metric, symbol Device:C
- removed D201, D202, D205, D206, D207: PMEG3030EP,115, Diode_SMD:D_SOD-128, symbol Device:D_Schottky
- removed FB202: 120R, Inductor_SMD:L_0603_1608Metric, symbol Device:FerriteBead
- added D203: D5V0L1B2S9-7, Diode_SMD:D_SOD-923, symbol Device:D_TVS
- added D204: GBLC03CI, Diode_SMD:D_SOD-323, symbol Device:D_TVS
- added J201: Conn_01x03_Male, Connector_PinHeader_2.54mm:PinHeader_1x03_P2.54mm_Horizontal, symbol Connector:Conn_01x03_Male
- added TP201, TP202, TP203: TestPoint, TestPoint:TestPoint_Pad_D2.0mm, symbol Connector:TestPoint
- renumbered C207 to C205, C208 to C206, D203 to D201, D204 to D202, FB203 to FB202, J201 to J202
Connections:
- net +3V3: now also C202.1, U201.2 (VO), D204.2 (A2), J201.2 (Pin_2), TP202.1
- net +5V: now also C201.1, U201.3 (VI), D203.2 (A2), J201.3 (Pin_3), TP201.1
- net GND: now also D203.1 (A1), D204.1 (A1), J201.1 (Pin_1), TP203.1
- net PI4.3V3: now also FB202.1
- net PWRU_IN: now also FB201.1
Other:
- note removed: "FPGA 3V3 Power"
- moved on the sheet: C204, C205, C206, FB201, FB202

Commit message: Update 7/30
Parts:
- J201: footprint Connector_PinHeader_2.54mm:PinHeader_1x03_P2.54mm_Horizontal -> Connector_PinHeader_2.54mm:PinHeader_1x03_P2.54mm_Vertical
Changed lines of the file:
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@@
       (effects (font (size 1.27 1.27)) (justify right))
     )
-    (property "Footprint" "Connector_PinHeader_2.54mm:PinHeader_1x03_P2.54mm_Horizontal" (id 2) (at 234.95 40.64 0)
+    (property "Footprint" "Connector_PinHeader_2.54mm:PinHeader_1x03_P2.54mm_Vertical" (id 2) (at 234.95 40.64 0)
       (effects (font (size 1.27 1.27)) hide)
     )

Commit message: Update 8/2
Parts:
- added J203: Conn_01x02_Male, Connector_PinHeader_2.54mm:PinHeader_1x02_P2.54mm_Vertical, symbol Connector:Conn_01x02_Male
Connections:
- net +3V3: now also J201.3 (Pin_3), TP201.1; no longer J201.2 (Pin_2), TP202.1
- net +5V: now also J201.2 (Pin_2), TP202.1, J203.1 (Pin_1); no longer J201.3 (Pin_3), TP201.1
- net GND: now also J203.2 (Pin_2)
Changed lines of the file:
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@@
 (kicad_sch (version 20211123) (generator eeschema)
   (paper "A4")
+  (junction (at 124.46 109.855) (diameter 0) (color 0 0 0 0)
+  )
+  (junction (at 123.825 66.675) (diameter 0) (color 0 0 0 0)
+  )
+  (junction (at 204.492 40.64) (diameter 0) (color 0 0 0 0)
+  )
+  (junction (at 214.63 31.115) (diameter 0) (color 0 0 0 0)
+  )
+  (junction (at 214.63 40.64) (diameter 0) (color 0 0 0 0)
+  )
+  (junction (at 52.07 53.975) (diameter 0) (color 0 0 0 0)
+  )
+  (junction (at 100.33 100.965) (diameter 0) (color 0 0 0 0)
+  )
+  (junction (at 214.63 50.8) (diameter 0) (color 0 0 0 0)
+  )
+  (junction (at 52.07 48.895) (diameter 0) (color 0 0 0 0)
+  )
+  (junction (at 112.395 109.855) (diameter 0) (color 0 0 0 0)
+  )
+  (junction (at 113.665 75.565) (diameter 0) (color 0 0 0 0)
+  )
   (junction (at 204.47 31.115) (diameter 0) (color 0 0 0 0)
-  )
-  (junction (at 124.46 109.855) (diameter 0) (color 0 0 0 0)
-  )
-  (junction (at 123.825 66.675) (diameter 0) (color 0 0 0 0)
-  )
-  (junction (at 214.63 31.115) (diameter 0) (color 0 0 0 0)
-  )
-  (junction (at 214.63 40.64) (diameter 0) (color 0 0 0 0)
-  )
-  (junction (at 52.07 53.975) (diameter 0) (color 0 0 0 0)
-  )
-  (junction (at 100.33 100.965) (diameter 0) (color 0 0 0 0)
-  )
-  (junction (at 214.63 50.8) (diameter 0) (color 0 0 0 0)
-  )
-  (junction (at 52.07 48.895) (diameter 0) (color 0 0 0 0)
-  )
-  (junction (at 112.395 109.855) (diameter 0) (color 0 0 0 0)
-  )
-  (junction (at 113.665 75.565) (diameter 0) (color 0 0 0 0)
-  )
-  (junction (at 204.47 40.64) (diameter 0) (color 0 0 0 0)
   )
   (junction (at 123.19 32.385) (diameter 0) (color 0 0 0 0)
@@
     (stroke (width 0) (type default) (color 0 0 0 0))
   )
+  (wire (pts (xy 223.52 73.025) (xy 228.6 73.025))
+    (stroke (width 0) (type default) (color 0 0 0 0))
+  )
+  (wire (pts (xy 204.47 31.115) (xy 214.63 31.115))
+    (stroke (width 0) (type default) (color 0 0 0 0))
+  )
   (polyline (pts (xy 179.07 54.61) (xy 179.07 22.86))
     (stroke (width 0) (type default) (color 0 0 0 0))
@@
     (stroke (width 0) (type default) (color 0 0 0 0))
   )
+  (wire (pts (xy 204.492 40.64) (xy 214.63 40.64))
+    (stroke (width 0) (type default) (color 0 0 0 0))
+  )
   (polyline (pts (xy 144.78 54.61) (xy 179.07 54.61))
     (stroke (width 0) (type default) (color 0 0 0 0))
   )
-  (wire (pts (xy 204.47 31.115) (xy 214.63 31.115))
-    (stroke (width 0) (type default) (color 0 0 0 0))
-  )
   (wire (pts (xy 113.665 75.565) (xy 123.825 75.565))
     (stroke (width 0) (type default) (color 0 0 0 0))
@@
     (stroke (width 0) (type default) (color 0 0 0 0))
   )
+  (wire (pts (xy 223.52 70.485) (xy 228.6 70.485))
+    (stroke (width 0) (type default) (color 0 0 0 0))
+  )
   (wire (pts (xy 59.69 40.005) (xy 59.69 41.275))
     (stroke (width 0) (type default) (color 0 0 0 0))
@@
     (stroke (width 0) (type default) (color 0 0 0 0))
   )
-  (wire (pts (xy 204.47 40.64) (xy 214.63 40.64))
-    (stroke (width 0) (type default) (color 0 0 0 0))
-  )
   (wire (pts (xy 100.965 66.675) (xy 104.775 66.675))
     (stroke (width 0) (type default) (color 0 0 0 0))
@@
     (stroke (width 0) (type default) (color 0 0 0 0))
   )
-  (wire (pts (xy 194.31 40.64) (xy 204.47 40.64))
+  (wire (pts (xy 194.31 40.64) (xy 204.492 40.64))
     (stroke (width 0) (type default) (color 0 0 0 0))
   )
@@
     (effects (font (size 1.27 1.27)) (justify left))
   )
-  (symbol (lib_id "power:+5V") (at 204.47 31.115 0) (unit 1)
-    (in_bom yes) (on_board yes) (fields_autoplaced)
-    (property "Reference" "#PWR0201" (id 0) (at 204.47 34.925 0)
-      (effects (font (size 1.27 1.27)) hide)
-    )
-    (property "Value" "+5V" (id 1) (at 204.47 26.035 0))
-    (property "Footprint" "" (id 2) (at 204.47 31.115 0)
-      (effects (font (size 1.27 1.27)) hide)
-    )
-    (property "Datasheet" "" (id 3) (at 204.47 31.115 0)
-      (effects (font (size 1.27 1.27)) hide)
-    )
-    (pin "1")
-  )
   (symbol (lib_id "Device:LED") (at 163.83 44.45 180) (unit 1)
     (in_bom yes) (on_board yes) (fields_autoplaced)
@@
     (pin "2")
   )
+  (symbol (lib_id "Connector:Conn_01x02_Male") (at 218.44 70.485 0) (unit 1)
+    (in_bom yes) (on_board yes) (fields_autoplaced)
+    (property "Reference" "J203" (id 0) (at 219.075 64.77 0))
+    (property "Value" "Conn_01x02_Male" (id 1) (at 219.075 67.31 0))
+    (property "Footprint" "Connector_PinHeader_2.54mm:PinHeader_1x02_P2.54mm_Vertical" (id 2) (at 218.44 70.485 0)
+      (effects (font (size 1.27 1.27)) hide)
+    )
+    (property "Datasheet" "~" (id 3) (at 218.44 70.485 0)
+      (effects (font (size 1.27 1.27)) hide)
+    )
+    (pin "1")
+    (pin "2")
+  )
   (symbol (lib_id "power:GND") (at 63.5 40.005 0) (unit 1)
     (in_bom yes) (on_board yes) (fields_autoplaced)
@@
     (pin "1")
     (pin "2")
+  )
+  (symbol (lib_id "power:+3V3") (at 204.47 31.115 0) (unit 1)
+    (in_bom yes) (on_board yes) (fields_autoplaced)
+    (property "Reference" "#PWR?" (id 0) (at 204.47 34.925 0)
+      (effects (font (size 1.27 1.27)) hide)
+    )
+    (property "Value" "+3V3" (id 1) (at 204.47 25.4 0))
+    (property "Footprint" "" (id 2) (at 204.47 31.115 0)
+      (effects (font (size 1.27 1.27)) hide)
+    )
+    (property "Datasheet" "" (id 3) (at 204.47 31.115 0)
+      (effects (font (size 1.27 1.27)) hide)
+    )
+    (pin "1")
   )
   (symbol (lib_id "Connector:USB_C_Receptacle_USB2.0") (at 34.925 48.895 0) (unit 1)
@@
     (pin "2")
   )
+  (symbol (lib_id "power:+5V") (at 228.6 70.485 0) (unit 1)
+    (in_bom yes) (on_board yes) (fields_autoplaced)
+    (property "Reference" "#PWR0213" (id 0) (at 228.6 74.295 0)
+      (effects (font (size 1.27 1.27)) hide)
+    )
+    (property "Value" "+5V" (id 1) (at 228.6 65.405 0))
+    (property "Footprint" "" (id 2) (at 228.6 70.485 0)
+      (effects (font (size 1.27 1.27)) hide)
+    )
+    (property "Datasheet" "" (id 3) (at 228.6 70.485 0)
+      (effects (font (size 1.27 1.27)) hide)
+    )
+    (pin "1")
+  )
   (symbol (lib_id "power:PWR_FLAG") (at 194.31 50.8 0) (unit 1)
     (in_bom yes) (on_board yes) (fields_autoplaced)
@@
     (pin "2")
   )
+  (symbol (lib_id "power:GND") (at 228.6 73.025 0) (unit 1)
+    (in_bom yes) (on_board yes) (fields_autoplaced)
+    (property "Reference" "#PWR0216" (id 0) (at 228.6 79.375 0)
+      (effects (font (size 1.27 1.27)) hide)
+    )
+    (property "Value" "GND" (id 1) (at 228.6 78.105 0))
+    (property "Footprint" "" (id 2) (at 228.6 73.025 0)
+      (effects (font (size 1.27 1.27)) hide)
+    )
+    (property "Datasheet" "" (id 3) (at 228.6 73.025 0)
+      (effects (font (size 1.27 1.27)) hide)
+    )
+    (pin "1")
+  )
   (symbol (lib_id "Connector:TestPoint") (at 214.63 31.115 0) (unit 1)
     (in_bom yes) (on_board yes) (fields_autoplaced)
@@
   (symbol (lib_id "power:GND") (at 130.81 111.125 0) (unit 1)
     (in_bom yes) (on_board yes) (fields_autoplaced)
-    (property "Reference" "#PWR0217" (id 0) (at 130.81 117.475 0)
+    (property "Reference" "#PWR0219" (id 0) (at 130.81 117.475 0)
       (effects (font (size 1.27 1.27)) hide)
     )
@@
   (symbol (lib_id "power:+3V3") (at 133.985 100.965 0) (unit 1)
     (in_bom yes) (on_board yes) (fields_autoplaced)
-    (property "Reference" "#PWR0216" (id 0) (at 133.985 104.775 0)
+    (property "Reference" "#PWR0218" (id 0) (at 133.985 104.775 0)
       (effects (font (size 1.27 1.27)) hide)
     )
@@
   (symbol (lib_id "power:GND") (at 27.305 73.025 0) (unit 1)
     (in_bom yes) (on_board yes) (fields_autoplaced)
-    (property "Reference" "#PWR0213" (id 0) (at 27.305 79.375 0)
+    (property "Reference" "#PWR0214" (id 0) (at 27.305 79.375 0)
       (effects (font (size 1.27 1.27)) hide)
     )
@@
   (symbol (lib_id "power:GND") (at 108.585 76.835 0) (unit 1)
     (in_bom yes) (on_board yes) (fields_autoplaced)
-    (property "Reference" "#PWR0215" (id 0) (at 108.585 83.185 0)
+    (property "Reference" "#PWR0217" (id 0) (at 108.585 83.185 0)
       (effects (font (size 1.27 1.27)) hide)
     )
@@
   (symbol (lib_id "power:GND") (at 34.925 73.025 0) (unit 1)
     (in_bom yes) (on_board yes) (fields_autoplaced)
-    (property "Reference" "#PWR0214" (id 0) (at 34.925 79.375 0)
+    (property "Reference" "#PWR0215" (id 0) (at 34.925 79.375 0)
       (effects (font (size 1.27 1.27)) hide)
     )
@@
     )
     (property "Datasheet" "" (id 3) (at 34.925 73.025 0)
-      (effects (font (size 1.27 1.27)) hide)
-    )
-    (pin "1")
-  )
-  (symbol (lib_id "power:+3V3") (at 204.47 40.64 0) (unit 1)
-    (in_bom yes) (on_board yes) (fields_autoplaced)
-    (property "Reference" "#PWR0207" (id 0) (at 204.47 44.45 0)
-      (effects (font (size 1.27 1.27)) hide)
-    )
-    (property "Value" "+3V3" (id 1) (at 204.47 34.925 0))
-    (property "Footprint" "" (id 2) (at 204.47 40.64 0)
-      (effects (font (size 1.27 1.27)) hide)
-    )
-    (property "Datasheet" "" (id 3) (at 204.47 40.64 0)
       (effects (font (size 1.27 1.27)) hide)
     )
@@
     (pin "2")
   )
+  (symbol (lib_id "power:+5V") (at 204.492 40.64 0) (unit 1)
+    (in_bom yes) (on_board yes) (fields_autoplaced)
+    (property "Reference" "#PWR?" (id 0) (at 204.492 44.45 0)
+      (effects (font (size 1.27 1.27)) hide)
+    )
+    (property "Value" "+5V" (id 1) (at 204.492 35.56 0))
+    (property "Footprint" "" (id 2) (at 204.492 40.64 0)
+      (effects (font (size 1.27 1.27)) hide)
+    )
+    (property "Datasheet" "" (id 3) (at 204.492 40.64 0)
+      (effects (font (size 1.27 1.27)) hide)
+    )
+    (pin "1")
+  )
   (symbol (lib_id "Device:FerriteBead") (at 108.585 66.675 90) (unit 1)
