File: PSU.kicad_sch (KiCad schematic)
At the start: 25 parts, among them J201 USB_C_Receptacle_USB2.0, J202 Conn_01x02_Male, U201 AZ1117IH-3.3TRG1

Commit message: Complete SPI Design
Parts:
- added C209, C210: 0.1u, Capacitor_SMD:C_0402_1005Metric, symbol Device:C
- added D208: PMEG40, Diode_SMD:D_SOD-323, symbol Device:D_Schottky
- added FB204: 120R, Inductor_SMD:L_0603_1608Metric, symbol Device:FerriteBead
- added J202: Conn_01x06_Male, Connector_PinHeader_2.54mm:PinHeader_1x06_P2.54mm_Horizontal, symbol Connector:Conn_01x06_Male
- added TP201, TP202, TP203, TP204, TP205: TestPoint, TestPoint:TestPoint_Plated_Hole_D4.0mm, symbol Connector:TestPoint
- C201: LCSC (none) -> C76991; LCSC Part Number (none) -> C76991
- C202: LCSC (none) -> C907955; LCSC Part Number (none) -> C907955
- C203, C204, C205, C206, C207, C208: LCSC (none) -> C1525; LCSC Part Number (none) -> C1525
- D201, D202, D205, D206, D207: LCSC (none) -> C36975; LCSC Part Number (none) -> C36975
- D203: LCSC (none) -> C136765; LCSC Part Number (none) -> C136765
- D204: LCSC (none) -> C131223; LCSC Part Number (none) -> C131223
- FB201, FB202, FB203: LCSC (none) -> C279682; LCSC Part Number (none) -> C279682
- J201: LCSC (none) -> C165948; LCSC Part Number (none) -> C165948
- J203: renamed from J202; footprint Connector_PinHeader_2.00mm:PinHeader_1x02_P2.00mm_Vertical -> Connector_PinHeader_2.54mm:PinHeader_1x02_P2.54mm_Horizontal; LCSC (none) -> C2905424; LCSC Part Number (none) -> C2905424
- R201: value 250 -> 220; LCSC (none) -> C25091; LCSC Part Number (none) -> C25091
- R202, R203: LCSC (none) -> C105872; LCSC Part Number (none) -> C105872
- R204: LCSC (none) -> C159101; LCSC Part Number (none) -> C159101
- U201: LCSC (none) -> C108495; LCSC Part Number (none) -> C108495
Connections:
- net +3V3: now also C210.1, FB204.2, J202.3 (Pin_3), J202.4 (Pin_4), TP202.1
- net +5V: now also J202.1 (Pin_1), J202.2 (Pin_2), TP201.1
- net EXT5V_IN: now also TP204.1
- net GND: now also C209.2, C210.2, J202.5 (Pin_5), J202.6 (Pin_6), TP203.1, TP205.1
- new net: D208.1 (K), FB204.1
- new net PI4.3V3: C209.1, D208.2 (A)
Other:
- note added: "Pi4 3V3 Power"
- note added: "Test Points"

Commit message: Update to v1.2
Parts:
- removed TP201, TP202, TP203, TP204, TP205: TestPoint, TestPoint:TestPoint_Plated_Hole_D4.0mm, symbol Connector:TestPoint
Changed lines of the file:
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@@
-    (stroke (width 0) (type default) (color 0 0 0 0))
-  )
-  (wire (pts (xy 237.49 73.66) (xy 245.745 73.66))
     (stroke (width 0) (type default) (color 0 0 0 0))
   )
@@
     (stroke (width 0) (type default) (color 0 0 0 0))
   )
-  (wire (pts (xy 236.855 43.18) (xy 245.11 43.18))
-    (stroke (width 0) (type default) (color 0 0 0 0))
-  )
   (wire (pts (xy 50.165 38.735) (xy 51.435 38.735))
     (stroke (width 0) (type default) (color 0 0 0 0))
@@
     (stroke (width 0) (type default) (color 0 0 0 0))
   )
-  (wire (pts (xy 236.855 49.53) (xy 245.11 49.53))
-    (stroke (width 0) (type default) (color 0 0 0 0))
-  )
   (wire (pts (xy 63.5 117.475) (xy 63.5 118.745))
     (stroke (width 0) (type default) (color 0 0 0 0))
@@
     (stroke (width 0) (type default) (color 0 0 0 0))
   )
-  (wire (pts (xy 236.855 55.88) (xy 245.11 55.88))
-    (stroke (width 0) (type default) (color 0 0 0 0))
-  )
   (wire (pts (xy 35.56 99.695) (xy 38.1 99.695))
     (stroke (width 0) (type default) (color 0 0 0 0))
@@
   )
   (wire (pts (xy 210.82 58.42) (xy 210.82 59.055))
-    (stroke (width 0) (type default) (color 0 0 0 0))
-  )
-  (wire (pts (xy 237.49 86.36) (xy 245.745 86.36))
     (stroke (width 0) (type default) (color 0 0 0 0))
   )
@@
     (property "Sayfalar Arası Referanslar" "${INTERSHEET_REFS}" (id 0) (at 64.6129 33.5756 0)
       (effects (font (size 1.27 1.27)) (justify left) hide)
-    )
-  )
-  (global_label "EXT5V_IN" (shape input) (at 237.49 73.66 180) (fields_autoplaced)
-    (effects (font (size 1.27 1.27)) (justify right))
-    (property "Sayfalar Arası Referanslar" "${INTERSHEET_REFS}" (id 0) (at 226.5498 73.5806 0)
-      (effects (font (size 1.27 1.27)) (justify right) hide)
     )
   )
@@
     (pin "2")
   )
-  (symbol (lib_id "power:+5V") (at 236.855 43.18 0) (unit 1)
-    (in_bom yes) (on_board yes)
-    (property "Reference" "#PWR0207" (id 0) (at 236.855 46.99 0)
-      (effects (font (size 1.27 1.27)) hide)
-    )
-    (property "Value" "+5V" (id 1) (at 234.315 40.64 0))
-    (property "Footprint" "" (id 2) (at 236.855 43.18 0)
-      (effects (font (size 1.27 1.27)) hide)
-    )
-    (property "Datasheet" "" (id 3) (at 236.855 43.18 0)
-      (effects (font (size 1.27 1.27)) hide)
-    )
-    (pin "1")
-  )
   (symbol (lib_id "Device:D_Schottky") (at 128.27 32.385 180) (unit 1)
     (in_bom yes) (on_board yes)
@@
     (pin "2")
   )
-  (symbol (lib_id "Connector:TestPoint") (at 245.745 73.66 0) (unit 1)
-    (in_bom yes) (on_board yes) (fields_autoplaced)
-    (property "Reference" "TP204" (id 0) (at 247.65 69.0879 0)
-      (effects (font (size 1.27 1.27)) (justify left))
-    )
-    (property "Value" "TestPoint" (id 1) (at 247.65 71.6279 0)
-      (effects (font (size 1.27 1.27)) (justify left))
-    )
-    (property "Footprint" "TestPoint:TestPoint_Plated_Hole_D4.0mm" (id 2) (at 250.825 73.66 0)
-      (effects (font (size 1.27 1.27)) hide)
-    )
-    (property "Datasheet" "~" (id 3) (at 250.825 73.66 0)
-      (effects (font (size 1.27 1.27)) hide)
-    )
-    (pin "1")
-  )
   (symbol (lib_id "power:GND") (at 38.1 102.235 0) (unit 1)
     (in_bom yes) (on_board yes) (fields_autoplaced)
@@
     )
     (property "Datasheet" "" (id 3) (at 38.1 102.235 0)
-      (effects (font (size 1.27 1.27)) hide)
-    )
-    (pin "1")
-  )
-  (symbol (lib_id "power:GND") (at 237.49 86.36 0) (unit 1)
-    (in_bom yes) (on_board yes) (fields_autoplaced)
-    (property "Reference" "#PWR0221" (id 0) (at 237.49 92.71 0)
-      (effects (font (size 1.27 1.27)) hide)
-    )
-    (property "Value" "GND" (id 1) (at 237.49 91.44 0))
-    (property "Footprint" "" (id 2) (at 237.49 86.36 0)
-      (effects (font (size 1.27 1.27)) hide)
-    )
-    (property "Datasheet" "" (id 3) (at 237.49 86.36 0)
-      (effects (font (size 1.27 1.27)) hide)
-    )
-    (pin "1")
-  )
-  (symbol (lib_id "Connector:TestPoint") (at 245.11 55.88 0) (unit 1)
-    (in_bom yes) (on_board yes) (fields_autoplaced)
-    (property "Reference" "TP203" (id 0) (at 247.015 51.3079 0)
-      (effects (font (size 1.27 1.27)) (justify left))
-    )
-    (property "Value" "TestPoint" (id 1) (at 247.015 53.8479 0)
-      (effects (font (size 1.27 1.27)) (justify left))
-    )
-    (property "Footprint" "TestPoint:TestPoint_Plated_Hole_D4.0mm" (id 2) (at 250.19 55.88 0)
-      (effects (font (size 1.27 1.27)) hide)
-    )
-    (property "Datasheet" "~" (id 3) (at 250.19 55.88 0)
       (effects (font (size 1.27 1.27)) hide)
     )
@@
     (pin "1")
   )
-  (symbol (lib_id "Connector:TestPoint") (at 245.11 49.53 0) (unit 1)
-    (in_bom yes) (on_board yes) (fields_autoplaced)
-    (property "Reference" "TP202" (id 0) (at 247.015 44.9579 0)
-      (effects (font (size 1.27 1.27)) (justify left))
-    )
-    (property "Value" "TestPoint" (id 1) (at 247.015 47.4979 0)
-      (effects (font (size 1.27 1.27)) (justify left))
-    )
-    (property "Footprint" "TestPoint:TestPoint_Plated_Hole_D4.0mm" (id 2) (at 250.19 49.53 0)
-      (effects (font (size 1.27 1.27)) hide)
-    )
-    (property "Datasheet" "~" (id 3) (at 250.19 49.53 0)
-      (effects (font (size 1.27 1.27)) hide)
-    )
-    (pin "1")
-  )
   (symbol (lib_id "Device:C") (at 123.19 37.465 0) (unit 1)
     (in_bom yes) (on_board yes)
@@
     (pin "1")
   )
-  (symbol (lib_id "power:+3V3") (at 236.855 49.53 0) (unit 1)
-    (in_bom yes) (on_board yes)
-    (property "Reference" "#PWR0211" (id 0) (at 236.855 53.34 0)
-      (effects (font (size 1.27 1.27)) hide)
-    )
-    (property "Value" "+3V3" (id 1) (at 233.68 47.625 0))
-    (property "Footprint" "" (id 2) (at 236.855 49.53 0)
-      (effects (font (size 1.27 1.27)) hide)
-    )
-    (property "Datasheet" "" (id 3) (at 236.855 49.53 0)
-      (effects (font (size 1.27 1.27)) hide)
-    )
-    (pin "1")
-  )
   (symbol (lib_id "power:GND") (at 210.82 59.055 0) (unit 1)
     (in_bom yes) (on_board yes) (fields_autoplaced)
@@
     (pin "2")
   )
-  (symbol (lib_id "power:GND") (at 236.855 55.88 0) (unit 1)
-    (in_bom yes) (on_board yes) (fields_autoplaced)
-    (property "Reference" "#PWR0213" (id 0) (at 236.855 62.23 0)
-      (effects (font (size 1.27 1.27)) hide)
-    )
-    (property "Value" "GND" (id 1) (at 236.855 60.96 0))
-    (property "Footprint" "" (id 2) (at 236.855 55.88 0)
-      (effects (font (size 1.27 1.27)) hide)
-    )
-    (property "Datasheet" "" (id 3) (at 236.855 55.88 0)
-      (effects (font (size 1.27 1.27)) hide)
-    )
-    (pin "1")
-  )
   (symbol (lib_id "Device:C") (at 64.77 158.75 0) (unit 1)
     (in_bom yes) (on_board yes) (fields_autoplaced)
@@
     (pin "1")
   )
-  (symbol (lib_id "Connector:TestPoint") (at 245.745 86.36 0) (unit 1)
-    (in_bom yes) (on_board yes) (fields_autoplaced)
-    (property "Reference" "TP205" (id 0) (at 247.65 81.7879 0)
-      (effects (font (size 1.27 1.27)) (justify left))
-    )
-    (property "Value" "TestPoint" (id 1) (at 247.65 84.3279 0)
-      (effects (font (size 1.27 1.27)) (justify left))
-    )
-    (property "Footprint" "TestPoint:TestPoint_Plated_Hole_D4.0mm" (id 2) (at 250.825 86.36 0)
-      (effects (font (size 1.27 1.27)) hide)
-    )
-    (property "Datasheet" "~" (id 3) (at 250.825 86.36 0)
-      (effects (font (size 1.27 1.27)) hide)
-    )
-    (pin "1")
-  )
   (symbol (lib_id "power:GND") (at 112.395 76.835 0) (unit 1)
     (in_bom yes) (on_board yes) (fields_autoplaced)
@@
       (effects (font (size 1.27 1.27)) hide)
     )
-    (pin "1")
-  )
-  (symbol (lib_id "Connector:TestPoint") (at 245.11 43.18 0) (unit 1)
-    (in_bom yes) (on_board yes) (fields_autoplaced)
-    (property "Reference" "TP201" (id 0) (at 247.015 38.6079 0)
-      (effects (font (size 1.27 1.27)) (justify left))
-    )
-    (property "Value" "TestPoint" (id 1) (at 247.015 41.1479 0)
-      (effects (font (size 1.27 1.27)) (justify left))
-    )
-    (property "Footprint" "TestPoint:TestPoint_Plated_Hole_D4.0mm" (id 2) (at 250.19 43.18 0)
-      (effects (font (size 1.27 1.27)) hide)
-    )
-    (property "Datasheet" "~" (id 3) (at 250.19 43.18 0)
-      (effects (font (size 1.27 1.27)) hide)
-    )

Commit message: Complete Design
Parts:
- removed C205, C206: 0.1u, Capacitor_SMD:C_0402_1005Metric, symbol Device:C
- removed D206: PMEG40, Diode_SMD:D_SOD-323, symbol Device:D_Schottky
- removed FB202: 120R, Inductor_SMD:L_0603_1608Metric, symbol Device:FerriteBead
- removed J203: Conn_01x02_Male, Connector_PinHeader_2.54mm:PinHeader_1x02_P2.54mm_Horizontal, symbol Connector:Conn_01x02_Male
- J202: footprint Connector_PinHeader_2.54mm:PinHeader_1x06_P2.54mm_Horizontal -> Connector_PinHeader_2.54mm:PinHeader_1x06_P2.54mm_Vertical; LCSC C56816 -> (none); LCSC Part Number C56816 -> (none)
