File: PSU.kicad_sch (KiCad schematic)
At the start: 25 parts, among them J201 USB_C_Receptacle_USB2.0, J202 Conn_01x06_Male, U201 AZ1117IH-3.3TRG1

Commit message: Complete V1.3
Parts:
- D204: LCSC C131223 -> C165977; LCSC Part Number C131223 -> C165977
Changed lines of the file:
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@@
       (effects (font (size 1.27 1.27)) hide)
     )
-    (property "LCSC Part Number" "C131223" (id 4) (at 163.83 44.45 0)
+    (property "LCSC Part Number" "C165977" (id 4) (at 163.83 44.45 0)
       (effects (font (size 1.27 1.27)) hide)
     )
-    (property "LCSC" "C131223" (id 5) (at 163.83 44.45 0)
+    (property "LCSC" "C165977" (id 5) (at 163.83 44.45 0)
       (effects (font (size 1.27 1.27)) hide)
     )
