File: FTDI-GPIO.kicad_sch (KiCad schematic)
At the start: 30 parts, among them J301 Conn_02x06_Odd_Even, J302 Conn_01x04_Male, U301 FT2232HL, U302 93LC56BT-I/OT, Y301 12MHz

Commit message: Update 2nd iteration
Parts:
- removed C301, C302, C303, C304, C305, C306, C307, C310, C312, C315: 0.1u, Capacitor_SMD:C_0402_1005Metric, symbol Device:C
- removed C308: 3.3u, Capacitor_SMD:C_0402_1005Metric, symbol Device:C
- removed C309, C311: 4.7u, Capacitor_SMD:C_0402_1005Metric, symbol Device:C
- removed C313, C314: 27p, Capacitor_SMD:C_0402_1005Metric, symbol Device:C
- removed FB301, FB302: 600R, Inductor_SMD:L_0603_1608Metric, symbol Device:FerriteBead
- removed J301: Conn_02x06_Odd_Even, Connector_PinHeader_2.54mm:PinHeader_2x06_P2.54mm_Vertical, symbol Connector_Generic:Conn_02x06_Odd_Even
- removed J302: Conn_01x04_Male, Connector_PinHeader_2.54mm:PinHeader_1x04_P2.54mm_Horizontal, symbol Connector:Conn_01x04_Male
- removed R301, R302: 12k, Resistor_SMD:R_0402_1005Metric, symbol Device:R
- removed R303, R304, R305: 10k, Resistor_SMD:R_0402_1005Metric, symbol Device:R
- removed R306: 2.2k, Resistor_SMD:R_0402_1005Metric, symbol Device:R
- removed RN301, RN302: 10k, Resistor_SMD:R_Array_Convex_2x0402, symbol Device:R_Pack02
- removed U301: FT2232HL, Package_QFP:LQFP-64_10x10mm_P0.5mm, symbol Interface_USB:FT2232HL
- removed U302: 93LC56BT-I/OT, Package_TO_SOT_SMD:SOT-23-6, symbol Memory_EEPROM:93LCxxBxxOT
- removed Y301: 12MHz, Crystal:Crystal_SMD_HC49-SD, symbol Device:Crystal
- added C701, C702, C703, C704, C705, C706, C707, C710, C712, C715, C716, C717: 0.1u, Capacitor_SMD:C_0402_1005Metric, symbol Device:C
- added C708: 3.3u, Capacitor_SMD:C_0402_1005Metric, symbol Device:C
- added C709, C711: 4.7u, Capacitor_SMD:C_0402_1005Metric, symbol Device:C
- added C713, C714: 27p, Capacitor_SMD:C_0402_1005Metric, symbol Device:C
- added D701: D5V0L1B2S9-7, Diode_SMD:D_SOD-923, symbol Device:D_TVS
- added FB701, FB702: 600R, Inductor_SMD:L_0603_1608Metric, symbol Device:FerriteBead
- added FB703: 120R, Inductor_SMD:L_0603_1608Metric, symbol Device:FerriteBead
- added J701: Conn_02x02_Odd_Even, Connector_PinHeader_2.54mm:PinHeader_2x02_P2.54mm_Vertical, symbol Connector_Generic:Conn_02x02_Odd_Even
- added J702, J703: Conn_01x08_Male, Connector_PinHeader_2.54mm:PinHeader_1x08_P2.54mm_Vertical, symbol Connector:Conn_01x08_Male
- added J704: USB_C_Receptacle_USB2.0, Connector_USB:USB_C_Receptacle_HRO_TYPE-C-31-M-12, symbol Connector:USB_C_Receptacle_USB2.0
- added R701, R702: 12k, Resistor_SMD:R_0402_1005Metric, symbol Device:R
- added R703, R704, R705: 10k, Resistor_SMD:R_0402_1005Metric, symbol Device:R
- added R706, R707: 5.1k, Resistor_SMD:R_0402_1005Metric, symbol Device:R
- added R708: 2.2k, Resistor_SMD:R_0402_1005Metric, symbol Device:R
- added U701: FT2232HL, Package_QFP:LQFP-64_10x10mm_P0.5mm, symbol Interface_USB:FT2232HL
- added U702: 93LC56BT-I/OT, Package_TO_SOT_SMD:SOT-23-6, symbol Memory_EEPROM:93LCxxBxxOT
- added Y701: 12MHz, Crystal:Crystal_SMD_HC49-SD, symbol Device:Crystal
Connections:
- net +1V8: now also C705.1, C706.1, C707.1, C708.1, U701.12 (VCORE), U701.37 (VCORE), U701.49 (VREGOUT), U701.64 (VCORE)
- net +3V3: now also C701.1, C702.1, C703.1, C704.1, C715.1, FB701.1, FB702.1, J701.2 (Pin_2), J701.4 (Pin_4), R702.2, R703.1, R704.1, R705.1, U701.20 (VCCIO), U701.31 (VCCIO), U701.42 (VCCIO), U701.50 (VREGIN), U701.56 (VCCIO), U702.6 (VCC)
- net EECLK: now also R704.2, U701.62 (EECLK), U702.4 (CLK)
- net EECS: now also R705.2, U701.63 (EECS), U702.5 (CS)
- net EEDATA: now also R708.2, U701.61 (EEDATA), U702.3 (DI)
- net GND: now also C701.2, C702.2, C703.2, C704.2, C705.2, C706.2, C707.2, C708.2, C709.2, C710.2, C711.2, C712.2, C713.1, C714.1, C715.2, C716.2, C717.2, D701.1 (A1), J704.A1 (GND), J704.A12 (GND), J704.B1 (GND), J704.B12 (GND), J704.S1 (SHIELD), R701.2, R706.2, R707.1, U701.13 (TEST), U702.2 (GND)
- net VPHY: now also C709.1, C710.1, FB701.2, U701.4 (VPHY)
- net VPLL: now also C711.1, C712.1, FB702.2, U701.9 (VPLL)
- net XCSI: now also C713.2, U701.2 (OSCI), Y701.1
- net XCSO: now also C714.2, U701.3 (OSCO), Y701.2
- new net: R703.2, R708.1, U702.1 (DO)
- new net: J704.A5 (CC1), R706.1
- new net: J704.B5 (CC2), R707.2
- new net: R701.1, U701.6 (REF)
- new net: R702.1, U701.14 (~{RESET})
- new net: U701.1 (GND), U701.10 (AGND), U701.11 (GND), U701.15 (GND), U701.25 (GND), U701.35 (GND), U701.47 (GND), U701.5 (GND), U701.51 (GND)
- new net +5V: C717.1, D701.2 (A2), FB703.2
- new net FTDI2.D+: J704.A6 (D+), J704.B6 (D+), U701.8 (DP)
- new net FTDI2.D-: J704.A7 (D-), J704.B7 (D-), U701.7 (DM)
- new net IO.SS6_0: J703.1 (Pin_1), U701.43 (BDBUS4)
- new net IO.SS6_1: J703.2 (Pin_2), U701.44 (BDBUS5)
- new net IO.SS6_2: J703.3 (Pin_3), U701.45 (BDBUS6)
- new net IO.SS6_3: J703.4 (Pin_4), U701.46 (BDBUS7)
- new net IO.SS6_4: J703.5 (Pin_5), U701.48 (BCBUS0)
- new net IO.SS6_5: J703.6 (Pin_6), U701.52 (BCBUS1)
- new net IO.SS6_6: J703.7 (Pin_7), U701.53 (BCBUS2)
- new net IO.SS6_7: J703.8 (Pin_8), U701.54 (BCBUS3)
- new net IO.SS7_0: J702.1 (Pin_1), U701.22 (ADBUS5)
- new net IO.SS7_1: J702.2 (Pin_2), U701.23 (ADBUS6)
- new net IO.SS7_2: J702.3 (Pin_3), U701.24 (ADBUS7)
- new net IO.SS7_3: J702.4 (Pin_4), U701.26 (ACBUS0)
- new net IO.SS7_4: J702.5 (Pin_5), U701.27 (ACBUS1)
- new net IO.SS7_5: J702.6 (Pin_6), U701.28 (ACBUS2)
- new net IO.SS7_6: J702.7 (Pin_7), U701.29 (ACBUS3)
- new net IO.SS7_7: J702.8 (Pin_8), U701.30 (ACBUS4)
- new net MCP5.PWR: J701.1 (Pin_1)
- new net MCP5.SEL: J701.3 (Pin_3), U701.21 (ADBUS4)
- new net PWRU_IN2: C716.1, FB703.1, J704.A4 (VBUS), J704.A9 (VBUS), J704.B4 (VBUS), J704.B9 (VBUS)
- no-connect marks 28 -> 19
Other:
- note added: "USB PWR Filtering"
- note added: "USB_C"
- note removed: "FTDI USB-SPI & SPI Peripheral"
- note removed: "Jumper Headers for selecting FTDI or Header"

Commit message: Update 7/30
Parts:
- removed J701: Conn_02x02_Odd_Even, Connector_PinHeader_2.54mm:PinHeader_2x02_P2.54mm_Vertical, symbol Connector_Generic:Conn_02x02_Odd_Even
- added J702, J704: Conn_01x08_Male, Connector_PinHeader_2.54mm:PinHeader_1x08_P2.54mm_Vertical, symbol Connector:Conn_01x08_Male
- renumbered J702 to J701, J704 to J705
Connections:
- net MCP5.SEL is gone; now on net IO.SS7_4: U701.21 (ADBUS4)
- net GND: now also U701.1 (GND), U701.10 (AGND), U701.11 (GND), U701.15 (GND), U701.25 (GND), U701.35 (GND), U701.47 (GND), U701.5 (GND), U701.51 (GND)
- net IO.SS6_0: now also U701.26 (ACBUS0); no longer U701.43 (BDBUS4)
- net IO.SS6_1: now also U701.27 (ACBUS1); no longer U701.44 (BDBUS5)
- net IO.SS6_2: now also U701.28 (ACBUS2); no longer U701.45 (BDBUS6)
- net IO.SS6_3: now also U701.29 (ACBUS3); no longer U701.46 (BDBUS7)
- net IO.SS6_4: now also U701.30 (ACBUS4); no longer U701.48 (BCBUS0)
- net IO.SS6_5: now also U701.32 (ACBUS5); no longer U701.52 (BCBUS1)
- net IO.SS6_6: now also U701.33 (ACBUS6); no longer U701.53 (BCBUS2)
- net IO.SS6_7: now also U701.34 (ACBUS7); no longer U701.54 (BCBUS3)
- net IO.SS7_0: now also U701.16 (ADBUS0); no longer U701.22 (ADBUS5)
- net IO.SS7_1: now also U701.17 (ADBUS1); no longer U701.23 (ADBUS6)
- net IO.SS7_2: now also U701.18 (ADBUS2); no longer U701.24 (ADBUS7)
- net IO.SS7_3: now also U701.19 (ADBUS3); no longer U701.26 (ACBUS0)
- net IO.SS7_4: no longer U701.27 (ACBUS1)
- net IO.SS7_5: now also U701.22 (ADBUS5); no longer U701.28 (ACBUS2)
- net IO.SS7_6: now also U701.23 (ADBUS6); no longer U701.29 (ACBUS3)
- net IO.SS7_7: now also U701.24 (ADBUS7); no longer U701.30 (ACBUS4)
- net IO.LEFT0: now reaches U701.38 (BDBUS0)
- net IO.LEFT0: now also J702.1 (Pin_1)
- net IO.LEFT1: now reaches U701.39 (BDBUS1)
- net IO.LEFT1: now also J702.2 (Pin_2)
- net IO.LEFT2: now reaches U701.40 (BDBUS2)
- net IO.LEFT2: now also J702.3 (Pin_3)
- net IO.LEFT3: now reaches U701.41 (BDBUS3)
- net IO.LEFT3: now also J702.4 (Pin_4)
- net IO.RIGHT4: now reaches U701.55 (BCBUS4)
- net IO.RIGHT4: now also J704.5 (Pin_5)
- net IO.RIGHT5: now reaches U701.57 (BCBUS5)
- net IO.RIGHT5: now also J704.6 (Pin_6)
- net IO.RIGHT6: now reaches U701.58 (BCBUS6)
- net IO.RIGHT6: now also J704.7 (Pin_7)
- net IO.RIGHT7: now reaches U701.59 (BCBUS7)
- net IO.RIGHT7: now also J704.8 (Pin_8)
- new net IO.LEFT4: J702.5 (Pin_5), U701.43 (BDBUS4)
- new net IO.LEFT5: J702.6 (Pin_6), U701.44 (BDBUS5)
- new net IO.LEFT6: J702.7 (Pin_7), U701.45 (BDBUS6)
- new net IO.LEFT7: J702.8 (Pin_8), U701.46 (BDBUS7)
- new net IO.RIGHT0: J704.1 (Pin_1), U701.48 (BCBUS0)
- new net IO.RIGHT1: J704.2 (Pin_2), U701.52 (BCBUS1)
- new net IO.RIGHT2: J704.3 (Pin_3), U701.53 (BCBUS2)
- new net IO.RIGHT3: J704.4 (Pin_4), U701.54 (BCBUS3)
- no-connect marks 19 -> 4

Commit message: Update 8/2
Parts:
- removed J701, J702, J703, J704: Conn_01x08_Male, Connector_PinHeader_2.54mm:PinHeader_1x08_P2.54mm_Vertical, symbol Connector:Conn_01x08_Male
- renumbered J705 to J701
Connections:
- net EECLK renamed EECLK2
- net EECS renamed EECS2
- net EEDATA renamed EEDATA2
- net VPHY renamed VPHY2
- net VPLL renamed VPLL2

Commit message: Complete Design v2
Parts:
- U701: value FT2232HL -> FT4232HL-REEL; symbol Interface_USB:FT2232HL -> Interface_USB:FT4232H; LCSC C27882 -> C56742; LCSC Part Number C27882 -> C56742
Other:
- moved on the sheet: U701
Changed lines of the file:
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@@
   (junction (at 80.645 187.96) (diameter 0) (color 0 0 0 0)
   )
-  (junction (at 85.09 157.48) (diameter 0) (color 0 0 0 0)
+  (junction (at 85.09 154.94) (diameter 0) (color 0 0 0 0)
   )
   (junction (at 179.705 69.215) (diameter 0) (color 0 0 0 0)
@@
   (junction (at 176.53 69.215) (diameter 0) (color 0 0 0 0)
   )
-  (junction (at 74.93 157.48) (diameter 0) (color 0 0 0 0)
+  (junction (at 74.93 154.94) (diameter 0) (color 0 0 0 0)
   )
-  (junction (at 80.01 157.48) (diameter 0) (color 0 0 0 0)
+  (junction (at 80.01 154.94) (diameter 0) (color 0 0 0 0)
   )
   (junction (at 207.01 232.41) (diameter 0) (color 0 0 0 0)
   )
-  (junction (at 77.47 157.48) (diameter 0) (color 0 0 0 0)
+  (junction (at 77.47 154.94) (diameter 0) (color 0 0 0 0)
   )
   (junction (at 210.185 44.45) (diameter 0) (color 0 0 0 0)
@@
   (junction (at 95.25 43.18) (diameter 0) (color 0 0 0 0)
   )
-  (junction (at 87.63 157.48) (diameter 0) (color 0 0 0 0)
+  (junction (at 87.63 154.94) (diameter 0) (color 0 0 0 0)
   )
-  (junction (at 90.17 157.48) (diameter 0) (color 0 0 0 0)
+  (junction (at 90.17 154.94) (diameter 0) (color 0 0 0 0)
   )
   (junction (at 173.355 34.925) (diameter 0) (color 0 0 0 0)
@@
   (junction (at 223.52 69.215) (diameter 0) (color 0 0 0 0)
   )
-  (junction (at 82.55 157.48) (diameter 0) (color 0 0 0 0)
+  (junction (at 82.55 154.94) (diameter 0) (color 0 0 0 0)
   )
   (junction (at 145.415 205.74) (diameter 0) (color 0 0 0 0)
@@
     (stroke (width 0) (type default) (color 0 0 0 0))
   )
-  (wire (pts (xy 69.85 156.21) (xy 69.85 157.48))
+  (wire (pts (xy 69.85 153.67) (xy 69.85 154.94))
     (stroke (width 0) (type default) (color 0 0 0 0))
   )
@@
     (stroke (width 0) (type default) (color 0 0 0 0))
   )
-  (wire (pts (xy 69.85 157.48) (xy 74.93 157.48))
+  (wire (pts (xy 69.85 154.94) (xy 74.93 154.94))
     (stroke (width 0) (type default) (color 0 0 0 0))
   )
@@
     (stroke (width 0) (type default) (color 0 0 0 0))
   )
-  (wire (pts (xy 90.17 157.48) (xy 92.71 157.48))
+  (wire (pts (xy 90.17 154.94) (xy 92.71 154.94))
     (stroke (width 0) (type default) (color 0 0 0 0))
   )
@@
     (stroke (width 0) (type default) (color 0 0 0 0))
   )
-  (wire (pts (xy 85.09 157.48) (xy 87.63 157.48))
+  (wire (pts (xy 85.09 154.94) (xy 87.63 154.94))
     (stroke (width 0) (type default) (color 0 0 0 0))
   )
@@
     (stroke (width 0) (type default) (color 0 0 0 0))
   )
-  (wire (pts (xy 77.47 157.48) (xy 80.01 157.48))
+  (wire (pts (xy 77.47 154.94) (xy 80.01 154.94))
     (stroke (width 0) (type default) (color 0 0 0 0))
   )
@@
     (stroke (width 0) (type default) (color 0 0 0 0))
   )
-  (wire (pts (xy 87.63 156.21) (xy 87.63 157.48))
+  (wire (pts (xy 87.63 153.67) (xy 87.63 154.94))
     (stroke (width 0) (type default) (color 0 0 0 0))
   )
@@
     (stroke (width 0) (type default) (color 0 0 0 0))
   )
-  (wire (pts (xy 90.17 156.21) (xy 90.17 157.48))
+  (wire (pts (xy 90.17 153.67) (xy 90.17 154.94))
     (stroke (width 0) (type default) (color 0 0 0 0))
   )
@@
     (stroke (width 0) (type default) (color 0 0 0 0))
   )
-  (wire (pts (xy 87.63 157.48) (xy 90.17 157.48))
+  (wire (pts (xy 87.63 154.94) (xy 90.17 154.94))
     (stroke (width 0) (type default) (color 0 0 0 0))
   )
@@
     (stroke (width 0) (type default) (color 0 0 0 0))
   )
-  (wire (pts (xy 82.55 157.48) (xy 85.09 157.48))
+  (wire (pts (xy 82.55 154.94) (xy 85.09 154.94))
     (stroke (width 0) (type default) (color 0 0 0 0))
   )
@@
     (stroke (width 0) (type default) (color 0 0 0 0))
   )
-  (wire (pts (xy 82.55 157.48) (xy 82.55 159.385))
+  (wire (pts (xy 82.55 154.94) (xy 82.55 156.845))
     (stroke (width 0) (type default) (color 0 0 0 0))
   )
@@
     (stroke (width 0) (type default) (color 0 0 0 0))
   )
-  (wire (pts (xy 82.55 156.21) (xy 82.55 157.48))
+  (wire (pts (xy 82.55 153.67) (xy 82.55 154.94))
     (stroke (width 0) (type default) (color 0 0 0 0))
   )
@@
     (stroke (width 0) (type default) (color 0 0 0 0))
   )
-  (wire (pts (xy 92.71 156.21) (xy 92.71 157.48))
+  (wire (pts (xy 92.71 153.67) (xy 92.71 154.94))
     (stroke (width 0) (type default) (color 0 0 0 0))
   )
@@
     (stroke (width 0) (type default) (color 0 0 0 0))
   )
-  (wire (pts (xy 74.93 156.21) (xy 74.93 157.48))
+  (wire (pts (xy 74.93 153.67) (xy 74.93 154.94))
     (stroke (width 0) (type default) (color 0 0 0 0))
   )
@@
     (stroke (width 0) (type default) (color 0 0 0 0))
   )
-  (wire (pts (xy 77.47 156.21) (xy 77.47 157.48))
+  (wire (pts (xy 77.47 153.67) (xy 77.47 154.94))
     (stroke (width 0) (type default) (color 0 0 0 0))
   )
@@
     (stroke (width 0) (type default) (color 0 0 0 0))
   )
-  (wire (pts (xy 74.93 157.48) (xy 77.47 157.48))
+  (wire (pts (xy 74.93 154.94) (xy 77.47 154.94))
     (stroke (width 0) (type default) (color 0 0 0 0))
   )
@@
     (stroke (width 0) (type default) (color 0 0 0 0))
   )
-  (wire (pts (xy 85.09 156.21) (xy 85.09 157.48))
+  (wire (pts (xy 85.09 153.67) (xy 85.09 154.94))
     (stroke (width 0) (type default) (color 0 0 0 0))
   )
@@
     (stroke (width 0) (type default) (color 0 0 0 0))
   )
-  (wire (pts (xy 80.01 157.48) (xy 82.55 157.48))
+  (wire (pts (xy 80.01 154.94) (xy 82.55 154.94))
     (stroke (width 0) (type default) (color 0 0 0 0))
   )
@@
     (stroke (width 0) (type default) (color 0 0 0 0))
   )
-  (wire (pts (xy 80.01 156.21) (xy 80.01 157.48))
+  (wire (pts (xy 80.01 153.67) (xy 80.01 154.94))
     (stroke (width 0) (type default) (color 0 0 0 0))
   )
@@
     (pin "1")
   )
-  (symbol (lib_id "power:GND") (at 82.55 159.385 0) (unit 1)
+  (symbol (lib_id "power:GND") (at 82.55 156.845 0) (unit 1)
     (in_bom yes) (on_board yes) (fields_autoplaced)
-    (property "Reference" "#PWR0718" (id 0) (at 82.55 165.735 0)
+    (property "Reference" "#PWR0718" (id 0) (at 82.55 163.195 0)
       (effects (font (size 1.27 1.27)) hide)
     )
-    (property "Value" "GND" (id 1) (at 82.55 164.465 0))
-    (property "Footprint" "" (id 2) (at 82.55 159.385 0)
+    (property "Value" "GND" (id 1) (at 82.55 161.925 0))
+    (property "Footprint" "" (id 2) (at 82.55 156.845 0)
       (effects (font (size 1.27 1.27)) hide)
     )
-    (property "Datasheet" "" (id 3) (at 82.55 159.385 0)
+    (property "Datasheet" "" (id 3) (at 82.55 156.845 0)
       (effects (font (size 1.27 1.27)) hide)
     )
@@
     (pin "2")
   )
-  (symbol (lib_id "Interface_USB:FT2232HL") (at 85.09 100.33 0) (unit 1)
+  (symbol (lib_id "Interface_USB:FT4232H") (at 85.09 100.33 0) (unit 1)
     (in_bom yes) (on_board yes) (fields_autoplaced)
     (property "Reference" "U701" (id 0) (at 99.8094 42.545 0)
       (effects (font (size 1.27 1.27)) (justify left))
     )
-    (property "Value" "FT2232HL" (id 1) (at 99.8094 45.085 0)
+    (property "Value" "FT4232HL-REEL" (id 1) (at 99.8094 45.085 0)
       (effects (font (size 1.27 1.27)) (justify left))
     )
@@
       (effects (font (size 1.27 1.27)) hide)
     )
-    (property "Datasheet" "https://www.ftdichip.com/Support/Documents/DataSheets/ICs/DS_FT2232H.pdf" (id 3) (at 85.09 100.33 0)
+    (property "Datasheet" "https://ftdichip.com/wp-content/uploads/2020/08/DS_FT4232H.pdf" (id 3) (at 85.09 100.33 0)
       (effects (font (size 1.27 1.27)) hide)
     )
-    (property "LCSC" "C27882" (id 4) (at 85.09 100.33 0)
+    (property "LCSC" "C56742" (id 4) (at 85.09 100.33 0)
       (effects (font (size 1.27 1.27)) hide)
     )
-    (property "LCSC Part Number" "C27882" (id 5) (at 85.09 100.33 0)
+    (property "LCSC Part Number" "C56742" (id 5) (at 85.09 100.33 0)
       (effects (font (size 1.27 1.27)) hide)
     )
