File: Pi4.kicad_sch (KiCad schematic)
At the start: 3 parts, among them U601 RASPBERRY_PI_4B_4GB

Commit message: Update 1
Connections:
- net IO.SCK: now also U601.5 (GPIO3/SCL1); no longer U601.23 (GPIO11/SPI_SCLK)
- net IO.IO0: now reaches U601.29 (GPIO5)
- net IO.SDA: now reaches U601.3 (GPIO2/SDA1)
- net IO.IO1: now reaches U601.31 (GPIO6)
- net IO.IO2: now reaches U601.32 (GPIO12)
- net IO.IO3: now reaches U601.33 (GPIO13)
- net IO.SDI: no longer names the net of U601.21 (GPIO9/SPI_MISO)
- net IO.SDO: no longer names the net of U601.19 (GPIO10/SPI_MOSI)
- net IO.~{CS}: no longer names the net of U601.26 (GPIO7/~{SPI_CE1~{})
Changed lines of the file:
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@@
+    (stroke (width 0) (type default) (color 0 0 0 0))
+  )
+  (wire (pts (xy 74.93 69.215) (xy 78.74 69.215))
     (stroke (width 0) (type default) (color 0 0 0 0))
   )
@@
     (stroke (width 0) (type default) (color 0 0 0 0))
   )
-  (polyline (pts (xy 225.425 150.495) (xy 225.425 163.83))
+  (polyline (pts (xy 213.36 150.495) (xy 213.36 163.83))
     (stroke (width 0) (type default) (color 0 0 0 0))
   )
@@
   )
   (wire (pts (xy 147.32 71.12) (xy 152.4 71.12))
+    (stroke (width 0) (type default) (color 0 0 0 0))
+  )
+  (wire (pts (xy 129.54 81.915) (xy 132.08 81.915))
     (stroke (width 0) (type default) (color 0 0 0 0))
   )
@@
     (stroke (width 0) (type default) (color 0 0 0 0))
   )
-  (wire (pts (xy 74.93 102.235) (xy 78.74 102.235))
+  (wire (pts (xy 129.54 86.995) (xy 132.08 86.995))
     (stroke (width 0) (type default) (color 0 0 0 0))
   )
-  (polyline (pts (xy 225.425 163.83) (xy 278.765 163.83))
+  (polyline (pts (xy 213.36 163.83) (xy 278.765 163.83))
     (stroke (width 0) (type default) (color 0 0 0 0))
   )
@@
     (stroke (width 0) (type default) (color 0 0 0 0))
   )
+  (wire (pts (xy 129.54 89.535) (xy 132.08 89.535))
+    (stroke (width 0) (type default) (color 0 0 0 0))
+  )
   (wire (pts (xy 156.845 71.12) (xy 156.845 70.485))
     (stroke (width 0) (type default) (color 0 0 0 0))
@@
     (stroke (width 0) (type default) (color 0 0 0 0))
   )
+  (wire (pts (xy 129.54 84.455) (xy 132.08 84.455))
+    (stroke (width 0) (type default) (color 0 0 0 0))
+  )
   (wire (pts (xy 130.175 69.215) (xy 133.35 69.215))
     (stroke (width 0) (type default) (color 0 0 0 0))
   )
   (wire (pts (xy 129.54 67.945) (xy 130.175 67.945))
+    (stroke (width 0) (type default) (color 0 0 0 0))
+  )
+  (bus (pts (xy 245.745 156.845) (xy 256.54 156.845))
     (stroke (width 0) (type default) (color 0 0 0 0))
   )
@@
     (stroke (width 0) (type default) (color 0 0 0 0))
   )
-  (bus (pts (xy 252.095 158.75) (xy 254 158.75))
-    (stroke (width 0) (type default) (color 0 0 0 0))
-  )
   (wire (pts (xy 129.54 62.865) (xy 131.445 62.865))
     (stroke (width 0) (type default) (color 0 0 0 0))
@@
     (stroke (width 0) (type default) (color 0 0 0 0))
   )
-  (wire (pts (xy 74.93 109.855) (xy 78.74 109.855))
-    (stroke (width 0) (type default) (color 0 0 0 0))
-  )
   (wire (pts (xy 130.81 121.285) (xy 130.81 118.745))
     (stroke (width 0) (type default) (color 0 0 0 0))
@@
     (stroke (width 0) (type default) (color 0 0 0 0))
   )
-  (wire (pts (xy 74.93 107.315) (xy 78.74 107.315))
+  (wire (pts (xy 74.93 71.755) (xy 78.74 71.755))
     (stroke (width 0) (type default) (color 0 0 0 0))
   )
@@
     (stroke (width 0) (type default) (color 0 0 0 0))
   )
-  (wire (pts (xy 74.93 104.775) (xy 78.74 104.775))
+  (bus (pts (xy 238.76 153.035) (xy 255.27 153.035))
     (stroke (width 0) (type default) (color 0 0 0 0))
   )
@@
     (stroke (width 0) (type default) (color 0 0 0 0))
   )
-  (polyline (pts (xy 278.765 150.495) (xy 225.425 150.495))
+  (polyline (pts (xy 278.765 150.495) (xy 213.36 150.495))
     (stroke (width 0) (type default) (color 0 0 0 0))
   )
@@
     (effects (font (size 1.27 1.27) (thickness 0.254) bold) (justify left bottom))
   )
-  (global_label "IO.~{CS}" (shape output) (at 74.93 102.235 180) (fields_autoplaced)
+  (global_label "IO.SCK" (shape input) (at 74.93 71.755 180) (fields_autoplaced)
     (effects (font (size 1.27 1.27)) (justify right))
-    (property "Intersheet References" "${INTERSHEET_REFS}" (id 0) (at 67.4974 102.1556 0)
+    (property "Intersheet References" "${INTERSHEET_REFS}" (id 0) (at 66.2274 71.6756 0)
       (effects (font (size 1.27 1.27)) (justify right) hide)
     )
   )
-  (global_label "IO.SDO" (shape output) (at 74.93 107.315 180) (fields_autoplaced)
-    (effects (font (size 1.27 1.27)) (justify right))
-    (property "Intersheet References" "${INTERSHEET_REFS}" (id 0) (at 66.1669 107.2356 0)
-      (effects (font (size 1.27 1.27)) (justify right) hide)
+  (global_label "IO.IO0" (shape bidirectional) (at 132.08 81.915 0) (fields_autoplaced)
+    (effects (font (size 1.27 1.27)) (justify left))
+    (property "Intersheet References" "${INTERSHEET_REFS}" (id 0) (at 140.1779 81.8356 0)
+      (effects (font (size 1.27 1.27)) (justify left) hide)
     )
   )
@@
     )
   )
-  (global_label "IO{SCK, SDO, SDI, ~{CS}}" (shape bidirectional) (at 252.095 158.75 180) (fields_autoplaced)
+  (global_label "IO.IO3" (shape bidirectional) (at 132.08 89.535 0) (fields_autoplaced)
+    (effects (font (size 1.27 1.27)) (justify left))
+    (property "Intersheet References" "${INTERSHEET_REFS}" (id 0) (at 140.1779 89.4556 0)
+      (effects (font (size 1.27 1.27)) (justify left) hide)
+    )
+  )
+  (global_label "IO{IO0, IO1, IO2, IO3}" (shape bidirectional) (at 238.76 153.035 180) (fields_autoplaced)
     (effects (font (size 1.27 1.27)) (justify right))
-    (property "Intersheet References" "${INTERSHEET_REFS}" (id 0) (at 228.2129 158.6706 0)
+    (property "Intersheet References" "${INTERSHEET_REFS}" (id 0) (at 215.4221 152.9556 0)
       (effects (font (size 1.27 1.27)) (justify right) hide)
     )
   )
-  (global_label "IO.SCK" (shape output) (at 74.93 104.775 180) (fields_autoplaced)
+  (global_label "IO.IO1" (shape bidirectional) (at 132.08 84.455 0) (fields_autoplaced)
+    (effects (font (size 1.27 1.27)) (justify left))
+    (property "Intersheet References" "${INTERSHEET_REFS}" (id 0) (at 140.1779 84.3756 0)
+      (effects (font (size 1.27 1.27)) (justify left) hide)
+    )
+  )
+  (global_label "IO.IO2" (shape bidirectional) (at 132.08 86.995 0) (fields_autoplaced)
+    (effects (font (size 1.27 1.27)) (justify left))
+    (property "Intersheet References" "${INTERSHEET_REFS}" (id 0) (at 140.1779 86.9156 0)
+      (effects (font (size 1.27 1.27)) (justify left) hide)
+    )
+  )
+  (global_label "IO.SDA" (shape input) (at 74.93 69.215 180) (fields_autoplaced)
     (effects (font (size 1.27 1.27)) (justify right))
-    (property "Intersheet References" "${INTERSHEET_REFS}" (id 0) (at 66.2274 104.6956 0)
+    (property "Intersheet References" "${INTERSHEET_REFS}" (id 0) (at 66.4088 69.1356 0)
       (effects (font (size 1.27 1.27)) (justify right) hide)
     )
   )
-  (global_label "IO.SDI" (shape input) (at 74.93 109.855 180) (fields_autoplaced)
+  (global_label "IO{SCK, SDA}" (shape bidirectional) (at 245.745 156.845 180) (fields_autoplaced)
     (effects (font (size 1.27 1.27)) (justify right))
-    (property "Intersheet References" "${INTERSHEET_REFS}" (id 0) (at 66.8926 109.7756 0)
+    (property "Intersheet References" "${INTERSHEET_REFS}" (id 0) (at 230.8133 156.7656 0)
       (effects (font (size 1.27 1.27)) (justify right) hide)
     )
   )
-  (hierarchical_label "IO{SCK, SDO, SDI, ~{CS}}" (shape input) (at 254 158.75 0)
+  (hierarchical_label "IO{IO0, IO1, IO2, IO3}" (shape bidirectional) (at 255.27 153.035 0)
     (effects (font (size 1.27 1.27)) (justify left))
   )
+  (hierarchical_label "IO{SCK, SDA}" (shape input) (at 256.54 156.845 0)
+    (effects (font (size 1.27 1.27)) (justify left))
+  )

Commit message: Update 2nd iteration
Parts:
- added RN601: 10k, Resistor_SMD:R_Array_Convex_2x0402, symbol Device:R_Pack02
Connections:
- net INTA.MCP5: now reaches U601.11 (GPIO17/GPIO_GEN0)
- net INTA.MCP6: now reaches U601.12 (GPIO18/GPIO_GEN1)
- net INTB.MCP5: now reaches U601.13 (GPIO27/GPIO_GEN2)
- net INTB.MCP6: now reaches U601.15 (GPIO22/GPIO_GEN3)
- net INTA.MCP7: now reaches U601.16 (GPIO23/GPIO_GEN4)
- net INTB.MCP7: now reaches U601.18 (GPIO24/GPIO_GEN5)
- net IO.SDA0: now reaches U601.27 (ID_SD)
- net IO.SDA0: now also RN601.4 (R1.2)
- net IO.SCK0: now reaches U601.28 (ID_SC)
- net IO.SCK0: now also RN601.3 (R2.2)
- net INTA.MCP3: now reaches U601.35 (GPIO19)
- net INTB.MCP2: now reaches U601.36 (GPIO16)
- net INTB.MCP4: now reaches U601.37 (GPIO26)
- net INTB.MCP3: now reaches U601.38 (GPIO20)
- net INTA.MCP4: now reaches U601.40 (GPIO21)
- net IO.IO0 renamed INTA.MCP0
- net IO.IO1 renamed INTB.MCP0
- net IO.IO2 renamed INTA.MCP1
- net IO.IO3 renamed INTA.MCP2
- net IO.SCK renamed IO.SCK1
- net IO.SDA renamed IO.SDA1
- new net +3V3: RN601.1 (R1.1), RN601.2 (R2.1)
- no-connect marks 10 -> 17

Commit message: Update 7/30
Parts:
- added J601, J602: Conn_02x02_Odd_Even, Connector_PinHeader_2.54mm:PinHeader_2x02_P2.54mm_Vertical, symbol Connector_Generic:Conn_02x02_Odd_Even
Connections:
- net +3V3: now also J601.2 (Pin_2), J601.4 (Pin_4), J602.2 (Pin_2), J602.4 (Pin_4)
- net MCP5.SEL: now reaches U601.22 (GPIO25/GPIO_GEN6)
- net MCP5.SEL: now also J601.3 (Pin_3)
- net MCP6.SEL: now reaches U601.24 (GPIO8/~{SPI_CE0~{})
- net MCP6.SEL: now also J602.3 (Pin_3)
- new net MCP5.PWR: J601.1 (Pin_1)
- new net MCP6.PWR: J602.1 (Pin_1)
- no-connect marks 17 -> 15
Other:
- moved on the sheet: RN601

Commit message: Update 8/2
Connections:
- net INTA.MCP0: now also U601.31 (GPIO6); no longer U601.29 (GPIO5)
- net INTA.MCP1: now also U601.33 (GPIO13); no longer U601.32 (GPIO12)
- net INTA.MCP2: now also U601.29 (GPIO5); no longer U601.33 (GPIO13)
- net INTA.MCP3: now also U601.38 (GPIO20); no longer U601.35 (GPIO19)
- net INTA.MCP4: now also U601.35 (GPIO19); no longer U601.40 (GPIO21)
- net INTA.MCP5: now also U601.22 (GPIO25/GPIO_GEN6); no longer U601.11 (GPIO17/GPIO_GEN0)
- net INTB.MCP0: now also U601.32 (GPIO12); no longer U601.31 (GPIO6)
- net INTB.MCP2: now also U601.26 (GPIO7/~{SPI_CE1~{}); no longer U601.36 (GPIO16)
- net INTB.MCP3: now also U601.37 (GPIO26); no longer U601.38 (GPIO20)
- net INTB.MCP4: now also U601.36 (GPIO16); no longer U601.37 (GPIO26)
- net INTB.MCP5: now also U601.21 (GPIO9/SPI_MISO); no longer U601.13 (GPIO27/GPIO_GEN2)
- net INTB.MCP6: now also U601.11 (GPIO17/GPIO_GEN0); no longer U601.15 (GPIO22/GPIO_GEN3)
- net INTB.MCP7: now also U601.15 (GPIO22/GPIO_GEN3); no longer U601.18 (GPIO24/GPIO_GEN5)
- net MCP5.SEL: now also U601.24 (GPIO8/~{SPI_CE0~{}); no longer U601.22 (GPIO25/GPIO_GEN6)
- net MCP6.SEL: now also U601.40 (GPIO21); no longer U601.24 (GPIO8/~{SPI_CE0~{})

Commit message: Complete Design v2
Parts:
- removed U601: RASPBERRY_PI_4B_4GB, ECELab_Footprints:MODULE_RASPBERRY_PI_4B_4GB, symbol ECELab_PartsLibrary:RASPBERRY_PI_4B_4GB
- added J603: Raspberry Pi 4B, Connector_PinSocket_2.54mm:PinSocket_2x20_P2.54mm_Vertical, symbol Connector_Generic:Conn_02x20_Odd_Even
- J601, J602: LCSC (none) -> C492419; LCSC Part Number (none) -> C492419
Connections:
- net +5V: now also J603.2 (5V), J603.4 (5V)
- net GND: now also J603.14 (GND), J603.20 (GND), J603.25 (GND), J603.30 (GND), J603.34 (GND), J603.39 (GND), J603.6 (GND), J603.9 (GND)
- net INTA.MCP0: now also J603.31 (GPIO6)
- net INTA.MCP1: now also J603.33 (GPIO13)
- net INTA.MCP2: now also J603.29 (GPIO5)
- net INTA.MCP3: now also J603.38 (GPIO20)
- net INTA.MCP4: now also J603.35 (GPIO19)
- net INTA.MCP5: now also J603.22 (GPIO25/GPIO_GEN6)
- net INTA.MCP6: now also J603.12 (GPIO18/GPIO_GEN1)
- net INTA.MCP7: now also J603.16 (GPIO23/GPIO_GEN4)
- net INTB.MCP0: now also J603.32 (GPIO12)
- net INTB.MCP2: now also J603.26 (GPIO7/~{SPI_CE1~{})
- net INTB.MCP3: now also J603.37 (GPIO26)
- net INTB.MCP4: now also J603.36 (GPIO16)
- net INTB.MCP5: now also J603.21 (GPIO9/SPI_MISO)
- net INTB.MCP6: now also J603.11 (GPIO17/GPIO_GEN0)
- net INTB.MCP7: now also J603.15 (GPIO22/GPIO_GEN3)
- net IO.SCK0: now also J603.28 (ID_SC)
- net IO.SCK1: now also J603.5 (GPIO3/SCL1)
- net IO.SDA0: now also J603.27 (ID_SD)
- net IO.SDA1: now also J603.3 (GPIO2/SDA1)
- net MCP5.SEL: now also J603.24 (GPIO8/~{SPI_CE0~{})
- net MCP6.SEL: now also J603.40 (GPIO21)
- net PI4.3V3: now also J603.1 (3V3), J603.17 (3V3)
Changed lines of the file:
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@@
+      (effects (font (size 1.27 1.27)) hide)
+    )
+    (property "LCSC" "C492419" (id 4) (at 220.345 65.405 0)
+      (effects (font (size 1.27 1.27)) hide)
+    )
+    (property "LCSC Part Number" "C492419" (id 5) (at 220.345 65.405 0)
       (effects (font (size 1.27 1.27)) hide)
     )
@@
     (pin "4")
   )
-  (symbol (lib_id "ECELab_PartsLibrary:RASPBERRY_PI_4B_4GB") (at 104.14 94.615 0) (unit 1)
+  (symbol (lib_id "power:+5V") (at 152.4 60.96 0) (unit 1)
     (in_bom yes) (on_board yes) (fields_autoplaced)
-    (property "Reference" "U601" (id 0) (at 104.14 55.88 0))
-    (property "Value" "RASPBERRY_PI_4B_4GB" (id 1) (at 104.14 58.42 0))
-    (property "Footprint" "ECELab_Footprints:MODULE_RASPBERRY_PI_4B_4GB" (id 2) (at 104.14 94.615 0)
-      (effects (font (size 1.27 1.27)) (justify bottom) hide)
-    )
-    (property "Datasheet" "" (id 3) (at 104.14 94.615 0)
+    (property "Reference" "#PWR0601" (id 0) (at 152.4 64.77 0)
       (effects (font (size 1.27 1.27)) hide)
     )
-    (property "PARTREV" "4" (id 4) (at 104.14 94.615 0)
-      (effects (font (size 1.27 1.27)) (justify bottom) hide)
+    (property "Value" "+5V" (id 1) (at 152.4 55.88 0))
+    (property "Footprint" "" (id 2) (at 152.4 60.96 0)
+      (effects (font (size 1.27 1.27)) hide)
     )
-    (property "STANDARD" "Manufacturer Recommendations" (id 5) (at 104.14 94.615 0)
-      (effects (font (size 1.27 1.27)) (justify bottom) hide)
+    (property "Datasheet" "" (id 3) (at 152.4 60.96 0)
+      (effects (font (size 1.27 1.27)) hide)
     )
-    (property "SNAPEDA_PN" "RASPBERRY PI 4B/4GB" (id 6) (at 104.14 94.615 0)
-      (effects (font (size 1.27 1.27)) (justify bottom) hide)
+    (pin "1")
+  )
+  (symbol (lib_id "power:+3V3") (at 236.855 80.645 0) (unit 1)
+    (in_bom yes) (on_board yes) (fields_autoplaced)
+    (property "Reference" "#PWR0604" (id 0) (at 236.855 84.455 0)
+      (effects (font (size 1.27 1.27)) hide)
     )
-    (property "MAXIMUM_PACKAGE_HEIGHT" "16 mm" (id 7) (at 104.14 94.615 0)
-      (effects (font (size 1.27 1.27)) (justify bottom) hide)
+    (property "Value" "+3V3" (id 1) (at 236.855 75.565 0))
+    (property "Footprint" "" (id 2) (at 236.855 80.645 0)
+      (effects (font (size 1.27 1.27)) hide)
     )
-    (property "MANUFACTURER" "Raspberry Pi" (id 8) (at 104.14 94.615 0)
-      (effects (font (size 1.27 1.27)) (justify bottom) hide)
+    (property "Datasheet" "" (id 3) (at 236.855 80.645 0)
+      (effects (font (size 1.27 1.27)) hide)
+    )
+    (pin "1")
+  )
+  (symbol (lib_id "Connector_Generic:Conn_02x20_Odd_Even") (at 104.14 86.36 0) (unit 1)
+    (in_bom yes) (on_board yes) (fields_autoplaced)
+    (property "Reference" "J603" (id 0) (at 104.14 55.88 0))
+    (property "Value" "Raspberry Pi 4B" (id 1) (at 104.14 58.42 0))
+    (property "Footprint" "Connector_PinSocket_2.54mm:PinSocket_2x20_P2.54mm_Vertical" (id 2) (at 104.14 86.36 0)
+      (effects (font (size 1.27 1.27)) hide)
+    )
+    (property "Datasheet" "~" (id 3) (at 104.14 86.36 0)
+      (effects (font (size 1.27 1.27)) hide)
+    )
+    (property "LCSC" "C2977589" (id 4) (at 104.14 86.36 0)
+      (effects (font (size 1.27 1.27)) hide)
+    )
+    (property "LCSC Part Number" "C2977589" (id 5) (at 104.14 86.36 0)
+      (effects (font (size 1.27 1.27)) hide)
     )
     (pin "1")
@@
     (pin "S4")
   )
-  (symbol (lib_id "power:+5V") (at 152.4 60.96 0) (unit 1)
-    (in_bom yes) (on_board yes) (fields_autoplaced)
-    (property "Reference" "#PWR0601" (id 0) (at 152.4 64.77 0)
-      (effects (font (size 1.27 1.27)) hide)
-    )
-    (property "Value" "+5V" (id 1) (at 152.4 55.88 0))
-    (property "Footprint" "" (id 2) (at 152.4 60.96 0)
-      (effects (font (size 1.27 1.27)) hide)
-    )
-    (property "Datasheet" "" (id 3) (at 152.4 60.96 0)
-      (effects (font (size 1.27 1.27)) hide)
-    )
-    (pin "1")
-  )
-  (symbol (lib_id "power:+3V3") (at 236.855 80.645 0) (unit 1)
-    (in_bom yes) (on_board yes) (fields_autoplaced)
-    (property "Reference" "#PWR0604" (id 0) (at 236.855 84.455 0)
-      (effects (font (size 1.27 1.27)) hide)
-    )
-    (property "Value" "+3V3" (id 1) (at 236.855 75.565 0))
-    (property "Footprint" "" (id 2) (at 236.855 80.645 0)
-      (effects (font (size 1.27 1.27)) hide)
-    )
-    (property "Datasheet" "" (id 3) (at 236.855 80.645 0)
-      (effects (font (size 1.27 1.27)) hide)
-    )
-    (pin "1")
-  )
   (symbol (lib_id "power:GND") (at 130.81 135.255 0) (unit 1)
     (in_bom yes) (on_board yes) (fields_autoplaced)
@@
       (effects (font (size 1.27 1.27)) hide)
     )
+    (property "LCSC" "C492419" (id 4) (at 220.98 80.645 0)
+      (effects (font (size 1.27 1.27)) hide)
+    )
+    (property "LCSC Part Number" "C492419" (id 5) (at 220.98 80.645 0)
+      (effects (font (size 1.27 1.27)) hide)
+    )
