File: Pi4.kicad_sch (KiCad schematic)
At the start: 3 parts, among them U601 RASPBERRY_PI_4B_4GB

Commit message: Draft 1 complete
Parts:
- C601, C602: LCSC (none) -> C1525; LCSC Part Number (none) -> C1525
Changed lines of the file:
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@@
+      (effects (font (size 1.27 1.27)) hide)
+    )
+    (property "LCSC Part Number" "C1525" (id 4) (at 147.32 66.675 0)
+      (effects (font (size 1.27 1.27)) hide)
+    )
+    (property "LCSC" "C1525" (id 5) (at 147.32 66.675 0)
       (effects (font (size 1.27 1.27)) hide)
     )
@@
       (effects (font (size 1.27 1.27)) hide)
     )
+    (property "LCSC Part Number" "C1525" (id 4) (at 156.845 66.675 0)
+      (effects (font (size 1.27 1.27)) hide)
+    )
+    (property "LCSC" "C1525" (id 5) (at 156.845 66.675 0)
+      (effects (font (size 1.27 1.27)) hide)
+    )

Commit message: Complete Design
Parts:
- removed U601: RASPBERRY_PI_4B_4GB, ECELab_Footprints:MODULE_RASPBERRY_PI_4B_4GB, symbol ECELab_PartsLibrary:RASPBERRY_PI_4B_4GB
- added J601: Raspberry Pi 4B, Connector_PinSocket_2.54mm:PinSocket_2x20_P2.54mm_Vertical, symbol Connector_Generic:Conn_02x20_Odd_Even
Connections:
- net +5V: now also J601.2 (5V), J601.4 (5V)
- net GND: now also J601.14 (GND), J601.20 (GND), J601.25 (GND), J601.30 (GND), J601.34 (GND), J601.39 (GND), J601.6 (GND), J601.9 (GND)
- net IO.SCK: now also J601.5 (GPIO3/SCL1)
- net IO.SDA: now also J601.3 (GPIO2/SDA1)
- net PI4.3V3: now also J601.1 (3V3), J601.17 (3V3)
- no-connect marks 10 -> 34
Changed lines of the file:
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@@
   (no_connect (at 78.74 132.08))
   (no_connect (at 78.74 129.54))
+  (no_connect (at 78.74 104.775))
+  (no_connect (at 78.74 107.315))
+  (no_connect (at 78.74 109.855))
+  (no_connect (at 129.54 102.235))
+  (no_connect (at 129.54 74.295))
+  (no_connect (at 129.54 76.835))
+  (no_connect (at 129.54 81.915))
+  (no_connect (at 129.54 84.455))
+  (no_connect (at 129.54 86.995))
+  (no_connect (at 129.54 89.535))
+  (no_connect (at 129.54 92.075))
+  (no_connect (at 129.54 94.615))
+  (no_connect (at 129.54 97.155))
+  (no_connect (at 129.54 99.695))
+  (no_connect (at 78.74 74.295))
+  (no_connect (at 78.74 79.375))
+  (no_connect (at 78.74 81.915))
+  (no_connect (at 78.74 84.455))
+  (no_connect (at 78.74 86.995))
+  (no_connect (at 78.74 89.535))
+  (no_connect (at 78.74 92.075))
+  (no_connect (at 78.74 94.615))
+  (no_connect (at 78.74 99.695))
+  (no_connect (at 78.74 102.235))
   (wire (pts (xy 129.54 121.285) (xy 130.81 121.285))
     (stroke (width 0) (type default) (color 0 0 0 0))
@@
     (pin "2")
   )
-  (symbol (lib_id "power:GND") (at 152.4 72.39 0) (unit 1)
+  (symbol (lib_id "Connector_Generic:Conn_02x20_Odd_Even") (at 104.14 86.36 0) (unit 1)
     (in_bom yes) (on_board yes) (fields_autoplaced)
-    (property "Reference" "#PWR0602" (id 0) (at 152.4 78.74 0)
-      (effects (font (size 1.27 1.27)) hide)
-    )
-    (property "Value" "GND" (id 1) (at 152.4 77.47 0))
-    (property "Footprint" "" (id 2) (at 152.4 72.39 0)
-      (effects (font (size 1.27 1.27)) hide)
-    )
-    (property "Datasheet" "" (id 3) (at 152.4 72.39 0)
-      (effects (font (size 1.27 1.27)) hide)
-    )
-    (pin "1")
-  )
-  (symbol (lib_id "ECELab_PartsLibrary:RASPBERRY_PI_4B_4GB") (at 104.14 94.615 0) (unit 1)
-    (in_bom yes) (on_board yes) (fields_autoplaced)
-    (property "Reference" "U601" (id 0) (at 104.14 55.88 0))
-    (property "Value" "RASPBERRY_PI_4B_4GB" (id 1) (at 104.14 58.42 0))
-    (property "Footprint" "ECELab_Footprints:MODULE_RASPBERRY_PI_4B_4GB" (id 2) (at 104.14 94.615 0)
-      (effects (font (size 1.27 1.27)) (justify bottom) hide)
-    )
-    (property "Datasheet" "" (id 3) (at 104.14 94.615 0)
-      (effects (font (size 1.27 1.27)) hide)
-    )
-    (property "PARTREV" "4" (id 4) (at 104.14 94.615 0)
-      (effects (font (size 1.27 1.27)) (justify bottom) hide)
-    )
-    (property "STANDARD" "Manufacturer Recommendations" (id 5) (at 104.14 94.615 0)
-      (effects (font (size 1.27 1.27)) (justify bottom) hide)
-    )
-    (property "SNAPEDA_PN" "RASPBERRY PI 4B/4GB" (id 6) (at 104.14 94.615 0)
-      (effects (font (size 1.27 1.27)) (justify bottom) hide)
-    )
-    (property "MAXIMUM_PACKAGE_HEIGHT" "16 mm" (id 7) (at 104.14 94.615 0)
-      (effects (font (size 1.27 1.27)) (justify bottom) hide)
-    )
-    (property "MANUFACTURER" "Raspberry Pi" (id 8) (at 104.14 94.615 0)
-      (effects (font (size 1.27 1.27)) (justify bottom) hide)
+    (property "Reference" "J601" (id 0) (at 104.14 55.88 0))
+    (property "Value" "Raspberry Pi 4B" (id 1) (at 104.14 58.42 0))
+    (property "Footprint" "Connector_PinSocket_2.54mm:PinSocket_2x20_P2.54mm_Vertical" (id 2) (at 104.14 86.36 0)
+      (effects (font (size 1.27 1.27)) hide)
+    )
+    (property "Datasheet" "~" (id 3) (at 104.14 86.36 0)
+      (effects (font (size 1.27 1.27)) hide)
+    )
+    (property "LCSC" "C2977589" (id 4) (at 104.14 86.36 0)
+      (effects (font (size 1.27 1.27)) hide)
+    )
+    (property "LCSC Part Number" "C2977589" (id 5) (at 104.14 86.36 0)
+      (effects (font (size 1.27 1.27)) hide)
     )
     (pin "1")
@@
     (pin "S4")
   )
+  (symbol (lib_id "power:GND") (at 152.4 72.39 0) (unit 1)
+    (in_bom yes) (on_board yes) (fields_autoplaced)
+    (property "Reference" "#PWR0602" (id 0) (at 152.4 78.74 0)
+      (effects (font (size 1.27 1.27)) hide)
+    )
+    (property "Value" "GND" (id 1) (at 152.4 77.47 0))
+    (property "Footprint" "" (id 2) (at 152.4 72.39 0)
+      (effects (font (size 1.27 1.27)) hide)
+    )
+    (property "Datasheet" "" (id 3) (at 152.4 72.39 0)
+      (effects (font (size 1.27 1.27)) hide)
+    )
+    (pin "1")
+  )
   (symbol (lib_id "power:+5V") (at 152.4 60.96 0) (unit 1)
